File: ADC1.sch (EAGLE design)
At the start: 69 parts, among them IC1 STM32F303K8T6, IC2 TC7WZ07FK, IC3 ESP32-WROVER, J1 SJ-1608, J2 SJ-1608, J3 SJ-1608, J4 SJ-1608, J5 SJ-2012, J6 SJ-1608, J7 SJ-2012, J8 SJ-1608, X1 12MHz

Commit message: ほぼ完成
Parts:
- added C19, C25: 470p, my_rcl:C-1608
- added C20: 10u, my_rcl:C-3225
- added C21, C26, C27, C28, C29, C30, C32, C36, C37, C38, C39, C40, C41, C42, C44, C48, C49, C50, C51, C52, C53: 0.1u, my_rcl:C-1608
- added C22: 27p, my_rcl:C-1608
- added C23, C24: 1n, my_rcl:C-1608
- added C31, C33, C34, C35, C43, C45, C46, C47: 10u, my_rcl:C-2012
- added C54, C55: 100u, my_rcl:CPOLE2.5-8
- added CON1: USB-A, my_connector:USB-A
- added CON2: SWD_CON, my_connector:SWD_CON
- added DR1, DR2, DR3, DR4: HOLE-3.2, my_connector:HOLE-3.2
- added FB2, FB3, FB4: FB, my_rcl:FB
- added IC10: NJM11100, my_ic:NJM11100
- added IC11, IC9: 3.3V, my_ic:NJM2863
- added IC12: LME49721, my_ic:OPA-2-SOP
- added IC13: NJM4580, my_ic:OPA-2-SOP
- added IC14: NJM12888F18, my_ic:NJM12888
- added IC15: NJM2845-3.3, my_ic:78X-SOP
- added IC16: -5V, my_ic:79LX
- added IC17: +5V, my_ic:78LX
- added IC8: OCT_BUFFER-SO6, my_ic:OCT_BUFFER-SO6
- added J10, J9: SJ-1608, my_rcl:SJ-1608
- added R30, R31, R44, R45: 22, my_rcl:R-1608
- added R34, R35, R36, R37, R38, R39, R42, R43, R48: 1k, my_rcl:R-1608
- added R40: 0, my_rcl:R-1608J
- added R41: 10k, my_rcl:R-1608
- added R46: 6.8k, my_rcl:R-1608
- added R47: 2.4k, my_rcl:R-1608
- added TP10: ESP_EN, my_connector:TESTPIN
- added TP11: ESP_BOOT, my_connector:TESTPIN
- added TP12: ESP_TX, my_connector:TESTPIN
- added TP13, TP20: GND, my_connector:TESTPIN
- added TP14: ESP_RX, my_connector:TESTPIN
- added TP15, TP16, TP18: GND, my_connector:TESTPIN-BIG
- added TP17: V+, my_connector:TESTPIN-BIG
- added TP19: V-, my_connector:TESTPIN-BIG
- added TP4: VBUS, my_connector:TESTPIN
- added TP5: UART_3V3, my_connector:TESTPIN
- added TP6: UART_RX, my_connector:TESTPIN
- added TP7: UART_GND, my_connector:TESTPIN
- added TP8: UART_TX, my_connector:TESTPIN
- added TP9: +3V3D, my_connector:TESTPIN
- C11: value 1n -> 0.1u
- C12: value 1n -> 3300p
- C13: value 0.1u -> 1u; device my_rcl:C-1608 -> my_rcl:C-2012
- C14: value (none) -> 27p
- C16: value (none) -> 0.1u
- C17: value (none) -> 470p
- C18: device my_rcl:C-3216 -> my_rcl:C-2012
- C7: value 1u -> 10u
- IC1: value STM32F303K8T6 -> STM32G431KB; device my_ic:STM32F303K8T6 -> my_ic:STM32G431KB
- IC2: value TC7WZ07FK -> 7404; device my_ic:TC7WZ07FK -> my_ic:7404
- IC4: value (none) -> LME49721
- IC5: value (none) -> NJM4580
- IC6: value (none) -> MCP331X1; device my_ic:OPA-2-SOP -> my_ic:MCP331X1
- IC7: value (none) -> OCT_BUFFER-SO6; device my_ic:OPA-2-SOP -> my_ic:OCT_BUFFER-SO6
- J5: value SJ-2012 -> IN3_DC
- J6: value SJ-1608 -> IN1_DC; device my_rcl:SJ-1608 -> my_rcl:SJ-2012
- J7: value SJ-2012 -> SJ-1608; device my_rcl:SJ-2012 -> my_rcl:SJ-1608
- R12: value 10 -> 1k
- R13: value 10 -> 37; device my_rcl:R-1608 -> my_rcl:R-1608J
- R20: value 10k -> 1k
- R24, R25, R27: value 1k -> 37; device my_rcl:R-1608 -> my_rcl:R-1608J
- R28, R29: value 10k -> 37; device my_rcl:R-1608 -> my_rcl:R-1608J
- TP1: value AIN1 -> AIN3
- TP2: value AIN2 -> AIN1
Connections:
- removed net ADC2+: J2.2, J6.2, R12.1
- removed net ADC2-: J4.2, J8.2, R13.1
- removed net VCOM1: C13.1, IC4G$1.+IN, IC4G$2.+IN, IC6G$1.+IN, IC6G$2.+IN, R18.1, R19.2
- new net +1V8: C11.1, C33.1, IC14.VOUT, IC6.AVDD
- new net +5V: C41.1, C42.1, C46.1, C48.1, C50.1, IC12G$3.V+, IC13G$3.V+, IC17.OUT, IC4G$3.V+, IC5G$3.V+
- new net -5V: C47.2, C49.2, C51.2, IC13G$3.V-, IC16.OUT, IC5G$3.V-
- new net ADC3+: J1.2, R10.1
- new net ADC3-: J3.2, R11.1
- new net ADC_CNVST: IC2G$3.IN, R29.1
- new net ADC_SCK: IC2G$1.IN, R27.1
- new net ADC_SDO: IC2G$2.OUT, R28.1
- new net ESP_BOOT: IC3.GPIO0, TP11.1
- new net N$32: CON1.D-, R30.1
- new net N$33: CON1.D+, R31.1
- new net N$35: IC7.C, R38.2, R48.2
- new net N$38: R36.1, R37.2
- new net N$39: C29.1, IC4G$2.+IN, R20.2, R22.2
- new net N$40: R18.1, R19.2
- new net N$41: C27.1, IC12G$2.+IN, R23.1, R37.1
- new net N$42: IC12G$2.-IN, R12.1, R32.2
- new net N$43: C19.2, IC12G$1.-IN, R34.1, R35.2
- new net N$44: C30.1, IC12G$1.+IN, R23.2, R26.2
- new net N$45: IC13G$2.-IN, IC13G$2.OUT, R42.1
- new net N$46: IC12G$2.OUT, J2.1, R12.2
- new net N$47: C19.1, IC12G$1.OUT, J4.1, R32.1, R34.2
- new net N$48: C20.1, J6.1, TP2.1
- new net N$49: C20.2, IC13G$2.+IN, J6.2, R41.2
- new net N$50: IC1.PA7, R29.2
- new net N$51: C16.1, IC9.BYPASS
- new net N$52: C24.2, IC6.AIN+, R44.2
- new net N$53: C23.1, IC6.AIN-, R45.2
- new net N$54: IC1.PA4, R40.2
- new net N$55: C22.2, IC13G$1.+IN, R39.2
- new net N$56: C26.1, IC11.BYPASS
- new net N$57: C22.1, IC13G$1.OUT, R35.1, R43.2
- new net N$58: IC2G$5.OUT, IC2G$6.IN
- new net N$59: C32.1, IC14.BYPASS
- new net N$60: IC2G$4.OUT, IC2G$5.IN
- new net N$61: C36.1, IC10.BYPASS
- new net N$62: IC10.VADJ, R46.1, R47.2
- new net N$63: C42.2, IC12G$3.V-, J8.2
- new net N$64: C41.2, IC4G$3.V-, J10.2
- new net N$65: C43.1, FB4.2, IC15.IN
- new net N$66: C44.1, IC1.NRST
- new net UART_3V3: C37.1, IC7.A, IC8.V+, R48.1, TP5.1
- new net UART_GND: C37.2, IC8.GND, TP7.1
- new net UART_RX: R38.1, TP6.1
- new net UART_TX: IC8.OUT, TP8.1
- new net USB_DM: IC1.PA11, R30.2
- new net USB_DP: IC1.PA12, R31.2
- new net V+: C39.1, C40.1, C45.1, C52.1, C54.1, FB4.1, IC10.EN, IC10.VIN, IC11.CONTROL, IC11.VIN, IC14.CONTROL, IC14.VIN, IC17.IN, IC9.CONTROL, IC9.VIN, TP17.1
- new net V-: C53.2, C55.2, IC16.IN, TP19.1
- new net VBUS: CON1.VBUS, TP4.1
- new net VDDA: C3.1, C7.1, FB1.1, IC1.VDDA
- new net VREF: C34.1, FB3.1, IC10.VOUT, R36.2, R46.2
- net +3V3: now also C18.1, C38.1, FB1.2, IC7.V+, IC8.A, IC9.VOUT; no longer C6.1, FB1.1, IC2G$4.V+, R20.2, R28.2
- net +3V3A: now also C21.1, C31.1, FB2.1, IC11.VOUT, IC2G$7.V+; no longer C3.1, C7.1, FB1.2, IC1.VDDA/VREF+
- net +3V3D: now also C35.1, IC15.OUT, TP9.1
- net ADC1+: now also J4.2, R44.1; no longer J1.2, R10.1
- net ADC1-: now also J2.2, J7.2, R45.1; no longer J3.2, R11.1
- net DAC1: now also IC5G$2.+IN, R40.1; no longer IC1.PA6, IC7G$1.+IN
- net ESP_EN: now also TP10.1
- net ESP_RX: now also TP14.1
- net ESP_TX: now also TP12.1
- net GND: now also C12.2, C16.2, C18.2, C21.2, C23.2, C24.1, C25.2, C26.2, C27.2, C28.2, C29.2, C30.2, C31.2, C32.2, C33.2, C34.2, C35.2, C36.2, C38.2, C39.2, C40.2, C43.2, C44.2, C45.2, C46.2, C47.1, C48.2, C49.1, C50.2, C51.1, C52.2, C53.1, C54.2, C55.1, CON1.GND, CON1.XT, CON2.GND, IC1.BOOT0, IC1.VSSA, IC10.GND, IC11.GND, IC13G$1.-IN, IC14.GND, IC15.GND, IC16.GND, IC17.GND, IC2G$4.IN, IC2G$7.V-, IC6.GND, IC7.GND, IC9.GND, J10.1, J7.1, J8.1, R22.1, R26.1, R41.1, R47.1, TP13.1, TP15.1, TP16.1, TP18.1, TP20.1; no longer C12.1, IC2G$4.V-, R19.1, R23.1, R29.1, R33.1
- net N$14: now also C28.1, IC4G$1.+IN, R19.1, R20.1; no longer IC2G$1.P$1, R5.2
- net N$15: now also C6.1, FB2.2, IC6.DVIO, J9.2; no longer IC2G$2.P$2, R6.2
- net N$16: now also C12.1, C13.1, FB3.2, IC6.VREF; no longer IC2G$3.P$1, R7.2
- net N$19: now also IC2G$3.OUT, R13.2; no longer C12.2, IC1.PA4, R12.2
- net N$20: now also IC2G$2.IN, R25.2; no longer C11.1, IC1.PA5, R13.2
- net N$22: no longer R20.1
- net N$23: now also IC5G$1.OUT, R17.1; no longer R22.1, R23.2
- net N$24: now also IC5G$2.-IN, IC5G$2.OUT; no longer IC7G$1.-IN, IC7G$1.OUT
- net N$25: now also IC6.SDO, R25.1; no longer C18.1, J7.1, TP2.1
- net N$26: no longer J2.1
- net N$27: no longer J4.1
- net N$28: now also IC6.SCLK; no longer IC6G$1.-IN, R25.2
- net N$29: now also IC6.CNVST, R13.1; no longer C18.2, IC5G$2.+IN, J7.2, R28.1, R29.2
- net N$30: now also IC6.SDI, J9.1; no longer C16.2, IC6G$2.-IN, R26.1, R27.2
- net N$31: now also IC2G$1.OUT, R24.2; no longer IC5G$2.OUT, R27.1, R32.2
- net N$34: now also IC8.C; no longer IC5G$2.-IN, R32.1
- net N$36: now also IC1.PA5, R27.2; no longer IC6G$1.OUT, J6.1, R24.2
- net N$37: now also IC1.PA6, R28.2; no longer C16.1, IC6G$2.OUT, J8.1, R25.1, R26.2
- net N$4: now also C25.1, R39.1, R42.2, R43.1; no longer IC5G$1.OUT, R17.1, R22.2
- net SPI_MISO: now also R6.2; no longer IC2G$2.P$1
- net SPI_MOSI: now also R5.2; no longer IC2G$1.P$2
- net SPI_SCK: now also R7.2; no longer IC2G$3.P$2
- net STM_RX: now also IC1.PA10, IC7.OUT; no longer IC1.PA9
- net STM_TX: now also CON2.TX, IC1.PA9, R33.1; no longer IC1.PA10
- net SWCLK: now also CON2.SWCLK, IC1.PA14/SWCLK; no longer IC1.PA14
- net SWDIO: now also CON2.SWDIO, IC1.PA13/SWDIO; no longer IC1.PA13
Other:
- moved on the sheet: C11, C12, C13, C16, C18, C3, C4, C5, C6, C7, FB1, IC5G$2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

Commit message: 発注
Parts:
- removed R2, R3, R4: 37, my_rcl:R-1608J
- added C56: 10u, my_rcl:C-2012
- C13: value 1u -> 10u
- C4, C5: value 27p -> 22p
- IC1: value STM32G431KB -> STM32G431
- IC11, IC9: device my_ic:NJM2863 -> my_ic:TAR5SB33
- IC15: value NJM2845-3.3 -> LM1117GS; device my_ic:78X-SOP -> my_ic:LM1117GS
- R1: value 37 -> 10k; device my_rcl:R-1608J -> my_rcl:R-1608
Connections:
- removed net N$13: IC3.GPIO23, R4.1
- removed net N$50: IC1.PA7, R29.2
- removed net N$58: IC2G$5.OUT, IC2G$6.IN
- removed net N$60: IC2G$4.OUT, IC2G$5.IN
- net +3V3D: now also R1.2
- net ESP_BOOT: now also R1.1
- net GND: now also C56.2, IC13G$1.+IN, IC2G$6.IN; no longer IC13G$1.-IN, IC2G$4.IN
- net N$11: now also IC2G$5.IN, IC2G$6.OUT; no longer IC3.GPIO18, R2.1
- net N$12: now also IC2G$4.IN, IC2G$5.OUT; no longer IC3.GPIO19, R1.1
- net N$15: now also C56.1
- net N$55: now also IC13G$1.-IN; no longer IC13G$1.+IN
- net N$9: now also IC1.PB0, R29.2; no longer IC3.GPIO5, R3.1
- net SPI_CS: now also IC3.GPIO5; no longer R3.2
- net SPI_MISO: now also IC3.GPIO19; no longer R1.2
- net SPI_MOSI: now also IC3.GPIO23; no longer R4.2
- net SPI_SCK: now also IC3.GPIO18; no longer R2.2
Other:
- moved on the sheet: IC13G$1, IC15, IC2G$4, IC2G$6, J9, R1, R29
