File: ADC2.sch (EAGLE design)
At the start: 166 parts, among them IC1 FPGA CORE BOARD, IC10 AK1110, IC11 AD4001, IC12 TAR5SB33, IC13 74HC3G34, IC14 TC7WH74FU, IC15 NJM12888F18, IC16 TAR5SB33, IC2 OPA, IC3 OPA-DIFF, IC4 DCDC2, IC5 OPA-DIFF, IC6 OPA-DIFF, IC7 LM317-L, IC8 LM337-L, IC9 LM337-L, J1 DC, J10 ADC+, J11 GND, J12 ADC-, J2 DC, J3 VCOM, J4 GND, J5 VCOM, J6 V-, J7 V-, J8 V-, J9 V-, X1 12MHz

Commit message: AD4134
Parts:
- removed J10: ADC+, my_rcl:SJ-1608
- removed J11: GND, my_rcl:SJ-1608
- removed J12: ADC-, my_rcl:SJ-1608
- removed J5: VCOM, my_rcl:SJ-3-1608
- removed J6, J7, J8, J9: V-, my_rcl:SJ-3-2012
- removed JP1: GAIN, my_connector:PINHD-1X2
- added C65, C66, C67, C68, C69, C70, C71: 0.1u, my_rcl:C-1608
- added C72: 10u, my_rcl:C-1608
- added D2: LED, my_rcl:LED-SMD1608
- added FB7, FB8: FB, my_rcl:FB-1608FB
- added IC17: IOS6720FB, my_ic:SI8420
- added R48, R58: SDI, my_rcl:R-1608
- added R49, R59: LED, my_rcl:R-1608
- added R50: 10M, my_rcl:R-7.5
- added R51: ODR, my_rcl:R-1608
- added R52: DOUT, my_rcl:R-1608
- added R53: SUB, my_rcl:R-1608
- added R54: DCLK, my_rcl:R-1608
- added R55: SDO, my_rcl:R-1608
- added R56: CS, my_rcl:R-1608
- added R57: SCLK, my_rcl:R-1608
- added R60: 10k, my_rcl:R-1608
- added SW1: DC, my_connector:SS22E01G5
- added SW2: GAIN, my_connector:SW-1X3
- added TP13: GND, my_connector:TESTPIN
- added U1: DC-DC, my_ic:DC-DC
- C1, C2: device my_rcl:C-3225 -> my_rcl:C-5W
- C10: value 10u -> 1u; device my_rcl:C-2012 -> my_rcl:C-1608
- C11, C12: value 1n -> 0.1u
- C13: value 1.5n -> 100u; device my_rcl:C-1608 -> my_rcl:CPOLE2.5-6.5
- C14: value 1.5n -> 100u; device my_rcl:C-1608 -> my_rcl:CPOLE2.5-8
- C15: value 1u -> 100u; device my_rcl:C-1608 -> my_rcl:CPOLE2.5-8
- C16: value 1u -> 1n
- C17: value 0.1u -> 1n
- C19, C20: value 100u -> 0.1u; device my_rcl:CPOLE2.5-8 -> my_rcl:C-1608
- C23, C24: value 0.1u -> 270p
- C25, C26, C27: value 0.1u -> 10u; device my_rcl:C-1608 -> my_rcl:C-3216
- C28, C29: value 10p -> 100u; device my_rcl:C-1608 -> my_rcl:CPOLE2.5-6.5
- C30: value 0.1u -> 100u; device my_rcl:C-1608 -> my_rcl:CPOLE2.5-6.5
- C31, C62: value 0.1u -> 1u
- C32, C34: value 10u -> 1u; device my_rcl:C-3216 -> my_rcl:C-1608
- C33, C50: device my_rcl:C-3216 -> my_rcl:C-2012
- C35, C36: value 100u -> 10u; device my_rcl:CPOLE2.5-6.5 -> my_rcl:C-2012
- C37: value 100u -> 10u; device my_rcl:CPOLE2.5-6.5 -> my_rcl:C-3216
- C38: value 1u -> 0.1u
- C39, C40, C41: value 1u -> 10u; device my_rcl:C-1608 -> my_rcl:C-2012
- C42, C46, C52, C58, C64: value 10u -> 0.1u; device my_rcl:C-2012 -> my_rcl:C-1608
- C43: value 10u -> 0.1u; device my_rcl:C-3216 -> my_rcl:C-1608
- C44: value 470p -> 10u; device my_rcl:C-1608 -> my_rcl:C-2012
- C45: value 470p -> 0.1u
- C47: value 3300p -> 0.1u
- C48, C49, C53, C59, C61: value 0.1u -> 10u; device my_rcl:C-1608 -> my_rcl:C-2012
- C51: value DNP -> 0.1u
- C6: value 10p -> 0.1u
- C63: value 0.1u -> 10u
- C7: value 10p -> 1u
- C8: value 2.7n -> 100u; device my_rcl:C-1608 -> my_rcl:CPOLE2.5-8
- C9: value 2.7n -> 1u
- FB5, FB6: device my_rcl:FB -> my_rcl:FB-2012
- IC10: value AK1110 -> REF5040; device my_ic:AK1110 -> my_ic:REF5040
- IC11: value AD4001 -> 1.8V; device my_ic:MCP331X1 -> my_ic:TLV740
- IC12: value TAR5SB33 -> 1.8V; device my_ic:TAR5SB33 -> my_ic:TLV740
- IC13: value 74HC3G34 -> 2.7V; device my_ic:74HC3G34 -> my_ic:TLV740
- IC14: value TC7WH74FU -> ISO6720FB; device my_ic:TC7WH74FU -> my_ic:SI8420
- IC15: value NJM12888F18 -> ISO6720FB; device my_ic:NJM12888 -> my_ic:SI8420
- IC16: value TAR5SB33 -> IOS6720FB; device my_ic:TAR5SB33 -> my_ic:SI8420
- IC3: value OPA-DIFF -> 7808; device my_ic:OPA-DIFF -> my_ic:78LX
- IC4: value DCDC2 -> LM317-L; device my_ic:DCDC2 -> my_ic:LM317-L
- IC5, IC6: value OPA-DIFF -> LM337-L; device my_ic:OPA-DIFF -> my_ic:LM337-L
- IC7: value LM317-L -> OPA1633; device my_ic:LM317-L -> my_ic:OPA-DIFF
- IC8: value LM337-L -> AK1110; device my_ic:LM337-L -> my_ic:AK1110
- IC9: value LM337-L -> AD4134; device my_ic:LM337-L -> my_ic:AD4134
- J1, J2: value DC -> V-; device my_rcl:SJ-1608 -> my_rcl:SJ-3-2012
- J3: value VCOM -> ADC+; device my_rcl:SJ-3-1608 -> my_rcl:SJ-1608
- J4: value GND -> ADC-; device my_rcl:SJ-2012 -> my_rcl:SJ-1608
- R10, R11: value 100 -> 1k
- R13, R14: value 1k -> 360
- R17, R18: value 1k -> 680
- R19: value 1k -> 330
- R20, R21, R22, R23: value 1k -> 120
- R24, R26, R27, R29, R30, R31: value 1k -> 22
- R25, R28: value 3.6k -> 22
- R3, R4: value 10k -> 100k
- R32: value 1k -> 10k
- R33, R34: value 680 -> 10k
- R35: value 330 -> 10k
- R36, R37: value 120 -> 10k
- R38: value 120 -> 47k
- R39: value 22 -> 47k
- R40: value 22 -> 39
- R41: value 37 -> 5.1k
- R42: value 37 -> ODR
- R43: value 37 -> DOUT
- R44: value 37 -> DCLK
- R45: value 37 -> SDO; device my_rcl:R-1608J -> my_rcl:R-1608
- R46: value 37 -> CS; device my_rcl:R-1608J -> my_rcl:R-1608
- R47: value 5.1k -> SCLK
- R5: value 22 -> 360; device my_rcl:R-1608J -> my_rcl:R-1608
- R6, R7: value 22 -> 10; device my_rcl:R-1608J -> my_rcl:R-1608
- R8: value 22 -> 10k; device my_rcl:R-1608J -> my_rcl:R-1608
- R9: value 22 -> 1k; device my_rcl:R-1608J -> my_rcl:R-1608
- X1: value 12MHz -> 48MHz
Connections:
- removed net +3V3A: C48.1, C54.1, C58.1, FB6.1, IC12.VOUT, IC13G$4.V+, IC14G$1.!CLR, IC14G$1.!PR, IC14G$2.V+
- removed net ADC+_LPF: C44.2, IC11.AIN+, R39.2
- removed net ADC-_LPF: C45.1, IC11.AIN-, R40.2
- removed net ADC_CNVST: IC14G$1.D, R9.2
- removed net ADC_CNVST_CLOCKED: IC14G$1.Q, R42.2
- removed net ADC_CNVST_FB: R45.2, R8.2
- removed net ADC_SCK: IC13G$2.IN, R6.2
- removed net CLK_8MHZ: R46.2, X1.OUT
- removed net N$57: FB2.1, J4.2
- new net +1V8_ISO: C63.1, C64.1, C65.1, C66.1, C67.1, FB7.2, IC14.VDD1, IC15.VDD1, IC16.VDD2, IC17.VDD2
- new net +3.6V: C54.1, C7.1, C8.1, FB4.1, IC13.IN
- new net +3V3D: FB8.2, IC1.+3V3@1, IC1.+3V3@2, IC1.+3V3@3, IC1.+3V3@4, IC1.+3V3@5, IC1.+3V3@6
- new net +3V3D_ISO: C68.1, C69.1, C70.1, C71.1, C72.1, FB8.1, IC14.VDD2, IC15.VDD2, IC16.VDD1, IC17.VDD1
- new net +5V_DEL: C48.1, IC11.EN, IC12.EN, IC13.EN, R38.2, R39.2
- new net +8V: C13.1, C31.1, IC3.OUT, IC8.EN, IC8.VIN_LDO1, IC8.VIN_LDO2
- new net ADC_2V7: C43.1, C45.1, C55.1, C57.1, C61.1, IC11.IN, IC12.IN, IC13.OUT, IC9.LDION, R41.2
- new net ADC_AVDD1V8: C56.1, C60.1, IC9.AVDD1V8
- new net ADC_CLKVDD: C46.1, C49.1, IC9.CLKVDD
- new net ADC_CS: IC9.FORMAT0/CS, R46.1
- new net ADC_DCLK: IC9.DCLK, R44.1
- new net ADC_DOUT: IC9.DOUT0, R43.1
- new net ADC_DVDD1V8: C51.1, C53.1, IC9.DVDD1V8
- new net ADC_ODR: IC9.ODR, R42.1
- new net ADC_SCLK: IC9.FORMAT1/SCLK, R47.1
- new net AVDD5V: C34.1, C36.1, C41.1, C42.1, IC10.VIN, IC8.VOUT_LDO2, IC9.AVDD5
- new net DGND: C68.2, C69.2, C70.2, C71.2, C72.2, FB1.1, IC1.GND@1, IC1.GND@10, IC1.GND@11, IC1.GND@12, IC1.GND@13, IC1.GND@14, IC1.GND@15, IC1.GND@16, IC1.GND@17, IC1.GND@18, IC1.GND@19, IC1.GND@2, IC1.GND@20, IC1.GND@3, IC1.GND@4, IC1.GND@5, IC1.GND@6, IC1.GND@7, IC1.GND@8, IC1.GND@9, IC14.GND2, IC15.GND2, IC16.GND1, IC17.GND1, R50.2, TP13.1
- new net FPGA_CS: IC1.IO23N_35/L2, R56.2
- new net FPGA_DCLK: IC1.IO7P_34/R2, R54.2
- new net FPGA_DCLK_SUB: IC1.IO12P_35/D4, R53.2
- new net FPGA_DOUT: IC1.IO7N_34/R1, R52.2
- new net FPGA_LED: IC1.IO2N_34/M1, R59.2
- new net FPGA_ODR: IC1.IO4N_34/P1, R51.2
- new net FPGA_SCLK: IC1.IO23P_35/L3, R57.2
- new net FPGA_SDI: IC1.IO2P_34/M2, R58.2
- new net FPGA_SDO: IC1.IO22P_35/K1, R55.2
- new net N$60: IC9.MODE, R37.1
- new net N$61: IC9.!PDN, R32.1
- new net N$62: IC9.!RESET, R33.1
- new net N$64: IC9.PIN/SPI, R36.1
- new net OSC_CLK: IC9.XTAL2/IN, R40.1
- new net VREFCAP: C37.1, C38.1, IC9.REFCAP
- net +1V8: now also C47.1, C50.1, FB7.1, IC11.OUT, IC9.IOVDD, R32.2, R33.2, R34.2, R35.2, R36.2, R37.2; no longer C49.1, C60.1, IC11.AVDD, IC15.VOUT
- net +5V: now also C32.1, C35.1, C52.1, IC8.VOUT_LDO1, IC9.DVDD5, R38.1; no longer C40.1, C42.1, C56.1, C61.1, IC10.VOUT_LDO1, IC12.CONTROL, IC12.VIN, IC15.CONTROL, IC15.VIN, IC16.CONTROL, IC16.VIN, R47.2
- net +9V: now also C11.1, C28.1, IC4.OUT, IC7G$2.EN, IC7G$2.V+, R20.2; no longer C17.1, C26.1, C30.1, C35.1, IC3G$1.EN, IC3G$2.V+, IC5G$1.EN, IC5G$2.V+, IC6G$1.EN, IC6G$2.V+, IC7.OUT, R36.2
- net -5V: now also C30.2, IC6.OUT, J1.1, J2.1, R22.2; no longer C37.2, IC9.OUT, J6.1, J7.1, J8.1, J9.1, R38.2
- net -9V: now also C29.2, IC5.OUT, J1.3, J2.3, R21.2; no longer C36.2, IC8.OUT, J6.3, J7.3, J8.3, J9.3, R37.2
- net ADC+: now also J3.2, R24.1, R26.1, R28.1, R30.1; no longer J10.2, R39.1
- net ADC-: now also J4.2, R25.1, R27.1, R29.1, R31.1; no longer J11.2, J12.2, R40.1
- net ADC_SDI: now also IC9.DEC2/SDI, R48.1; no longer IC13G$1.IN, R5.2
- net ADC_SDO: now also IC9.DEC3/SDO, R45.1, R60.2; no longer IC13G$3.OUT, R7.2
- net ADC_VCOM: now also C33.2, IC7G$1.CM; no longer C10.1, IC6G$1.CM, J3.3, J5.3, R24.2
- net GND: now also C10.1, C11.2, C12.1, C13.2, C14.2, C15.1, C16.2, C18.2, C19.1, C25.2, C26.1, C28.2, C29.1, C30.1, C31.2, C34.2, C36.2, C37.2, C44.2, C6.2, C65.2, C66.2, C67.2, C7.2, D2.K, IC10.GND, IC13.GND, IC14.GND1, IC15.GND1, IC16.GND2, IC17.GND2, IC3.GND, IC8.GND_LDO1, IC8.GND_LDO2, IC8.GND_REG, IC8.HT, IC9.AGND1V8, IC9.AGND5, IC9.CLKGND, IC9.CLKSEL, IC9.DGND1V8, IC9.DGND5, IC9.IOGND, IC9.REFGND, R17.1, R18.2, R19.2, R39.1, R50.1, R60.1, SW1.SHIELD, U1.GND1, U1.GND2; no longer C10.2, C15.2, C16.1, C18.1, C19.2, C23.2, C24.1, C25.1, C26.2, C30.2, C31.1, C34.1, C36.1, C37.1, C44.1, IC1.GND1@7, IC1.GND1@8, IC1.GND@1, IC1.GND@10, IC1.GND@11, IC1.GND@12, IC1.GND@13, IC1.GND@14, IC1.GND@15, IC1.GND@16, IC1.GND@19, IC1.GND@2, IC1.GND@20, IC1.GND@3, IC1.GND@4, IC1.GND@5, IC1.GND@6, IC1.GND@7, IC1.GND@8, IC1.GND@9, IC10.GND_LDO1, IC10.GND_LDO2, IC10.GND_REG, IC10.HT, IC13G$4.V-, IC14G$2.V-, IC15.GND, IC16.GND, IC4.GND, J11.1, J3.1, J4.1, J5.1, R24.1, R33.1, R34.2, R35.2
- net N$1: now also R10.1, R7.2, R8.1; no longer R11.2, R12.1, R14.1
- net N$10: now also IC15.IN1, R44.2; no longer IC1.IO4P_34/N1, R6.1
- net N$11: now also IC9.AIN3-, R31.2; no longer IC14G$1.!Q, R45.1
- net N$12: now also R10.2, R12.1; no longer R14.2, R16.1
- net N$13: now also IC9.AIN3+, R30.2; no longer IC13G$1.OUT, R41.2
- net N$15: now also IC9.AIN2-, R29.2; no longer C53.1, C55.1, FB6.2, IC11.DVIO
- net N$16: now also IC15.IN2, R45.2; no longer C46.1, C47.1, FB5.2, IC11.VREF
- net N$17: now also IC14.OUT2, R52.1; no longer IC1.IO4N_34/P1, R7.1
- net N$18: now also IC9.AIN2+, R28.2; no longer IC14G$1.CK, R46.1
- net N$19: now also C17.1, R12.2, R14.1, R16.1; no longer C29.1, IC6G$1.-IN, R30.2, R32.1
- net N$2: now also IC9.VCM, R23.2; no longer C29.2, IC6G$1.+OUT, J12.1, R32.2
- net N$20: now also IC9.AIN1-, R27.2; no longer IC13G$3.IN, R44.2
- net N$21: now also IC14.OUT1, R51.1; no longer IC1.IO7P_34/R2, R9.1
- net N$22: now also C23.2, IC7G$1.-OUT, J3.1, R15.2; no longer C28.1, IC6G$1.+IN, R29.2, R31.1
- net N$24: now also C23.1, IC7G$1.+IN, R13.2; no longer C8.1, R19.2, R21.1
- net N$25: now also IC9.AIN1+, R26.2; no longer IC11.SDO, R44.1
- net N$26: now also C24.1, IC7G$1.-IN, R14.2; no longer C9.1, R20.2, R22.1
- net N$27: now also IC15.OUT1, R53.1, R54.1; no longer C13.1, IC5G$1.+IN, R26.2
- net N$28: now also IC9.AIN0-, R25.2; no longer IC11.SCLK, R43.1
- net N$29: now also IC9.AIN0+, R24.2; no longer IC11.CNVST, R42.1
- net N$3: now also R6.2, R8.2, R9.1; no longer R10.2, R12.2, R13.1
- net N$30: now also R40.2, X1.OUT; no longer IC11.SDI, R41.1
- net N$31: now also C24.2, IC7G$1.+OUT, J4.1, R16.2; no longer IC13G$2.OUT, R43.2
- net N$32: now also IC15.OUT2, R55.1; no longer C12.2, C13.2, IC5G$1.-OUT, R25.2, R29.1
- net N$33: now also IC16.OUT2, R47.2; no longer C11.2, C14.2, IC5G$1.+OUT, R28.2, R30.1
- net N$34: now also IC16.OUT1, R46.2; no longer C14.1, IC5G$1.-IN, R27.2
- net N$35: now also IC17.OUT2, R49.2; no longer C12.1, R22.2, R27.1, R28.1
- net N$36: now also IC17.OUT1, R48.2; no longer C11.1, R21.2, R25.1, R26.1
- net N$37: now also IC16.IN2, R57.1; no longer C7.2, IC3G$1.+OUT, R18.2, R20.1
- net N$38: now also IC16.IN1, R56.1; no longer C6.2, IC3G$1.-OUT, R17.2, R19.1
- net N$39: now also IC17.IN2, R59.1; no longer C7.1, IC3G$1.-IN, R16.2, R18.1
- net N$4: now also R11.1, R9.2; no longer R13.2, R15.1
- net N$40: now also IC17.IN1, R58.1; no longer C6.1, IC3G$1.+IN, R15.2, R17.1
- net N$41: now also SW1.C2; no longer J1.1
- net N$42: now also SW1.C1; no longer J2.1
- net N$43: now also SW1.A2; no longer J1.2
- net N$44: now also SW1.A1; no longer J2.2
- net N$45: now also R6.1, SW2.2; no longer JP1.1, R10.1
- net N$46: now also R5.1, R7.1, SW2.1; no longer JP1.2, R11.1
- net N$47: now also D2.A, R49.1; no longer IC5G$1.CM, J5.2
- net N$48: now also C44.1, IC10.NR; no longer C62.1, IC16.BYPASS
- net N$49: now also IC9.DEC1/DCLKMODE, R35.1; no longer IC3G$1.CM, J3.2
- net N$5: now also C16.1, R11.2, R13.1, R15.1; no longer C28.2, IC6G$1.-OUT, J10.1, R31.2
- net N$50: now also IC9.DEC0/DCLKIO, R34.1; no longer C27.2, IC5G$2.V-, J8.2
- net N$51: now also FB4.2, U1.+5V; no longer C22.2, IC3G$2.V-, J7.2
- net N$52: now also C12.2, J1.2; no longer C18.2, J6.2
- net N$53: now also C25.1, IC4.ADJ, R17.2, R20.1; no longer C32.1, IC7.ADJ, R33.2, R36.1
- net N$54: now also C26.2, IC5.ADJ, R18.1, R21.1; no longer C33.2, IC8.ADJ, R34.1, R37.1
- net N$55: now also C27.2, IC6.ADJ, R19.1, R22.1; no longer C34.2, IC9.ADJ, R35.1, R38.1
- net N$56: now also FB1.2, FB3.1; no longer C57.1, IC12.BYPASS
- net N$58: now also R41.1; no longer R47.1
- net N$59: now also R5.2, SW2.3; no longer C59.1, IC15.BYPASS
- net N$6: now also C39.1, IC8.NP_LDO2; no longer IC1.IO7N_34/R1, R8.1
- net N$7: now also C40.1, IC8.NP_LDO1; no longer C52.1, IC10.NP_LDO1
- net N$70: now also FB5.1, U1.V+; no longer FB3.1, IC4.V+
- net N$71: now also FB6.1, U1.V-; no longer FB4.1, IC4.V-
- net N$74: now also C22.2, IC7G$2.V-, J2.2; no longer C31.2, IC6G$2.V-, J9.2
- net N$75: now also FB2.2, U1.VIN+; no longer FB1.2, IC4.VIN+
- net N$76: now also FB3.2, U1.VIN-; no longer FB2.2, IC4.VIN-
- net N$8: now also IC14.IN1, R42.2; no longer C50.1, C51.1, IC10.NP_LDO2
- net N$9: now also IC14.IN2, R43.2; no longer IC1.IO2P_34/M2, R5.1
- net V+: now also C14.1, C18.1, C6.1, C9.1, FB5.2, IC3.IN, IC4.IN; no longer C15.1, C19.1, C23.1, C38.1, C39.1, FB3.2, IC10.EN, IC10.VIN_LDO1, IC10.VIN_LDO2, IC7.IN
- net V-: now also C10.2, C15.2, C19.2, FB6.2, IC5.IN, IC6.IN; no longer C16.2, C24.2, C25.2, FB4.2, IC8.IN, IC9.IN
- net VCC_OSC: now also C58.1, C59.1, IC12.OUT; no longer C63.1, C64.1, IC16.VOUT
- net VIN: now also FB2.1; no longer FB1.1
- net VREF: now also C62.1, IC10.VOUT, IC9.REFIN; no longer C41.1, C43.1, FB5.1, IC10.VOUT_LDO2, R23.2
Other:
- moved on the sheet: C1, C10, C11, C12, C16, C17, C18, C2, C21, C22, C23, C24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
