File: ADC2.sch (EAGLE design)
At the start: 186 parts, among them IC1 FPGA CORE BOARD, IC10 REF5040, IC11 1.8V, IC12 1.8V, IC13 2.7V, IC14 ISO6720FB, IC15 ISO6720FB, IC16 IOS6720FB, IC17 IOS6720FB, IC2 OPA, IC3 7808, IC4 LM317-L, IC5 LM337-L, IC6 LM337-L, IC7 OPA1633, IC8 AK1110, IC9 AD4134, J1 V-, J2 V-, J3 ADC+, J4 ADC-, SW1 DC, SW2 GAIN, U1 DC-DC, X1 48MHz

Commit message: 発注
Parts:
- removed J3: ADC+, my_rcl:SJ-1608
- removed J4: ADC-, my_rcl:SJ-1608
- added C73, C74: 47p, my_rcl:C-1608
- added D3: TVS, my_rcl:ZENER-SMD2
- added R61, R62: 50, my_rcl:R-1608
- R10, R11, R12, R15, R16, R9: device my_rcl:R-1608 -> my_rcl:R-2012
Connections:
- net ADC+: now also C74.1, R15.2, R61.2; no longer J3.2
- net ADC-: now also C73.2, R16.2, R62.2; no longer J4.2
- net AVDD5V: now also D3.C
- net GND: now also C73.1, C74.2, D3.A
- net N$22: now also R61.1; no longer J3.1, R15.2
- net N$31: now also R62.1; no longer J4.1, R16.2
Other:
- moved on the sheet: C1, C16, C17, C2, C23, C24, C3, C4, C5, IC2G$1, IC2G$2, IC7G$1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

Commit message: 発注
Parts:
- added C75, C76, C77: 0.1u, my_rcl:C-1608
- added C78: 10u, my_rcl:C-1608
- added C79, C80: 100p, my_rcl:C-1608
- added CON1: IN-, my_connector:SMA-142-0701-801
- added CON2: IN+, my_connector:SMA-142-0701-801
- added IC18: IOS6720FB, my_ic:SI8420
- added J3: CLKSEL, my_rcl:SJ-3-1608
- added R63, R64, R65, R66: 10k, my_rcl:R-1608
- added SW3: FSEL, my_rcl:DIPSW-4
- added TP14, TP15: GND, my_connector:TESTPIN
- added TP16: +9V, my_connector:TESTPIN
- added TP17: -9V, my_connector:TESTPIN
- added TP18: -5V, my_connector:TESTPIN
- C1: device my_rcl:C-5W -> my_rcl:C-1608
- C10, C62: value 1u -> 0.1u
- C11, C38, C68: value 0.1u -> 1u
- C12, C18, C19: value 0.1u -> 100u; device my_rcl:C-1608 -> my_rcl:CPOLE2.5-8
- C13: value 100u -> 1u; device my_rcl:CPOLE2.5-6.5 -> my_rcl:C-1608
- C14: value 100u -> 1u; device my_rcl:CPOLE2.5-8 -> my_rcl:C-1608
- C15: value 100u -> 0.1u; device my_rcl:CPOLE2.5-8 -> my_rcl:C-1608
- C16: value 1n -> 0.1u
- C17: value 1n -> 100u; device my_rcl:C-1608 -> my_rcl:CPOLE2.5-6.5
- C2: value 1u -> 1.5u
- C20, C21: value 0.1u -> 1n
- C23, C24: value 270p -> 0.1u
- C25, C26: value 10u -> 0.1u; device my_rcl:C-3216 -> my_rcl:C-1608
- C27: value 10u -> 270p; device my_rcl:C-3216 -> my_rcl:C-1608
- C28: value 100u -> 270p; device my_rcl:CPOLE2.5-6.5 -> my_rcl:C-1608
- C29, C30: value 100u -> 10u; device my_rcl:CPOLE2.5-6.5 -> my_rcl:C-3216
- C3: value DNP -> 1.5u; device my_rcl:C-1608 -> my_rcl:C-5W
- C31: value 1u -> 10u; device my_rcl:C-1608 -> my_rcl:C-3216
- C32: value 1u -> 68p
- C33: value 10u -> 68p; device my_rcl:C-2012 -> my_rcl:C-1608
- C34: value 1u -> 100u; device my_rcl:C-1608 -> my_rcl:CPOLE2.5-6.5
- C35, C36: value 10u -> 100u; device my_rcl:C-2012 -> my_rcl:CPOLE2.5-6.5
- C37: value 10u -> 1u; device my_rcl:C-3216 -> my_rcl:C-1608
- C4: value DNP -> 1u
- C40: value 10u -> 1u; device my_rcl:C-2012 -> my_rcl:C-1608
- C42, C45, C46, C47, C54, C56, C65, C66, C67: value 0.1u -> 10u; device my_rcl:C-1608 -> my_rcl:C-2012
- C43: value 0.1u -> 330u; device my_rcl:C-1608 -> my_rcl:CPOLE2.5-6.5
- C44, C48, C49, C53, C60: value 10u -> 0.1u; device my_rcl:C-2012 -> my_rcl:C-1608
- C50: device my_rcl:C-2012 -> my_rcl:C-3216
- C55: value 10u -> 2.2u
- C6: value 0.1u -> DNP
- C63, C72: value 10u -> 0.1u
- C69: value 0.1u -> 10u
- C7, C9: value 1u -> DNP
- C73, C74: value 47p -> 0.1u
- C8: value 100u -> DNP; device my_rcl:CPOLE2.5-8 -> my_rcl:C-1608
- D1: value PWR -> TVS; device my_rcl:LED-SMD1608 -> my_rcl:ZENER-SMD2
- D2: value LED -> PWR
- D3: value TVS -> CLIP; device my_rcl:ZENER-SMD2 -> my_rcl:LED-SMD1608
- IC10: value REF5040 -> AD4134; device my_ic:REF5040 -> my_ic:AD4134
- IC11: value 1.8V -> REF5040; device my_ic:TLV740 -> my_ic:REF5040
- IC13: value 2.7V -> 1.8V
- IC14: value ISO6720FB -> 2.7V; device my_ic:SI8420 -> my_ic:TLV740
- IC16: value IOS6720FB -> ISO6720FB
- IC2: value OPA -> AP22652; device my_ic:OPA-2-SOP -> my_ic:AP22652
- IC3: value 7808 -> OPA; device my_ic:78LX -> my_ic:OPA-2-SOP
- IC4: value LM317-L -> 7808; device my_ic:LM317-L -> my_ic:78LX
- IC5: value LM337-L -> LM317-L; device my_ic:LM337-L -> my_ic:LM317-L
- IC7: value OPA1633 -> LM337-L; device my_ic:OPA-DIFF -> my_ic:LM337-L
- IC8: value AK1110 -> OPA1633; device my_ic:AK1110 -> my_ic:OPA-DIFF
- IC9: value AD4134 -> AK1110; device my_ic:AD4134 -> my_ic:AK1110
- R1: value 10 -> 10k; device my_rcl:R-2012 -> my_rcl:R-1608
- R10, R9: value 1k -> 270
- R11, R12, R16: value 1k -> 510
- R13: value 360 -> 510; device my_rcl:R-1608 -> my_rcl:R-2012
- R14: value 360 -> 100
- R15: value 1k -> 100; device my_rcl:R-2012 -> my_rcl:R-1608
- R2: value 10 -> 20
- R20, R21: value 120 -> 51
- R24, R25: value 22 -> 120
- R26, R28, R29, R30, R31: value 22 -> 10; device my_rcl:R-1608 -> my_rcl:R-1608-3
- R27: value 22 -> 10
- R3: value 100k -> 20; device my_rcl:R-1608 -> my_rcl:R-2012
- R32: value 10k -> 10
- R33: value 10k -> 10; device my_rcl:R-1608 -> my_rcl:R-1608-3
- R38, R39: value 47k -> 10k
- R40: value 39 -> 47k
- R41: value 5.1k -> 47k
- R42: value ODR -> 39
- R43, R52: value DOUT -> 3.3k
- R44: value DCLK -> 10k
- R45: value SDO -> ODR
- R46: value CS -> DOUT
- R47, R57: value SCLK -> DCLK
- R48, R58: value SDI -> SDO
- R49, R59: value LED -> CS
- R5: value 360 -> 100k
- R50: value 10M -> SCLK; device my_rcl:R-7.5 -> my_rcl:R-1608
- R51: value ODR -> SDI
- R53: value SUB -> 10M; device my_rcl:R-1608 -> my_rcl:R-7.5
- R54: value DCLK -> ODR
- R55: value SDO -> DOUT
- R56: value CS -> SUB
- R6: value 10 -> 100
- R60: value 10k -> SCLK
- R61: value 50 -> SDI
- R62: value 50 -> LED
- R7: value 10 -> 24
- R8: value 10k -> 24
- SW1: value DC -> AC
- SW2: value GAIN -> GAIN H<>M
Connections:
- removed net N$17 (its old number): IC14.OUT2, R52.1
- new net DIPSW1: IC1.IO0_14/K12, R63.1, SW3.A1
- new net DIPSW2: IC1.IO5P_14/K13, R64.1, SW3.A2
- new net DIPSW3: IC1.IO12P_14/N14, R65.1, SW3.A3
- new net DIPSW4: IC1.IO12N_14/P14, R66.1, SW3.A4
- new net N$32: IC16.OUT2, R58.1
- new net N$57: IC10.CLKSEL, J3.2
- new net N$63: IC2.ILIM, R1.2
- new net VIN_LIM: C4.1, FB2.1, IC2.OUT
- net +1V8: now also C53.1, C56.1, IC10.IOVDD, IC12.OUT, R38.2, R39.2; no longer C47.1, C50.1, IC11.OUT, IC9.IOVDD, R32.2, R33.2
- net +1V8_ISO: now also C69.1, C70.1, C71.1, C72.1, C73.1, IC16.VDD1, IC18.VDD2; no longer C63.1, C64.1, C65.1, C66.1, C67.1, IC14.VDD1, IC16.VDD2
- net +3.6V: now also C11.1, C12.1, C60.1, IC14.IN; no longer C54.1, C7.1, C8.1, IC13.IN
- net +3V3D: now also R63.2, R64.2, R65.2, R66.2
- net +3V3D_ISO: now also C74.1, C75.1, C76.1, C77.1, C78.1, IC16.VDD2, IC18.VDD1; no longer C68.1, C69.1, C70.1, C71.1, C72.1, IC14.VDD2, IC16.VDD1
- net +5V: now also C38.1, C41.1, C58.1, IC10.DVDD5, IC9.VOUT_LDO1, R40.1; no longer C32.1, C35.1, C52.1, IC8.VOUT_LDO1, IC9.DVDD5, R38.1
- net +5V_DEL: now also C54.1, IC14.EN, R40.2, R41.2; no longer C48.1, IC11.EN, R38.2, R39.2
- net +8V: now also C17.1, C37.1, IC4.OUT, IC9.EN, IC9.VIN_LDO1, IC9.VIN_LDO2; no longer C13.1, C31.1, IC3.OUT, IC8.EN, IC8.VIN_LDO1, IC8.VIN_LDO2
- net +9V: now also C15.1, C25.1, C34.1, IC3G$3.V+, IC5.OUT, IC8G$2.EN, IC8G$2.V+, R22.2, TP16.1; no longer C11.1, C21.1, C28.1, IC2G$3.V+, IC4.OUT, IC7G$2.EN, IC7G$2.V+, R20.2
- net -5V: now also C36.2, IC7.OUT, R24.2, TP18.1; no longer C30.2, IC6.OUT, R22.2
- net -9V: now also C35.2, IC6.OUT, R23.2, TP17.1; no longer C29.2, IC5.OUT, R21.2
- net ADC+: now also C32.1, R13.2, R20.2, R32.1; no longer C74.1, R15.2, R24.1, R61.2
- net ADC-: now also C33.2, R21.2, R33.1; no longer C73.2, R25.1, R62.2
- net ADC_2V7: now also C49.1, C51.1, C63.1, C67.1, IC10.LDION, IC13.IN, IC14.OUT, R43.2; no longer C43.1, C45.1, C55.1, C57.1, IC11.IN, IC13.OUT, IC9.LDION, R41.2
- net ADC_AVDD1V8: now also C62.1, C66.1, IC10.AVDD1V8; no longer C56.1, C60.1, IC9.AVDD1V8
- net ADC_CLKVDD: now also C52.1, C55.1, IC10.CLKVDD, J3.1; no longer C46.1, C49.1, IC9.CLKVDD
- net ADC_CS: now also IC10.FORMAT0/CS, R49.1; no longer IC9.FORMAT0/CS, R46.1
- net ADC_DCLK: now also IC10.DCLK, R47.1; no longer IC9.DCLK, R44.1
- net ADC_DOUT: now also IC10.DOUT0, R46.1; no longer IC9.DOUT0, R43.1
- net ADC_DVDD1V8: now also C57.1, C59.1, IC10.DVDD1V8; no longer C51.1, C53.1, IC9.DVDD1V8
- net ADC_ODR: now also IC10.ODR, R45.1; no longer IC9.ODR, R42.1
- net ADC_SCLK: now also IC10.FORMAT1/SCLK, R50.1; no longer IC9.FORMAT1/SCLK, R47.1
- net ADC_SDI: now also IC10.DEC2/SDI, R51.1; no longer IC9.DEC2/SDI, R48.1
- net ADC_SDO: now also IC10.DEC3/SDO, R44.2, R48.1; no longer IC9.DEC3/SDO, R45.1, R60.2
- net ADC_VCOM: now also C39.2, IC8G$1.CM, R25.1; no longer C33.2, IC7G$1.CM, R23.1
- net AVDD5V: now also C40.1, C47.1, C48.1, D1.C, IC10.AVDD5, IC11.VIN, IC9.VOUT_LDO2; no longer C34.1, C36.1, C41.1, D3.C, IC10.VIN, IC8.VOUT_LDO2, IC9.AVDD5
- net DGND: now also C1.2, C4.2, C74.2, C75.2, C76.2, C77.2, C78.2, IC16.GND2, IC18.GND1, IC2.!EN, IC2.GND, R1.1, R53.2, SW3.B1, SW3.B2, SW3.B3, SW3.B4; no longer C68.2, C69.2, C70.2, C71.2, C72.2, IC14.GND2, IC16.GND1, R50.2
- net FPGA_CS: now also R59.2; no longer R56.2
- net FPGA_DCLK: now also R57.2; no longer R54.2
- net FPGA_DCLK_SUB: now also R56.2; no longer R53.2
- net FPGA_DOUT: now also R55.2; no longer R52.2
- net FPGA_LED: now also R62.2; no longer R59.2
- net FPGA_ODR: now also R54.2; no longer R51.2
- net FPGA_SCLK: now also R60.2; no longer R57.2
- net FPGA_SDI: now also R61.2; no longer R58.2
- net FPGA_SDO: now also R58.2; no longer R55.2
- net GND: now also C10.2, C12.2, C14.1, C15.2, C16.1, C20.2, C22.2, C23.1, C24.1, C29.2, C31.1, C35.1, C36.1, C39.1, C5.1, C68.2, C69.2, C7.1, C70.2, C71.2, C72.2, C73.2, CON1.GND, CON2.GND, D1.A, D3.K, IC10.AGND1V8, IC10.AGND5, IC10.CLKGND, IC10.DGND1V8, IC10.DGND5, IC10.IOGND, IC10.REFGND, IC14.GND, IC16.GND1, IC18.GND2, IC4.GND, IC9.GND_LDO1, IC9.GND_LDO2, IC9.GND_REG, IC9.HT, J3.3, R4.2, R41.1, R44.1, R5.1, R53.1, TP14.1, TP15.1; no longer C10.1, C12.1, C14.2, C15.1, C16.2, C20.1, C22.1, C27.1, C28.2, C29.1, C3.1, C31.2, C35.2, C36.2, C39.2, C5.2, C7.2, C73.1, C74.2, C8.2, D1.K, D3.A, IC10.GND, IC14.GND1, IC16.GND2, IC3.GND, IC8.GND_LDO1, IC8.GND_LDO2, IC8.GND_REG, IC8.HT, IC9.AGND1V8, IC9.AGND5, IC9.CLKGND, IC9.CLKSEL, IC9.DGND1V8, IC9.DGND5, IC9.IOGND, IC9.REFGND, R3.2, R39.1, R4.1, R50.1, R60.1
- net N$1: now also C80.1, IC3G$2.-IN, R8.2; no longer IC2G$2.-IN, R7.2, R8.1
- net N$10: now also IC16.IN1, R47.2; no longer IC15.IN1, R44.2
- net N$11: now also IC10.AIN3-, R33.2; no longer IC9.AIN3-, R31.2
- net N$12: now also C80.2, IC3G$2.OUT; no longer IC2G$2.OUT
- net N$13: now also IC10.AIN3+, R32.2; no longer IC9.AIN3+, R30.2
- net N$14: now also C5.2, C7.2, C8.1, IC3G$1.+IN, R2.2, R4.1; no longer C3.2, C4.1, IC2G$1.+IN, R1.2, R3.1
- net N$15: now also IC10.AIN2-, R31.2; no longer IC9.AIN2-, R29.2
- net N$16: now also IC16.IN2, R48.2; no longer IC15.IN2, R45.2
- net N$18: now also IC10.AIN2+, R30.2; no longer IC9.AIN2+, R28.2
- net N$19: now also C21.1, R15.1; no longer C17.1, R14.1
- net N$2: now also IC10.VCM, R25.2; no longer IC9.VCM, R23.2
- net N$20: now also IC10.AIN1-, R29.2; no longer IC9.AIN1-, R27.2
- net N$21: now also IC15.OUT1, R54.1; no longer IC14.OUT1, R51.1
- net N$22: now also C27.2, IC8G$1.-OUT, R20.1; no longer C23.2, IC7G$1.-OUT, R61.1
- net N$23: now also C6.1, C8.2, C9.1, IC3G$2.+IN, R3.2, R5.2; no longer C4.2, C5.1, IC2G$2.+IN, R2.2, R4.2
- net N$24: now also C27.1, IC8G$1.+IN, R14.2; no longer C23.1, IC7G$1.+IN, R13.2
- net N$25: now also IC10.AIN1+, R28.2; no longer IC9.AIN1+, R26.2
- net N$26: now also C28.1, IC8G$1.-IN, R15.2; no longer C24.1, IC7G$1.-IN, R14.2
- net N$27: now also IC16.OUT1, R56.1, R57.1; no longer IC15.OUT1, R53.1, R54.1
- net N$28: now also IC10.AIN0-, R27.2; no longer IC9.AIN0-, R25.2
- net N$29: now also IC10.AIN0+, R26.2; no longer IC9.AIN0+, R24.2
- net N$3: now also C79.1, IC3G$1.-IN, R7.2; no longer IC2G$1.-IN, R6.2, R8.2
- net N$30: now also R42.2; no longer R40.2
- net N$31: now also C28.2, IC8G$1.+OUT, R21.1; no longer C24.2, IC7G$1.+OUT, R62.1
- net N$33: now also IC17.OUT2, R50.2; no longer IC16.OUT2, R47.2
- net N$34: now also IC17.OUT1, R49.2; no longer IC16.OUT1, R46.2
- net N$35: now also IC18.OUT2, R52.2; no longer IC17.OUT2, R49.2
- net N$36: now also IC18.OUT1, R51.2; no longer IC17.OUT1, R48.2
- net N$37: now also IC17.IN2, R60.1; no longer IC16.IN2, R57.1
- net N$38: now also IC17.IN1, R59.1; no longer IC16.IN1, R56.1
- net N$39: now also IC18.IN2, R62.1; no longer IC17.IN2, R59.1
- net N$4: now also C79.2, IC3G$1.OUT; no longer IC2G$1.OUT
- net N$40: now also IC18.IN1, R61.1; no longer IC17.IN1, R58.1
- net N$41: now also C2.1, CON1.SIG; no longer C1.1
- net N$42: now also C3.1, CON2.SIG; no longer C2.1
- net N$43: now also C2.2, R2.1; no longer C1.2, R1.1
- net N$44: now also C3.2, R3.1; no longer C2.2, R2.1
- net N$45: now also R7.1; no longer R6.1
- net N$46: now also R6.1, R8.1; no longer R5.1, R7.1
- net N$47: now also D3.A, R52.1; no longer D2.A, R49.1
- net N$48: now also C50.1, IC11.NR; no longer C44.1, IC10.NR
- net N$49: now also IC10.DEC1/DCLKMODE, R37.1; no longer IC9.DEC1/DCLKMODE, R35.1
- net N$5: now also C20.1, R14.1; no longer C16.1, R15.1
- net N$50: now also IC10.DEC0/DCLKIO, R36.1; no longer IC9.DEC0/DCLKIO, R34.1
- net N$52: now also C16.2, IC3G$3.V-; no longer C12.2, IC2G$3.V-
- net N$53: now also C29.1, IC5.ADJ, R22.1; no longer C25.1, IC4.ADJ, R20.1
- net N$54: now also C30.2, IC6.ADJ, R23.1; no longer C26.2, IC5.ADJ, R21.1
- net N$55: now also C31.2, IC7.ADJ, R24.1; no longer C27.2, IC6.ADJ, R22.1
- net N$58: now also D2.A, R43.1; no longer D1.A, R41.1
- net N$59: now also R6.2; no longer R5.2
- net N$6: now also C45.1, IC9.NP_LDO2; no longer C39.1, IC8.NP_LDO2
- net N$60: now also IC10.MODE, R39.1; no longer IC9.MODE, R37.1
- net N$61: now also IC10.!PDN, R34.1; no longer IC9.!PDN, R32.1
- net N$62: now also IC10.!RESET, R35.1; no longer IC9.!RESET, R33.1
- net N$64: now also IC10.PIN/SPI, R38.1; no longer IC9.PIN/SPI, R36.1
- net N$7: now also C46.1, IC9.NP_LDO1; no longer C40.1, IC8.NP_LDO1
- net N$74: now also C26.2, IC8G$2.V-; no longer C22.2, IC7G$2.V-
- net N$8: now also IC15.IN1, R45.2; no longer IC14.IN1, R42.2
- net N$9: now also IC15.IN2, R46.2; no longer IC14.IN2, R43.2
- net OSC_CLK: now also IC10.XTAL2/IN, R42.1; no longer IC9.XTAL2/IN, R40.1
- net V+: now also C10.1, C13.1, C22.1, IC5.IN; no longer C14.1, C6.1, C9.1, IC3.IN
- net V-: now also C14.2, C23.2, C24.2, IC7.IN; no longer C10.2, C15.2, C20.2, IC5.IN
- net VCC_OSC: now also C64.1, C65.1, IC13.OUT; no longer C58.1, C59.1, IC12.OUT
- net VIN: now also C1.1, IC2.IN; no longer FB2.1
- net VREF: now also C68.1, IC10.REFIN, IC11.VOUT; no longer C62.1, IC10.VOUT, IC9.REFIN
- net VREFCAP: now also C43.1, C44.1, IC10.REFCAP; no longer C37.1, C38.1, IC9.REFCAP
Other:
- moved on the sheet: C1, C10, C11, C16, C2, C20, C21, C22, C23, C24, C25, C26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

Commit message: 入力回路変更
Parts:
- removed C80: 100p, my_rcl:C-1608
- removed J3: CLKSEL, my_rcl:SJ-3-1608
- removed SW3: FSEL, my_rcl:DIPSW-4
- added JP1: GAIN, my_connector:PINHD-1X2
- added TP19, TP20, TP21: GND, my_connector:TESTPIN-MID
- added TP22: VCOM, my_connector:TESTPIN
- added TP23: ADC+, my_connector:TESTPIN
- added TP24: ADC-, my_connector:TESTPIN
- C1: value 1u -> 1.5u; device my_rcl:C-1608 -> my_rcl:C-5
- C10: value 0.1u -> 68p; device my_rcl:C-1608 -> my_rcl:C-1608-3
- C11: value 1u -> 100p
- C12: value 100u -> 100p; device my_rcl:CPOLE2.5-8 -> my_rcl:C-1608
- C13: value 1u -> 0.1u
- C15, C22: value 0.1u -> 100u; device my_rcl:C-1608 -> my_rcl:CPOLE2.5-8
- C16: value 0.1u -> 1u
- C17: value 100u -> 1u; device my_rcl:CPOLE2.5-6.5 -> my_rcl:C-1608
- C18: device my_rcl:CPOLE2.5-8 -> my_rcl:CPOLE2.5-6.5
- C19: value 100u -> 100p; device my_rcl:CPOLE2.5-8 -> my_rcl:C-1608-3
- C2: device my_rcl:C-5W -> my_rcl:C-5
- C20: value 1n -> 100p; device my_rcl:C-1608 -> my_rcl:C-1608-3
- C21: value 1n -> 100u; device my_rcl:C-1608 -> my_rcl:CPOLE2.5-8
- C23, C24: value 0.1u -> 100p
- C27, C28: value 270p -> 0.1u
- C29, C50: value 10u -> 0.1u; device my_rcl:C-3216 -> my_rcl:C-1608
- C3: value 1.5u -> 1u; device my_rcl:C-5W -> my_rcl:C-1608
- C32: value 68p -> 10u; device my_rcl:C-1608 -> my_rcl:C-3216
- C33: value 68p -> 0.1u
- C34: value 100u -> 0.1u; device my_rcl:CPOLE2.5-6.5 -> my_rcl:C-1608
- C37: value 1u -> 100u; device my_rcl:C-1608 -> my_rcl:CPOLE2.5-6.5
- C39, C41: value 10u -> 1u; device my_rcl:C-2012 -> my_rcl:C-1608
- C4: value 1u -> 22p
- C40, C68: value 1u -> 10u; device my_rcl:C-1608 -> my_rcl:C-2012
- C43: value 330u -> 10u; device my_rcl:CPOLE2.5-6.5 -> my_rcl:C-2012
- C44: value 0.1u -> 330u; device my_rcl:C-1608 -> my_rcl:CPOLE2.5-6.5
- C45, C54, C59, C61, C65: value 10u -> 0.1u; device my_rcl:C-2012 -> my_rcl:C-1608
- C48, C57, C60, C62: value 0.1u -> 10u; device my_rcl:C-1608 -> my_rcl:C-2012
- C5: value DNP -> 22p
- C51: value 0.1u -> 10u; device my_rcl:C-1608 -> my_rcl:C-3216
- C55: value 2.2u -> 10u
- C56: value 10u -> 2.2u
- C6: value DNP -> 1u
- C69: value 10u -> 1u
- C70: value 0.1u -> 10u
- C78: value 10u -> 0.1u
- C79: value 100p -> 10u
- C8: device my_rcl:C-1608 -> my_rcl:C-1608-3
- IC15, IC16: value ISO6720FB -> SI8620
- IC17, IC18: value IOS6720FB -> SI8620
- IC3: device my_ic:OPA-2-SOP -> my_ic:OPA-1
- IC4: value 7808 -> OPA; device my_ic:78LX -> my_ic:OPA-2-SOP
- IC5: value LM317-L -> 7808; device my_ic:LM317-L -> my_ic:78LX
- IC6: value LM337-L -> LM317-L; device my_ic:LM337-L -> my_ic:LM317-L
- IC8: value OPA1633 -> LM337-L; device my_ic:OPA-DIFF -> my_ic:LM337-L
- J1: value V- -> V-SEL; device my_rcl:SJ-3-2012 -> my_rcl:SJ-3-1608
- J2: value V- -> CLKSEL; device my_rcl:SJ-3-2012 -> my_rcl:SJ-3-1608
- R1: value 10k -> 100k; device my_rcl:R-1608 -> my_rcl:R-1608-3
- R10: value 270 -> 24; device my_rcl:R-2012 -> my_rcl:R-1608-3
- R11: value 510 -> 24; device my_rcl:R-2012 -> my_rcl:R-1608-3
- R12, R13, R3: device my_rcl:R-2012 -> my_rcl:R-2012H
- R14: value 100 -> 1k
- R15: value 100 -> 270; device my_rcl:R-1608 -> my_rcl:R-2012H
- R16: value 510 -> 270; device my_rcl:R-2012 -> my_rcl:R-2012H
- R17, R18: value 680 -> 3.6k
- R19: value 330 -> 680
- R2: value 20 -> 100k; device my_rcl:R-2012 -> my_rcl:R-1608-3
- R20: value 51 -> 680
- R21: value 51 -> 330
- R4: value 100k -> 20; device my_rcl:R-1608 -> my_rcl:R-2012H
- R5: value 100k -> 50; device my_rcl:R-1608 -> my_rcl:R-1608-3
- R6: value 100 -> 50; device my_rcl:R-1608 -> my_rcl:R-1608-3
- R7: value 24 -> 10k
- R8: value 24 -> 1k; device my_rcl:R-1608 -> my_rcl:R-1608-3
- R9: value 270 -> 1k; device my_rcl:R-2012 -> my_rcl:R-1608-3
- SW2: value GAIN H<>M -> MODE-SW; device my_connector:SW-1X3 -> my_rcl:DIPSW-4
Connections:
- removed net N$26: C28.1, IC8G$1.-IN, R15.2
- removed net N$59: R6.2, SW2.3
- removed net N$74: C26.2, IC8G$2.V-, J2.2
- net +1V8: now also C54.1, C57.1; no longer C53.1, C56.1
- net +1V8_ISO: now also C74.1; no longer C69.1
- net +3.6V: now also C14.1, C15.1, C61.1; no longer C11.1, C12.1, C60.1
- net +3V3D_ISO: now also C79.1; no longer C74.1
- net +5V: now also C39.1, C42.1, C59.1, IC9.VOUT1; no longer C38.1, C41.1, C58.1, IC9.VOUT_LDO1
- net +5V_DEL: now also C55.1; no longer C54.1
- net +8V: now also C18.1, C38.1, IC5.OUT, IC9.VIN1, IC9.VIN2; no longer C17.1, C37.1, IC4.OUT, IC9.VIN_LDO1, IC9.VIN_LDO2
- net +9V: now also C28.1, C33.1, C35.1, IC3G$2.V+, IC4G$3.V+, IC6.OUT; no longer C15.1, C25.1, C34.1, IC3G$3.V+, IC5.OUT, IC8G$2.EN, IC8G$2.V+
- net -5V: now also C29.2, C37.2, IC4G$3.V-, IC8.OUT, J1.3; no longer C36.2, IC7.OUT, J1.1, J2.1
- net -9V: now also C36.2, IC7.OUT, J1.1; no longer C35.2, IC6.OUT, J1.3, J2.3
- net ADC+: now also C19.1, C23.1, R12.2, R15.2, R17.1, TP23.1; no longer C32.1, R13.2, R20.2
- net ADC-: now also C20.1, C24.1, R13.2, R18.1, TP24.1; no longer C33.2, R21.2
- net ADC_2V7: now also C50.1, C52.1, C62.1, C64.1, C68.1; no longer C49.1, C51.1, C61.1, C63.1, C67.1
- net ADC_AVDD1V8: now also C63.1, C67.1; no longer C62.1, C66.1
- net ADC_CLKVDD: now also C53.1, C56.1, J2.1; no longer C52.1, C55.1, J3.1
- net ADC_DVDD1V8: now also C58.1, C60.1; no longer C57.1, C59.1
- net ADC_VCOM: now also C40.2, R1.2, R14.1, R2.1, TP22.1; no longer C39.2, IC8G$1.CM
- net AVDD5V: now also C41.1, C43.1, C49.1, IC9.VOUT2; no longer C40.1, C42.1, C47.1, IC9.VOUT_LDO2
- net DGND: now also C3.2, C6.2, C79.2, R7.1, SW2.B1, SW2.B2, SW2.B3, SW2.B4; no longer C1.2, C4.2, C74.2, R1.1, SW3.B1, SW3.B2, SW3.B3, SW3.B4
- net DIPSW1: now also SW2.A1; no longer SW3.A1
- net DIPSW2: now also SW2.A2; no longer SW3.A2
- net DIPSW3: now also SW2.A3; no longer SW3.A3
- net DIPSW4: now also SW2.A4; no longer SW3.A4
- net GND: now also C14.2, C16.2, C17.1, C19.2, C22.1, C23.2, C24.2, C27.1, C28.2, C29.1, C30.2, C32.1, C33.2, C34.1, C35.2, C37.1, C39.2, C4.1, C40.1, C5.2, C74.2, IC5.GND, IC9.GND1, IC9.GND2, J2.3, R19.1, R20.2, R21.2, TP19.1, TP20.1, TP21.1; no longer C10.2, C11.2, C12.2, C14.1, C16.1, C17.2, C19.1, C22.2, C23.1, C24.1, C29.2, C30.1, C32.2, C33.1, C34.2, C35.1, C37.2, C39.1, C40.2, C5.1, C6.2, IC4.GND, IC9.GND_LDO1, IC9.GND_LDO2, J3.3, R17.1, R18.2, R19.2, R4.2, R5.1
- net N$1: now also C12.1, IC4G$2.-IN, R11.2, R13.1; no longer C80.1, IC3G$2.-IN, R10.1, R8.2
- net N$12: now also C5.1, R6.1; no longer C80.2, IC3G$2.OUT, R10.2, R12.1
- net N$14: now also IC4G$1.+IN, R3.2, R5.1; no longer C5.2, IC3G$1.+IN, R2.2, R4.1
- net N$19: now also IC3G$1.+IN, R17.2, R18.2; no longer C21.1, R12.2, R15.1, R16.1
- net N$22: now also C10.2, IC3G$1.-IN, R14.2; no longer C27.2, IC8G$1.-OUT, R20.1
- net N$23: now also IC4G$2.+IN, R4.2, R6.2; no longer C6.1, IC3G$2.+IN, R3.2, R5.2
- net N$24: now also C34.2, IC3G$2.V-, J1.2; no longer C27.1, IC8G$1.+IN, R14.2
- net N$3: now also C11.1, IC4G$1.-IN, R10.2, R12.1; no longer C79.1, IC3G$1.-IN, R7.2, R9.1
- net N$31: now also C11.2, IC4G$1.OUT, R15.1; no longer C28.2, IC8G$1.+OUT, R21.1
- net N$4: now also C4.2, R5.2; no longer C79.2, IC3G$1.OUT, R11.1, R9.2
- net N$41: now also C1.1; no longer C2.1
- net N$42: now also C2.1; no longer C3.1
- net N$43: now also C1.2, R1.1, R3.1; no longer C2.2, R2.1
- net N$44: now also C2.2, R2.2, R4.1; no longer C3.2, R3.1
- net N$45: now also JP1.1, R10.1, R8.1; no longer R7.1, SW2.2
- net N$46: now also JP1.2, R11.1, R9.1; no longer R6.1, R8.1, SW2.1
- net N$48: now also C51.1; no longer C50.1
- net N$5: now also C10.1, IC3G$1.OUT, R8.2, R9.2; no longer C20.1, R11.2, R13.1, R14.1
- net N$52: now also C12.2, IC4G$2.OUT, R16.1; no longer C16.2, IC3G$3.V-, J1.2
- net N$53: now also C30.1, IC6.ADJ, R19.2; no longer C29.1, IC5.ADJ, R17.2
- net N$54: now also C31.2, IC7.ADJ, R20.1; no longer C30.2, IC6.ADJ, R18.1
- net N$55: now also C32.2, IC8.ADJ, R21.1; no longer C31.2, IC7.ADJ, R19.1
- net N$57: now also J2.2; no longer J3.2
- net N$6: now also C46.1, IC9.NP2; no longer C45.1, IC9.NP_LDO2
- net N$63: now also R7.2; no longer R1.2
- net N$7: now also C47.1, IC9.NP1; no longer C46.1, IC9.NP_LDO1
- net V+: now also C16.1, C21.1, C25.1, IC6.IN; no longer C10.1, C18.1, C22.1, IC4.IN
- net V-: now also C17.2, C22.2, C26.2, C27.2, IC8.IN; no longer C14.2, C19.2, C23.2, C24.2, IC6.IN
- net VCC_OSC: now also C66.1; no longer C64.1
- net VIN: now also C3.1; no longer C1.1
- net VIN_LIM: now also C6.1; no longer C4.1
- net VREF: now also C69.1; no longer C68.1
- net VREFCAP: now also C45.1; no longer C43.1
Other:
- note added: "96Mbps min."
- moved on the sheet: C1, C10, C11, C13, C14, C16, C18, C2, C20, C23, C24, C25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

Commit message: 6層
Parts:
- R45, R46: device my_rcl:R-1608 -> my_rcl:R-1608-3
Changed lines of the file:
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@@
 <part name="IC15" library="my_ic" deviceset="SI8420" device="" value="SI8620"/>
 <part name="IC16" library="my_ic" deviceset="SI8420" device="" value="SI8620"/>
-<part name="R45" library="my_rcl" deviceset="R" device="-1608" value="ODR"/>
-<part name="R46" library="my_rcl" deviceset="R" device="-1608" value="DOUT"/>
+<part name="R45" library="my_rcl" deviceset="R" device="-1608-3" value="ODR"/>
+<part name="R46" library="my_rcl" deviceset="R" device="-1608-3" value="DOUT"/>
 <part name="R47" library="my_rcl" deviceset="R" device="-1608" value="DCLK"/>
 <part name="R48" library="my_rcl" deviceset="R" device="-1608" value="SDO"/>
