File: ADC2.sch (EAGLE design)
At the start: 161 parts, among them CON1 USB-A, CON2 SWD_CON, IC1 STM32G431KB, IC10 NJM11100, IC11 3.3V, IC12 LME49721, IC13 NJM4580, IC14 NJM12888F18, IC15 NJM2845-3.3, IC16 -5V, IC17 +5V, IC2 7404, IC3 ESP32-WROVER, IC4 LME49721, IC5 NJM4580, IC6 MCP331X1, IC7 OCT_BUFFER-SO6, IC8 OCT_BUFFER-SO6, IC9 3.3V, J1 SJ-1608, J10 SJ-1608, J2 SJ-1608, J3 SJ-1608, J4 SJ-1608, J5 IN3_DC, J6 IN1_DC, J7 SJ-1608, J8 SJ-1608, J9 SJ-1608, X1 12MHz

Commit message: ver2
Parts:
- removed J10: SJ-1608, my_rcl:SJ-1608
- added C56, C58: 10u, my_rcl:C-2012
- added C57, C59: 0.1u, my_rcl:C-1608
- added D1: PWR, my_rcl:LED-SMD1608
- added D2: OK, my_rcl:LED-SMD1608
- added D3: ERR, my_rcl:LED-SMD1608
- added D4, D5: CLAMP, my_rcl:DIODE-1N4148W
- added F1: 0.5A, my_rcl:FUSE-3216
- added FB5, FB6: FB-2012, my_rcl:FB-2012
- added IC18: LM4562, my_ic:OPA-2-DUAL
- added IC19: TC7WH74FU, my_ic:TC7WH74FU
- added IC20: NJM2845-33, my_ic:78X-SOP
- added IC21: -5V, my_ic:79LX
- added R49, R50: 1k, my_rcl:R-1608
- added R51: 10k, my_rcl:R-1608
- added R52: DNP, my_rcl:R-2012
- added SW1: Gain, my_connector:SW-1X3
- added TP21, TP30: VIN+, my_connector:TESTPIN
- added TP22, TP31: VIN-, my_connector:TESTPIN
- added TP23: (no value), my_connector:TESTPIN
- added TP24: VDD_OSC, my_connector:TESTPIN
- added TP25: OSC_EN, my_connector:TESTPIN
- added TP26: OSC_OUT, my_connector:TESTPIN
- added TP27, TP28, TP29: GND, my_connector:TESTPIN
- C10: value 1n -> 0.1u
- C13: value 1u -> 10u
- C14: value 27p -> 470p
- C15: value 10u -> DNP; device my_rcl:C-3225 -> my_rcl:C-1608
- C17: value 470p -> 10u; device my_rcl:C-1608 -> my_rcl:C-2012
- C19: value 470p -> 100p
- C20: device my_rcl:C-3225 -> my_rcl:C-5
- C22: value 27p -> 100p
- C23, C24: value 1n -> 470p
- C28: value 0.1u -> 1u
- C29: value 0.1u -> 100u; device my_rcl:C-1608 -> my_rcl:CPOLE2.5-6.5
- C35, C45, C46, C47: device my_rcl:C-2012 -> my_rcl:C-3216
- C4, C5: value 27p -> 22p
- C51: value 0.1u -> DNP; device my_rcl:C-1608 -> my_rcl:C-2012
- C7: value 10u -> 0.1u; device my_rcl:C-2012 -> my_rcl:C-1608
- C9: value 1n -> DNP
- FB1: value FB -> FB-2012; device my_rcl:FB -> my_rcl:FB-2012
- IC1: value STM32G431KB -> STM32G431
- IC11, IC9: value 3.3V -> TAR5SB33; device my_ic:NJM2863 -> my_ic:TAR5SB33
- IC12: value LME49721 -> LM4562; device my_ic:OPA-2-SOP -> my_ic:OPA-2-DUAL
- IC13: value NJM4580 -> LM4562; device my_ic:OPA-2-SOP -> my_ic:OPA-2-DUAL
- IC15: value NJM2845-3.3 -> AZ1117-3.3; device my_ic:78X-SOP -> my_ic:LM1117GS
- IC16: value -5V -> -9V
- IC17: value +5V -> +9V
- IC4: device my_ic:OPA-2-SOP -> my_ic:OPA-2-DUAL
- IC5: value NJM4580 -> TL431; device my_ic:OPA-2-SOP -> my_ic:TL431
- IC6: value MCP331X1 -> AD4001
- J1, J3, J9: value SJ-1608 -> SJ-2012; device my_rcl:SJ-1608 -> my_rcl:SJ-2012
- J5: value IN3_DC -> SJ-2012
- J8: value SJ-1608 -> short; device my_rcl:SJ-1608 -> my_rcl:SJ-2012
- R1: value 37 -> 10k; device my_rcl:R-1608J -> my_rcl:R-1608
- R10, R11: value 10 -> 37; device my_rcl:R-1608 -> my_rcl:R-1608J
- R15: value 1k -> 10k
- R17, R18, R19: value 1k -> 1.5k
- R20: value 1k -> 10; device my_rcl:R-1608 -> my_rcl:R-1608J
- R21: value 10k -> short; device my_rcl:R-1608 -> my_rcl:R-1608J
- R40: value 0 -> 10k; device my_rcl:R-1608J -> my_rcl:R-1608
- R41: value 10k -> 100k
- R46: value 6.8k -> 10k
- R47: value 2.4k -> 1.5k
- TP1: value AIN3 -> +D5V; device my_connector:TESTPIN-BIG -> my_connector:TESTPIN
- TP15: value GND -> -D5V; device my_connector:TESTPIN-BIG -> my_connector:TESTPIN
- TP17, TP18, TP19: device my_connector:TESTPIN-BIG -> my_connector:TESTPIN
- TP3: value AOUT1 -> GND; device my_connector:TESTPIN-BIG -> my_connector:TESTPIN
Connections:
- removed net +5V: C41.1, C42.1, C46.1, C48.1, C50.1, IC12G$3.V+, IC13G$3.V+, IC17.OUT, IC4G$3.V+, IC5G$3.V+
- removed net ADC3+: J1.2, R10.1
- removed net ADC3-: J3.2, R11.1
- removed net DAC1: C17.1, IC5G$2.+IN, R40.1
- removed net VDDA: C3.1, C7.1, FB1.1, IC1.VDDA
- new net +5.3V: C34.1, C57.1, IC10.VOUT, IC4G$3.V+, R46.2, R49.1, R51.2
- new net +5VD: C45.1, FB4.1, FB6.2, IC9.CONTROL, IC9.VIN
- new net +9V: C41.1, C46.1, C48.1, C7.1, D4.K, IC12G$3.V+, IC13G$3.V+, IC17.OUT, IC18G$3.V+
- new net -9V: C42.2, C47.2, C49.2, D5.A, IC12G$3.V-, IC13G$3.V-, IC16.OUT, J5.1
- new net ADC_CNVST_CLOCKED: IC19G$1.Q, R13.2
- new net ADC_CNVST_FB: IC2G$4.OUT, R11.1
- new net ADC_SDI: IC2G$1.IN, R4.1
- new net CLK_8MHZ: R3.2, TP26.1
- new net N$69: C43.1, FB4.2, IC15.IN, IC20.IN
- new net N$70: FB1.1, TP17.1
- new net N$71: FB5.1, TP19.1
- new net N$72: FB6.1, TP1.1
- new net N$73: C51.2, R52.2
- new net N$74: C50.2, IC18G$3.V-, J5.2, J9.2
- new net N$75: TP21.1, TP30.1
- new net N$76: TP22.1, TP31.1
- net +3V3: now also C3.1, D1.A, IC1.VDDA; no longer FB1.2, R18.2
- net +3V3A: now also C10.1, IC19G$1.!CLR, IC19G$1.!PR, IC19G$2.V+
- net +3V3D: now also IC20.OUT, R1.2
- net -5V: now also C58.2, IC21.OUT, J9.1; no longer C47.2, C49.2, C51.2, IC13G$3.V-, IC16.OUT, IC5G$3.V-
- net ADC_CNVST: now also IC19G$1.D; no longer IC2G$3.IN
- net ADC_SCK: now also IC2G$2.IN; no longer IC2G$1.IN
- net ADC_SDO: now also IC2G$3.OUT; no longer IC2G$2.OUT
- net ESP_BOOT: now also R1.1
- net GND: now also C14.2, C41.2, C42.1, C50.1, C56.2, C57.2, C58.1, C59.1, IC13G$1.+IN, IC19G$2.V-, IC20.GND, IC21.GND, IC2G$6.IN, IC4G$3.V-, IC5.GND, R16.1, R17.1, R18.1, R19.1, R50.1, R52.1, TP27.1, TP28.1, TP29.1, TP3.1; no longer C50.2, C51.1, C9.1, IC13G$1.-IN, IC2G$4.IN, J10.1, J8.1, R21.1, R22.1, TP15.1
- net N$10: now also IC1.PA7, R4.2; no longer C15.1, J5.1, TP1.1
- net N$11: now also IC19G$1.!Q, R10.1; no longer IC3.GPIO18, R2.1
- net N$12: now also C20.2, J6.2, R20.1; no longer IC3.GPIO19, R1.1
- net N$13: now also IC2G$1.OUT, R2.2; no longer IC3.GPIO23, R4.1
- net N$14: now also C9.1, IC12G$2.OUT, IC18G$2.+IN, J1.2, R12.2; no longer C28.1, IC4G$1.+IN, R19.1, R20.1
- net N$15: now also C56.1; no longer J9.2
- net N$18: now also IC19G$1.CK, R3.1; no longer IC4G$1.-IN, R15.1, R16.2
- net N$19: now also IC2G$4.IN, R10.2; no longer IC2G$3.OUT, R13.2
- net N$2: now also IC18G$2.-IN, IC18G$2.OUT, J1.1, J2.1; no longer C9.2, IC1.PA0, R10.2
- net N$20: now also IC2G$3.IN; no longer IC2G$2.IN
- net N$21: now also IC1.PA4, R11.2; no longer C14.2, IC4G$2.-IN, R14.1, R17.2
- net N$22: now also IC2G$5.IN, IC2G$6.OUT; no longer C15.2, IC5G$1.+IN, J5.2, R21.2
- net N$23: now also C15.1, IC4G$2.OUT, R21.1; no longer IC5G$1.-IN, IC5G$1.OUT, R17.1
- net N$24: now also J8.2, R35.1; no longer IC5G$2.-IN, IC5G$2.OUT, TP3.1
- net N$26: now also C19.2, IC12G$1.-IN, R14.2; no longer IC4G$1.OUT, J1.1, R15.2
- net N$27: now also D1.K, R17.2; no longer C14.1, IC4G$2.OUT, J3.1, R14.2, R16.1
- net N$30: now also R2.1; no longer J9.1
- net N$31: now also IC2G$2.OUT; no longer IC2G$1.OUT
- net N$39: now also IC13G$2.-IN, R15.1, R16.2, SW1.3; no longer C29.1, IC4G$2.+IN, R20.2, R22.2
- net N$40: now also D2.K, R18.2; no longer R18.1, R19.2
- net N$42: now also C9.2
- net N$43: now also C14.1, R14.1; no longer C19.2, IC12G$1.-IN
- net N$45: now also R15.2, SW1.1, SW1.2; no longer IC13G$2.-IN
- net N$46: now also D3.K, R19.2; no longer IC12G$2.OUT, J2.1, R12.2
- net N$47: now also IC18G$1.+IN, J3.2; no longer J4.1
- net N$49: now also D4.A, D5.K, R20.2; no longer C20.2, J6.2
- net N$5: now also IC18G$1.-IN, IC18G$1.OUT, J3.1, J4.1; no longer C10.1, IC1.PA1, R11.2
- net N$50: now also D3.A, IC1.PA3; no longer IC1.PA7, R29.2
- net N$54: now also D2.A, IC1.PA2; no longer IC1.PA4, R40.2
- net N$55: now also IC13G$1.-IN; no longer IC13G$1.+IN
- net N$57: now also J8.1; no longer R35.1
- net N$58: now also C15.2, IC4G$2.-IN, R22.1, R50.2; no longer IC2G$5.OUT, IC2G$6.IN
- net N$60: now also IC5.OUT, IC5.REF, R40.1, R49.2; no longer IC2G$4.OUT, IC2G$5.IN
- net N$62: now also R51.1
- net N$63: now also C28.1, C29.1, IC4G$1.+IN, IC4G$2.+IN, R40.2; no longer C42.2, IC12G$3.V-, J8.2
- net N$64: now also IC4G$1.-IN, IC4G$1.OUT; no longer C41.2, IC4G$3.V-, J10.2
- net N$65: now also F1.P$2, TP4.1; no longer C43.1, FB4.2, IC15.IN
- net N$9: now also IC1.PB0, R29.2; no longer IC3.GPIO5, R3.1
- net SPI_CS: now also IC3.GPIO5; no longer R3.2
- net SPI_MISO: now also IC3.GPIO19; no longer R1.2
- net SPI_MOSI: now also IC3.GPIO23; no longer R4.2
- net SPI_SCK: now also IC3.GPIO18; no longer R2.2
- net V+: now also FB1.2, TP24.1, TP25.1; no longer C45.1, FB4.1, IC9.CONTROL, IC9.VIN, TP17.1
- net V-: now also C59.2, FB5.2, IC21.IN; no longer TP19.1
- net VBUS: now also F1.P$1; no longer TP4.1
- net VREF: now also C17.1, C51.1, R21.2, R22.2; no longer C34.1, IC10.VOUT, R46.2
Other:
- moved on the sheet: C10, C14, C15, C16, C17, C18, C19, C20, C21, C22, C25, C26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

Commit message: ver2修正
Parts:
- removed C46, C47: 10u, my_rcl:C-3216
- removed C48, C49, C50, C52, C53, C57, C59: 0.1u, my_rcl:C-1608
- removed C51: DNP, my_rcl:C-2012
- removed C54, C55: 100u, my_rcl:CPOLE2.5-8
- removed C56, C58: 10u, my_rcl:C-2012
- removed CON1: USB-A, my_connector:USB-A
- removed CON2: SWD_CON, my_connector:SWD_CON
- removed D3: ERR, my_rcl:LED-SMD1608
- removed D4, D5: CLAMP, my_rcl:DIODE-1N4148W
- removed F1: 0.5A, my_rcl:FUSE-3216
- removed IC10: NJM11100, my_ic:NJM11100
- removed IC12, IC18: LM4562, my_ic:OPA-2-DUAL
- removed IC16: -9V, my_ic:79LX
- removed IC17: +9V, my_ic:78LX
- removed IC19: TC7WH74FU, my_ic:TC7WH74FU
- removed IC20: NJM2845-33, my_ic:78X-SOP
- removed IC21: -5V, my_ic:79LX
- removed R22, R23, R35, R36, R39, R42, R43, R48, R49, R50: 1k, my_rcl:R-1608
- removed R24, R27, R28, R29: 37, my_rcl:R-1608J
- removed R30, R44, R45: 22, my_rcl:R-1608
- removed R40, R46, R51: 10k, my_rcl:R-1608
- removed R41: 100k, my_rcl:R-1608
- removed R47: 1.5k, my_rcl:R-1608
- removed R52: DNP, my_rcl:R-2012
- removed TP10: ESP_EN, my_connector:TESTPIN
- removed TP11: ESP_BOOT, my_connector:TESTPIN
- removed TP12: ESP_TX, my_connector:TESTPIN
- removed TP13, TP20, TP27, TP28, TP29: GND, my_connector:TESTPIN
- removed TP14: ESP_RX, my_connector:TESTPIN
- removed TP24: VDD_OSC, my_connector:TESTPIN
- removed TP25: OSC_EN, my_connector:TESTPIN
- removed TP26: OSC_OUT, my_connector:TESTPIN
- removed TP6: UART_RX, my_connector:TESTPIN
- removed TP7: UART_GND, my_connector:TESTPIN
- removed TP8: UART_TX, my_connector:TESTPIN
- removed TP9: +3V3D, my_connector:TESTPIN
- removed X1: 12MHz, my_rcl:CRYSTALHC49S
- added U$9: FPGA_CORE_BOARD, my_ic:FPGA_CORE_BOARD
- C12: value 3300p -> 470p
- C13: value 10u -> 0.1u; device my_rcl:C-2012 -> my_rcl:C-1608
- C14, C24: value 470p -> 100p
- C15: value DNP -> 10u; device my_rcl:C-1608 -> my_rcl:C-2012
- C16: value 0.1u -> 10u; device my_rcl:C-1608 -> my_rcl:C-3216
- C17: device my_rcl:C-2012 -> my_rcl:C-3216
- C18, C33: value 10u -> 470p; device my_rcl:C-2012 -> my_rcl:C-1608
- C19, C22: value 100p -> 0.1u
- C20: value 10u -> 1u; device my_rcl:C-5 -> my_rcl:C-1608
- C21, C30, C41: value 0.1u -> 10u; device my_rcl:C-1608 -> my_rcl:C-2012
- C23: value 470p -> DNP
- C25: value 470p -> 10u; device my_rcl:C-1608 -> my_rcl:C-3216
- C28: value 1u -> 10u; device my_rcl:C-1608 -> my_rcl:C-2012
- C29: value 100u -> 0.1u; device my_rcl:CPOLE2.5-6.5 -> my_rcl:C-1608
- C3: value 0.01u -> 0.1u
- C32: value 0.1u -> 470p
- C35: value 10u -> 3300p; device my_rcl:C-3216 -> my_rcl:C-1608
- C38, C42: value 0.1u -> 1u
- C4: value 22p -> 0.1u
- C44: value 0.1u -> DNP
- C45: value 10u -> 1u; device my_rcl:C-3216 -> my_rcl:C-1608
- C5: value 22p -> 10u; device my_rcl:C-1608 -> my_rcl:C-5
- C8: value 0.1u -> 100u; device my_rcl:C-1608 -> my_rcl:CPOLE2.5-8
- C9: value DNP -> 100u; device my_rcl:C-1608 -> my_rcl:CPOLE2.5-8
- D1: value PWR -> CLAMP; device my_rcl:LED-SMD1608 -> my_rcl:DIODE-1N4148W
- D2: value OK -> CLAMP; device my_rcl:LED-SMD1608 -> my_rcl:DIODE-1N4148W
- FB2, FB3, FB4: value FB -> FB-2012; device my_rcl:FB -> my_rcl:FB-2012
- FB5, FB6: value FB-2012 -> FB; device my_rcl:FB-2012 -> my_rcl:FB
- IC1: value STM32G431 -> +9V; device my_ic:STM32G431KB -> my_ic:78LX
- IC11: value TAR5SB33 -> AD4001; device my_ic:TAR5SB33 -> my_ic:MCP331X1
- IC13: value LM4562 -> 7404; device my_ic:OPA-2-DUAL -> my_ic:7404
- IC14: value NJM12888F18 -> TC7WH74FU; device my_ic:NJM12888 -> my_ic:TC7WH74FU
- IC15: value AZ1117-3.3 -> OSC; device my_ic:LM1117GS -> my_ic:OSC
- IC2: value 7404 -> -9V; device my_ic:7404 -> my_ic:79LX
- IC3: value ESP32-WROVER -> -5V; device my_ic:ESP32-WROVER -> my_ic:79LX
- IC4: value LME49721 -> LM4562
- IC5: value TL431 -> AK1110; device my_ic:TL431 -> my_ic:AK1110
- IC6: value AD4001 -> LM4562; device my_ic:MCP331X1 -> my_ic:OPA-2-DUAL
- IC7: value OCT_BUFFER-SO6 -> LM4562; device my_ic:OCT_BUFFER-SO6 -> my_ic:OPA-2-DUAL
- IC8: value OCT_BUFFER-SO6 -> TAR5SB33; device my_ic:OCT_BUFFER-SO6 -> my_ic:TAR5SB33
- IC9: value TAR5SB33 -> NJM12888F18; device my_ic:TAR5SB33 -> my_ic:NJM12888
- J1: value SJ-2012 -> IN1_DC
- J2: value SJ-1608 -> SJ-2012; device my_rcl:SJ-1608 -> my_rcl:SJ-2012
- J4: value SJ-1608 -> short; device my_rcl:SJ-1608 -> my_rcl:SJ-2012
- J6: value IN1_DC -> SJ-2012
- J8: value short -> SJ-1608; device my_rcl:SJ-2012 -> my_rcl:SJ-1608
- J9: value SJ-2012 -> SJ-1608; device my_rcl:SJ-2012 -> my_rcl:SJ-1608
- R1: value 10k -> 10; device my_rcl:R-1608 -> my_rcl:R-1608J
- R10, R11, R13, R8: value 37 -> 1k; device my_rcl:R-1608J -> my_rcl:R-1608
- R15: value 10k -> 1k
- R17, R18, R19: value 1.5k -> 1k
- R2: value 37 -> 100k; device my_rcl:R-1608J -> my_rcl:R-1608
- R20: value 10 -> 1k; device my_rcl:R-1608J -> my_rcl:R-1608
- R21: value short -> 1k; device my_rcl:R-1608J -> my_rcl:R-1608
- R25: value 37 -> 22; device my_rcl:R-1608J -> my_rcl:R-1608
- R26: value 1k -> 22
- R3, R4, R5, R6, R7: value 37 -> 22
- R31: value 22 -> 37; device my_rcl:R-1608 -> my_rcl:R-1608J
- R32, R33, R34, R37, R38: value 1k -> 37; device my_rcl:R-1608 -> my_rcl:R-1608J
- TP4: value VBUS -> GND
- TP5: value UART_3V3 -> GND
Connections:
- removed net +3V3: C1.2, C18.1, C2.1, C3.1, C38.1, D1.A, IC1.VDDA, IC1.VDD_1, IC1.VDD_2, IC7.V+, IC8.A, IC9.VOUT
- removed net +3V3D: C35.1, IC15.OUT, IC20.OUT, IC3.3V3, R1.2, R9.2, TP9.1
- removed net +5.3V: C34.1, C57.1, IC10.VOUT, IC4G$3.V+, R46.2, R49.1, R51.2
- removed net +5VD: C45.1, FB4.1, FB6.2, IC9.CONTROL, IC9.VIN
- removed net ADC1+: J4.2, R44.1
- removed net ADC1-: J2.2, J7.2, R45.1
- removed net ESP_BOOT: IC3.GPIO0, R1.1, TP11.1
- removed net ESP_EN: C8.1, IC3.EN, R9.1, TP10.1
- removed net ESP_RX: IC3.U0RXD, TP14.1
- removed net ESP_TX: IC3.U0TXD, TP12.1
- removed net N$23: C15.1, IC4G$2.OUT, R21.1
- removed net N$27: D1.K, R17.2
- removed net N$32: CON1.D-, R30.1
- removed net N$33: CON1.D+, R31.1
- removed net N$34: IC8.C, R33.2
- removed net N$35: IC7.C, R38.2, R48.2
- removed net N$36: IC1.PA5, R27.2
- removed net N$37: IC1.PA6, R28.2
- removed net N$39: IC13G$2.-IN, R15.1, R16.2, SW1.3
- removed net N$40: D2.K, R18.2
- removed net N$46: D3.K, R19.2
- removed net N$50: D3.A, IC1.PA3
- removed net N$51: C16.1, IC9.BYPASS
- removed net N$52: C24.2, IC6.AIN+, R44.2
- removed net N$53: C23.1, IC6.AIN-, R45.2
- removed net N$54: D2.A, IC1.PA2
- removed net N$58: C15.2, IC4G$2.-IN, R22.1, R50.2
- removed net N$60: IC5.OUT, IC5.REF, R40.1, R49.2
- removed net N$61: C36.1, IC10.BYPASS
- removed net N$62: IC10.VADJ, R46.1, R47.2, R51.1
- removed net N$63: C28.1, C29.1, IC4G$1.+IN, IC4G$2.+IN, R40.2
- removed net N$64: IC4G$1.-IN, IC4G$1.OUT
- removed net N$65: F1.P$2, TP4.1
- removed net N$66: C44.1, IC1.NRST
- removed net N$69: C43.1, FB4.2, IC15.IN, IC20.IN
- removed net N$72: FB6.1, TP1.1
- removed net N$73: C51.2, R52.2
- removed net SPI_CS: IC3.GPIO5, R8.2
- removed net SPI_MISO: IC3.GPIO19, R6.2
- removed net SPI_MOSI: IC3.GPIO23, R5.2
- removed net SPI_SCK: IC3.GPIO18, R7.2
- removed net STM_RX: IC1.PA10, IC7.OUT
- removed net STM_TX: CON2.TX, IC1.PA9, R33.1
- removed net SWCLK: CON2.SWCLK, IC1.PA14/SWCLK
- removed net SWDIO: CON2.SWDIO, IC1.PA13/SWDIO
- removed net UART_3V3: C37.1, IC7.A, IC8.V+, R48.1, TP5.1
- removed net UART_GND: C37.2, IC8.GND, TP7.1
- removed net UART_RX: R38.1, TP6.1
- removed net UART_TX: IC8.OUT, TP8.1
- removed net USB_DM: IC1.PA11, R30.2
- removed net USB_DP: IC1.PA12, R31.2
- removed net VBUS: CON1.VBUS, F1.P$1
- new net +5V: C26.1, C42.1, C43.1, IC5.VOUT_LDO1, IC8.CONTROL, IC8.VIN, IC9.CONTROL, IC9.VIN
- new net ADC+: J9.2, R25.1
- new net ADC+_LPF: C32.2, IC11.AIN+, R25.2
- new net ADC-: J7.2, J8.2, R26.1
- new net ADC-_LPF: C33.1, IC11.AIN-, R26.2
- new net VIN: FB1.1, U$9.VIN1, U$9.VIN2, U$9.VIN3, U$9.VIN4
- net +1V8: now also C30.1, C37.1, IC11.AVDD, IC9.VOUT; no longer C11.1, C33.1, IC14.VOUT, IC6.AVDD
- net +3V3A: now also C28.1, C36.1, C40.1, FB6.1, IC13G$7.V+, IC14G$1.!CLR, IC14G$1.!PR, IC14G$2.V+, IC8.VOUT; no longer C10.1, C21.1, C31.1, FB2.1, IC11.VOUT, IC19G$1.!CLR, IC19G$1.!PR, IC19G$2.V+, IC2G$7.V+
- net +9V: now also C1.1, C16.1, C3.1, C6.1, D1.K, IC1.OUT, IC4G$3.V+, IC6G$3.V+, IC7G$3.V+; no longer C41.1, C46.1, C48.1, C7.1, D4.K, IC12G$3.V+, IC13G$3.V+, IC17.OUT, IC18G$3.V+
- net -5V: now also C15.2, IC3.OUT, J3.1; no longer C58.2, IC21.OUT, J9.1
- net -9V: now also C17.2, C2.2, C4.2, D2.A, IC2.OUT, IC4G$3.V-, IC6G$3.V-, J2.1; no longer C42.2, C47.2, C49.2, D5.A, IC12G$3.V-, IC13G$3.V-, IC16.OUT, J5.1
- net ADC_CNVST: now also IC14G$1.D, R3.2; no longer IC19G$1.D, R29.1
- net ADC_CNVST_CLOCKED: now also IC14G$1.Q, R32.2; no longer IC19G$1.Q, R13.2
- net ADC_CNVST_FB: now also IC13G$4.OUT, R4.2; no longer IC2G$4.OUT, R11.1
- net ADC_SCK: now also IC13G$2.IN, R6.2; no longer IC2G$2.IN, R27.1
- net ADC_SDI: now also IC13G$1.IN, R7.2; no longer IC2G$1.IN, R4.1
- net ADC_SDO: now also IC13G$3.OUT, R5.2; no longer IC2G$3.OUT, R28.1
- net CLK_8MHZ: now also IC15.OUT, R38.2; no longer R3.2, TP26.1
- net GND: now also C1.2, C11.1, C13.1, C15.1, C17.1, C19.2, C2.1, C20.2, C22.2, C32.1, C37.2, C4.1, C42.2, C7.1, C9.1, FB2.1, IC1.GND, IC13G$6.IN, IC13G$7.V-, IC14G$2.V-, IC2.GND, IC3.GND, IC4G$1.+IN, IC5.GND_LDO1, IC5.GND_LDO2, IC5.GND_REG, IC5.HT, IC8.GND, J8.1, R2.1, R8.2, TP4.1, TP5.1, U$9.GND1, U$9.GND10, U$9.GND11, U$9.GND12, U$9.GND13, U$9.GND14, U$9.GND15, U$9.GND16, U$9.GND17, U$9.GND18, U$9.GND19, U$9.GND2, U$9.GND20, U$9.GND3, U$9.GND4, U$9.GND5, U$9.GND6, U$9.GND7, U$9.GND8, U$9.GND9; no longer C1.1, C11.2, C13.2, C14.2, C17.2, C2.2, C23.2, C24.1, C32.2, C4.2, C42.1, C46.2, C47.1, C48.2, C49.1, C5.2, C50.1, C52.2, C53.1, C54.2, C55.1, C56.2, C57.2, C58.1, C59.1, C7.2, CON1.GND, CON1.XT, CON2.GND, IC1.BOOT0, IC1.VSSA, IC1.VSS_1, IC1.VSS_2, IC10.GND, IC13G$1.+IN, IC14.GND, IC16.GND, IC17.GND, IC19G$2.V-, IC20.GND, IC21.GND, IC2G$6.IN, IC2G$7.V-, IC3.GND1, IC3.GND2, IC3.GND3, IC4G$3.V-, IC5.GND, IC6.GND, IC7.GND, J7.1, R16.1, R18.1, R19.1, R26.1, R41.1, R47.1, R50.1, R52.1, TP13.1, TP20.1, TP27.1, TP28.1, TP29.1
- net N$1: now also R8.1, R9.1, SW1.3; no longer C5.1, IC1.PF0/OSC_IN, X1.2
- net N$10: now also R6.1, U$9.IO4P_34; no longer IC1.PA7, R4.2
- net N$11: now also IC14G$1.!Q, R37.1; no longer IC19G$1.!Q, R10.1
- net N$12: now also C5.2, J1.2, R1.1; no longer C20.2, J6.2, R20.1
- net N$13: now also IC13G$1.OUT, R31.2; no longer IC2G$1.OUT, R2.2
- net N$14: now also C23.1, IC6G$2.OUT, IC7G$2.+IN, J5.2, R19.2; no longer C9.1, IC12G$2.OUT, IC18G$2.+IN, J1.2, R12.2
- net N$15: now also C39.1, C41.1, FB6.2, IC11.DVIO; no longer C56.1, C6.1, FB2.2, IC6.DVIO
- net N$16: now also C34.1, C35.1, FB5.2, IC11.VREF; no longer C12.1, C13.1, FB3.2, IC6.VREF
- net N$17: now also R5.1, U$9.IO4N_34; no longer IC1.PA15, R8.1
- net N$18: now also IC14G$1.CK, R38.1; no longer IC19G$1.CK, R3.1
- net N$19: now also IC13G$4.IN, R37.2; no longer IC2G$4.IN, R10.2
- net N$2: now also IC7G$2.-IN, IC7G$2.OUT, J5.1, J7.1; no longer IC18G$2.-IN, IC18G$2.OUT, J1.1, J2.1
- net N$20: now also IC13G$3.IN, R34.2; no longer IC2G$3.IN, R25.2
- net N$21: now also R3.1, U$9.IO7P_34; no longer IC1.PA4, R11.2
- net N$22: now also IC13G$5.IN, IC13G$6.OUT; no longer IC2G$5.IN, IC2G$6.OUT
- net N$24: now also J4.2, R15.1; no longer J8.2, R35.1
- net N$25: now also IC11.SDO, R34.1; no longer IC6.SDO, R25.1
- net N$26: now also C24.2, IC6G$1.-IN, R18.2; no longer C19.2, IC12G$1.-IN, R14.2
- net N$28: now also IC11.SCLK, R33.1; no longer IC6.SCLK, R24.1
- net N$29: now also IC11.CNVST, R32.1; no longer IC6.CNVST, R13.1
- net N$3: now also IC4G$2.-IN, SW1.2; no longer C4.1, IC1.PF1_OSC_OUT, X1.1
- net N$30: now also IC11.SDI, R31.1; no longer IC6.SDI, R2.1
- net N$31: now also IC13G$2.OUT, R33.2; no longer IC2G$2.OUT, R24.2
- net N$38: now also R13.1, R14.2; no longer R36.1, R37.2
- net N$4: now also C12.1, R10.2, R11.1, R12.1; no longer C25.1, R39.1, R42.2, R43.1
- net N$41: now also C22.1, IC6G$2.+IN, R14.1, R16.1; no longer C27.1, IC12G$2.+IN, R23.1, R37.1
- net N$42: now also C23.2, IC6G$2.-IN, R19.1, R20.2; no longer C9.2, IC12G$2.-IN, R12.1, R32.2
- net N$43: now also C18.1, R15.2, R18.1, R21.1; no longer C14.1, R14.1, R34.1, R35.2
- net N$44: now also C19.1, IC6G$1.+IN, R16.2, R17.2; no longer C30.1, IC12G$1.+IN, R23.2, R26.2
- net N$45: now also IC4G$2.OUT, R10.1, R9.2; no longer IC13G$2.OUT, R15.2, R42.1, SW1.2
- net N$47: now also C24.1, IC6G$1.OUT, IC7G$1.+IN, J6.2, R20.1, R21.2; no longer C19.1, IC12G$1.OUT, IC18G$1.+IN, J3.2, R32.1, R34.2
- net N$48: now also C5.1, J1.1; no longer C20.1, J6.1
- net N$49: now also D1.A, D2.K, IC4G$2.+IN, R1.2, R2.2; no longer D4.A, D5.K, IC13G$2.+IN, R20.2, R41.2
- net N$5: now also IC7G$1.-IN, IC7G$1.OUT, J6.1, J9.1; no longer IC18G$1.-IN, IC18G$1.OUT, J3.1, J4.1
- net N$55: now also C14.2, IC4G$1.-IN, R12.2; no longer C22.2, IC13G$1.-IN, R39.2
- net N$56: now also C27.1, IC8.BYPASS; no longer C26.1, IC11.BYPASS
- net N$57: now also C14.1, IC4G$1.OUT, J4.1, R11.2; no longer C22.1, IC13G$1.OUT, J8.1, R43.2
- net N$59: now also C29.1, IC9.BYPASS; no longer C32.1, IC14.BYPASS
- net N$6: now also R4.1, U$9.IO7N_34; no longer IC1.PB3, R7.1
- net N$7: now also C31.1, IC5.NP_LDO1; no longer IC1.PB4, R6.1
- net N$70: now also FB3.1; no longer FB1.1
- net N$71: now also FB4.1; no longer FB5.1
- net N$74: now also C7.2, IC7G$3.V-, J2.2, J3.2; no longer C50.2, IC18G$3.V-, J5.2, J9.2
- net N$75: now also FB1.2
- net N$76: now also FB2.2
- net N$8: now also C25.1, C44.1, IC5.NP_LDO2; no longer IC1.PB5, R5.1
- net N$9: now also R7.1, U$9.IO2P_34; no longer IC1.PB0, R29.2
- net V+: now also C10.1, C38.1, C45.1, C8.1, FB3.2, IC1.IN, IC15.EN, IC15.VDD, IC5.EN, IC5.VIN_LDO1, IC5.VIN_LDO2; no longer C39.1, C40.1, C52.1, C54.1, FB1.2, IC10.EN, IC10.VIN, IC11.CONTROL, IC11.VIN, IC14.CONTROL, IC14.VIN, IC17.IN, TP24.1, TP25.1
- net V-: now also C11.2, C13.2, C9.2, FB4.2, IC2.IN, IC3.IN; no longer C53.2, C55.2, C59.2, FB5.2, IC16.IN, IC21.IN
- net VREF: now also C20.1, C21.1, FB5.1, IC5.VOUT_LDO2, R13.2; no longer C17.1, C51.1, FB3.1, R21.2, R22.2, R36.2
Other:
- note added: "ADC / OSC"
- note added: "DCDC / Board"
- note added: "FPGA IO"
- note added: "Input Buffer / LPF"
- note added: "LDOs / VREF"
- moved on the sheet: C1, C10, C11, C12, C13, C14, C15, C16, C17, C18, C19, C2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

Commit message: update
Parts:
- removed D2: CLAMP, my_rcl:DIODE-1N4148W
- removed SW1: Gain, my_connector:SW-1X3
- removed TP15: -D5V, my_connector:TESTPIN
- removed TP16: GND, my_connector:TESTPIN-BIG
- removed TP17: V+, my_connector:TESTPIN
- removed TP18: GND, my_connector:TESTPIN
- removed TP19: V-, my_connector:TESTPIN
- removed TP21: VIN+, my_connector:TESTPIN
- removed TP22: VIN-, my_connector:TESTPIN
- removed TP23: (no value), my_connector:TESTPIN
- removed U$9: FPGA_CORE_BOARD, my_ic:FPGA_CORE_BOARD
- added C46, C52, C55, C58, C60, C64: 10u, my_rcl:C-2012
- added C47: 3300p, my_rcl:C-1608
- added C48, C49, C53, C54, C56, C57, C59, C61, C62, C63: 0.1u, my_rcl:C-1608
- added C50: 10u, my_rcl:C-3216
- added C51: DNP, my_rcl:C-1608
- added IC10: AK1110, my_ic:AK1110
- added IC12, IC16: TAR5SB33, my_ic:TAR5SB33
- added J10: ADC+, my_rcl:SJ-1608
- added J11: GND, my_rcl:SJ-1608
- added J12: ADC-, my_rcl:SJ-1608
- added JP1: GAIN, my_connector:PINHD-1X2
- added R22, R23, R24, R27, R29, R30: 1k, my_rcl:R-1608
- added R28: 3.6k, my_rcl:R-1608
- added R35: 330, my_rcl:R-1608
- added R36: 120, my_rcl:R-1608
- added R39, R40: 22, my_rcl:R-1608
- added R41, R42, R43, R44: 37, my_rcl:R-1608
- added R45, R46: 37, my_rcl:R-1608J
- added R47: 5.1k, my_rcl:R-1608
- added TP10, TP11, TP12, TP7, TP8, TP9: GND, my_connector:TESTPIN
- added TP6: AIN-, my_connector:TESTPIN-MID
- added X1: 12MHz, my_rcl:OSC-KC7050
- C1, C2: value 0.1u -> 1u; device my_rcl:C-1608 -> my_rcl:C-3225
- C10: value 0.1u -> 10u; device my_rcl:C-1608 -> my_rcl:C-2012
- C11: value 0.1u -> 1n
- C12: value 470p -> 1n
- C13: value 0.1u -> 1.5n
- C14: value 100p -> 1.5n
- C15, C41: value 10u -> 1u; device my_rcl:C-2012 -> my_rcl:C-1608
- C16: value 10u -> 1u; device my_rcl:C-3216 -> my_rcl:C-1608
- C17, C25: value 10u -> 0.1u; device my_rcl:C-3216 -> my_rcl:C-1608
- C18: value 470p -> 0.1u
- C19: value 0.1u -> 100u; device my_rcl:C-1608 -> my_rcl:CPOLE2.5-8
- C20: value 1u -> 100u; device my_rcl:C-1608 -> my_rcl:CPOLE2.5-8
- C21, C30, C31: value 10u -> 0.1u; device my_rcl:C-2012 -> my_rcl:C-1608
- C23: value DNP -> 0.1u
- C24: value 100p -> 0.1u
- C28: value 10u -> 10p; device my_rcl:C-2012 -> my_rcl:C-1608
- C29, C6, C7: value 0.1u -> 10p
- C3, C4: value 0.1u -> DNP
- C32, C33: value 470p -> 10u; device my_rcl:C-1608 -> my_rcl:C-3216
- C34, C43: device my_rcl:C-2012 -> my_rcl:C-3216
- C35: value 3300p -> 100u; device my_rcl:C-1608 -> my_rcl:CPOLE2.5-6.5
- C36, C37: value 0.1u -> 100u; device my_rcl:C-1608 -> my_rcl:CPOLE2.5-6.5
- C39, C40: value 0.1u -> 1u
- C42: value 1u -> 10u; device my_rcl:C-1608 -> my_rcl:C-2012
- C44: value DNP -> 470p
- C45: value 1u -> 470p
- C5: value 10u -> DNP; device my_rcl:C-5 -> my_rcl:C-1608
- C8, C9: value 100u -> 2.7n; device my_rcl:CPOLE2.5-8 -> my_rcl:C-1608
- D1: value CLAMP -> PWR; device my_rcl:DIODE-1N4148W -> my_rcl:LED-SMD1608
- FB1, FB2, FB3, FB4: value FB-2012 -> FB
- IC1: value +9V -> FPGA CORE BOARD; device my_ic:78LX -> my_ic:FPGA_CORE_BOARD
- IC13: value 7404 -> 74HC3G34; device my_ic:7404 -> my_ic:74HC3G34
- IC15: value OSC -> NJM12888F18; device my_ic:OSC -> my_ic:NJM12888
- IC2: value -9V -> OPA; device my_ic:79LX -> my_ic:OPA-2-SOP
- IC3: value -5V -> OPA-DIFF; device my_ic:79LX -> my_ic:OPA-DIFF
- IC4: value LM4562 -> DCDC2; device my_ic:OPA-2-DUAL -> my_ic:DCDC2
- IC5: value AK1110 -> OPA-DIFF; device my_ic:AK1110 -> my_ic:OPA-DIFF
- IC6: value LM4562 -> OPA-DIFF; device my_ic:OPA-2-DUAL -> my_ic:OPA-DIFF
- IC7: value LM4562 -> LM317-L; device my_ic:OPA-2-DUAL -> my_ic:LM317-L
- IC8: value TAR5SB33 -> LM337-L; device my_ic:TAR5SB33 -> my_ic:LM337-L
- IC9: value NJM12888F18 -> LM337-L; device my_ic:NJM12888 -> my_ic:LM337-L
- J1: value IN1_DC -> DC; device my_rcl:SJ-2012 -> my_rcl:SJ-1608
- J2: value SJ-2012 -> DC; device my_rcl:SJ-2012 -> my_rcl:SJ-1608
- J3, J5: value SJ-2012 -> VCOM; device my_rcl:SJ-2012 -> my_rcl:SJ-3-1608
- J4: value short -> GND
- J6: value SJ-2012 -> V-; device my_rcl:SJ-2012 -> my_rcl:SJ-3-2012
- J7, J8, J9: value SJ-1608 -> V-; device my_rcl:SJ-1608 -> my_rcl:SJ-3-2012
- R1: device my_rcl:R-1608J -> my_rcl:R-2012
- R10, R11: value 1k -> 100
- R2: value 100k -> 10; device my_rcl:R-1608 -> my_rcl:R-2012
- R25: value 22 -> 3.6k
- R26: value 22 -> 1k
- R3, R4: value 22 -> 10k; device my_rcl:R-1608J -> my_rcl:R-1608
- R31, R32: value 37 -> 1k; device my_rcl:R-1608J -> my_rcl:R-1608
- R33, R34: value 37 -> 680; device my_rcl:R-1608J -> my_rcl:R-1608
- R37, R38: value 37 -> 120; device my_rcl:R-1608J -> my_rcl:R-1608
- R8: value 1k -> 22; device my_rcl:R-1608 -> my_rcl:R-1608J
- R9: value 10k -> 22; device my_rcl:R-1608 -> my_rcl:R-1608J
- TP1: value +D5V -> GND; device my_connector:TESTPIN -> my_connector:TESTPIN-MID
- TP2: value AIN1 -> AIN+; device my_connector:TESTPIN-BIG -> my_connector:TESTPIN-MID
- TP3: device my_connector:TESTPIN -> my_connector:TESTPIN-MID
Connections:
- new net ADC_VCOM: C10.1, IC6G$1.CM, J3.3, J5.3, R23.1, R24.2
- new net N$23: C4.2, C5.1, IC2G$2.+IN, R2.2, R4.2
- new net N$27: C13.1, IC5G$1.+IN, R26.2
- new net N$32: C12.2, C13.2, IC5G$1.-OUT, R25.2, R29.1
- new net N$33: C11.2, C14.2, IC5G$1.+OUT, R28.2, R30.1
- new net N$34: C14.1, IC5G$1.-IN, R27.2
- new net N$35: C12.1, R22.2, R27.1, R28.1
- new net N$36: C11.1, R21.2, R25.1, R26.1
- new net N$37: C7.2, IC3G$1.+OUT, R18.2, R20.1
- new net N$39: C7.1, IC3G$1.-IN, R16.2, R18.1
- new net N$40: C6.1, IC3G$1.+IN, R15.2, R17.1
- new net N$46: JP1.2, R11.1
- new net N$50: C27.2, IC5G$2.V-, J8.2
- new net N$51: C22.2, IC3G$2.V-, J7.2
- new net N$52: C18.2, IC2G$3.V-, J6.2
- new net N$53: C32.1, IC7.ADJ, R33.2, R36.1
- new net N$54: C33.2, IC8.ADJ, R34.1, R37.1
- new net N$58: D1.A, R47.1
- new net VCC_OSC: C63.1, C64.1, IC16.VOUT, X1.EN, X1.VCC
- net +1V8: now also C49.1, C60.1, IC15.VOUT; no longer C30.1, C37.1, IC9.VOUT
- net +3V3A: now also C48.1, C54.1, C58.1, IC12.VOUT, IC13G$4.V+; no longer C28.1, C36.1, C40.1, IC13G$7.V+, IC8.VOUT
- net +5V: now also C40.1, C56.1, C61.1, IC10.VOUT_LDO1, IC12.CONTROL, IC12.VIN, IC15.CONTROL, IC15.VIN, IC16.CONTROL, IC16.VIN, R47.2; no longer C26.1, C43.1, IC5.VOUT_LDO1, IC8.CONTROL, IC8.VIN, IC9.CONTROL, IC9.VIN
- net +9V: now also C17.1, C21.1, C26.1, C30.1, C35.1, IC2G$3.V+, IC3G$1.EN, IC3G$2.V+, IC5G$1.EN, IC5G$2.V+, IC6G$1.EN, IC6G$2.V+, IC7.OUT, R36.2; no longer C1.1, C16.1, C3.1, C6.1, D1.K, IC1.OUT, IC4G$3.V+, IC6G$3.V+, IC7G$3.V+
- net -5V: now also C37.2, IC9.OUT, J6.1, J7.1, J8.1, J9.1, R38.2; no longer C15.2, IC3.OUT, J3.1
- net -9V: now also C36.2, IC8.OUT, J6.3, J7.3, J8.3, J9.3, R37.2; no longer C17.2, C2.2, C4.2, D2.A, IC2.OUT, IC4G$3.V-, IC6G$3.V-, J2.1
- net ADC+: now also J10.2, R39.1; no longer J9.2, R25.1
- net ADC+_LPF: now also C44.2, R39.2; no longer C32.2, R25.2
- net ADC-: now also J11.2, J12.2, R40.1; no longer J7.2, J8.2, R26.1
- net ADC-_LPF: now also C45.1, R40.2; no longer C33.1, R26.2
- net ADC_CNVST: now also R9.2; no longer R3.2
- net ADC_CNVST_CLOCKED: now also R42.2; no longer R32.2
- net ADC_CNVST_FB: now also R45.2, R8.2; no longer IC13G$4.OUT, R4.2
- net ADC_SDI: now also R5.2; no longer R7.2
- net ADC_SDO: now also R7.2; no longer R5.2
- net CLK_8MHZ: now also R46.2, X1.OUT; no longer IC15.OUT, R38.2
- net GND: now also C15.2, C16.1, C17.2, C18.1, C20.1, C22.1, C23.2, C24.1, C25.1, C27.1, C3.1, C31.1, C32.2, C33.1, C34.1, C36.1, C37.1, C44.1, C46.2, C47.2, C48.2, C49.2, C5.2, C50.2, C51.2, C52.2, C53.2, C54.2, C55.2, C56.2, C57.2, C58.2, C59.2, C60.2, C61.2, C62.2, C63.2, C64.2, C9.2, D1.K, IC1.GND1@7, IC1.GND1@8, IC1.GND@1, IC1.GND@10, IC1.GND@11, IC1.GND@12, IC1.GND@13, IC1.GND@14, IC1.GND@15, IC1.GND@16, IC1.GND@19, IC1.GND@2, IC1.GND@20, IC1.GND@3, IC1.GND@4, IC1.GND@5, IC1.GND@6, IC1.GND@7, IC1.GND@8, IC1.GND@9, IC10.GND_LDO1, IC10.GND_LDO2, IC10.GND_REG, IC10.HT, IC12.GND, IC13G$4.V-, IC16.GND, IC4.GND, J11.1, J3.1, J4.1, J5.1, R24.1, R3.2, R33.1, R34.2, R35.2, R4.1, TP1.1, TP10.1, TP11.1, TP12.1, TP7.1, TP8.1, TP9.1, X1.GND; no longer C1.2, C11.1, C12.2, C13.1, C15.1, C16.2, C17.1, C18.2, C2.1, C20.2, C22.2, C25.2, C27.2, C28.2, C29.2, C3.2, C31.2, C32.1, C33.2, C34.2, C36.2, C37.2, C4.1, C44.2, C6.2, C7.1, C9.1, FB2.1, IC1.GND, IC13G$6.IN, IC13G$7.V-, IC2.GND, IC3.GND, IC4G$1.+IN, IC5.GND_LDO1, IC5.GND_LDO2, IC5.GND_REG, IC5.HT, IC8.GND, IC9.GND, J8.1, R17.1, R2.1, R8.2, TP16.1, TP18.1, U$9.GND1, U$9.GND10, U$9.GND11, U$9.GND12, U$9.GND13, U$9.GND14, U$9.GND15, U$9.GND16, U$9.GND17, U$9.GND18, U$9.GND19, U$9.GND2, U$9.GND20, U$9.GND3, U$9.GND4, U$9.GND5, U$9.GND6, U$9.GND7, U$9.GND8, U$9.GND9
- net N$1: now also IC2G$2.-IN, R11.2, R12.1, R14.1; no longer R8.1, R9.1, SW1.3
- net N$10: now also IC1.IO4P_34/N1; no longer U$9.IO4P_34
- net N$11: now also R45.1; no longer R37.1
- net N$12: now also IC2G$2.OUT, R14.2, R16.1; no longer C5.2, J1.2, R1.1
- net N$13: now also R41.2; no longer R31.2
- net N$14: now also C3.2, C4.1, IC2G$1.+IN, R1.2, R3.1; no longer C23.1, IC6G$2.OUT, IC7G$2.+IN, J5.2, R19.2
- net N$15: now also C53.1, C55.1; no longer C39.1, C41.1
- net N$16: now also C46.1, C47.1; no longer C34.1, C35.1
- net N$17: now also IC1.IO4N_34/P1, R7.1; no longer R5.1, U$9.IO4N_34
- net N$18: now also R46.1; no longer R38.1
- net N$19: now also C29.1, IC6G$1.-IN, R30.2, R32.1; no longer IC13G$4.IN, R37.2
- net N$2: now also C29.2, IC6G$1.+OUT, J12.1, R32.2; no longer IC7G$2.-IN, IC7G$2.OUT, J5.1, J7.1
- net N$20: now also R44.2; no longer R34.2
- net N$21: now also IC1.IO7P_34/R2, R9.1; no longer R3.1, U$9.IO7P_34
- net N$22: now also C28.1, IC6G$1.+IN, R29.2, R31.1; no longer IC13G$5.IN, IC13G$6.OUT
- net N$24: now also C8.1, R19.2, R21.1; no longer J4.2, R15.1
- net N$25: now also R44.1; no longer R34.1
- net N$26: now also C9.1, R20.2, R22.1; no longer C24.2, IC6G$1.-IN, R18.2
- net N$28: now also R43.1; no longer R33.1
- net N$29: now also R42.1; no longer R32.1
- net N$3: now also IC2G$1.-IN, R10.2, R12.2, R13.1; no longer IC4G$2.-IN, SW1.2
- net N$30: now also R41.1; no longer R31.1
- net N$31: now also R43.2; no longer R33.2
- net N$38: now also C6.2, IC3G$1.-OUT, R17.2, R19.1; no longer R13.1, R14.2
- net N$4: now also IC2G$1.OUT, R13.2, R15.1; no longer C12.1, R10.2, R11.1, R12.1
- net N$41: now also C1.1, J1.1, TP2.1; no longer C22.1, IC6G$2.+IN, R14.1, R16.1
- net N$42: now also C2.1, J2.1, TP6.1; no longer C23.2, IC6G$2.-IN, R19.1, R20.2
- net N$43: now also C1.2, J1.2, R1.1; no longer C18.1, R15.2, R18.1, R21.1
- net N$44: now also C2.2, J2.2, R2.1; no longer C19.1, IC6G$1.+IN, R16.2, R17.2
- net N$45: now also JP1.1; no longer IC4G$2.OUT, R9.2, SW1.1
- net N$47: now also IC5G$1.CM, J5.2; no longer C24.1, IC6G$1.OUT, IC7G$1.+IN, J6.2, R20.1, R21.2
- net N$48: now also C62.1, IC16.BYPASS; no longer C5.1, J1.1, TP2.1
- net N$49: now also IC3G$1.CM, J3.2; no longer D1.A, D2.K, IC4G$2.+IN, R1.2, R2.2
- net N$5: now also C28.2, IC6G$1.-OUT, J10.1, R31.2; no longer IC7G$1.-IN, IC7G$1.OUT, J6.1, J9.1
- net N$55: now also C34.2, IC9.ADJ, R35.1, R38.1; no longer C14.2, IC4G$1.-IN, R12.2
- net N$56: now also C57.1, IC12.BYPASS; no longer C27.1, IC8.BYPASS
- net N$57: now also FB2.1, J4.2; no longer C14.1, IC4G$1.OUT, J4.1, R11.2
- net N$59: now also C59.1, IC15.BYPASS; no longer C29.1, IC9.BYPASS
- net N$6: now also IC1.IO7N_34/R1, R8.1; no longer R4.1, U$9.IO7N_34
- net N$7: now also C52.1, IC10.NP_LDO1; no longer C31.1, IC5.NP_LDO1
- net N$70: now also IC4.V+; no longer TP17.1
- net N$71: now also IC4.V-; no longer TP19.1
- net N$74: now also C31.2, IC6G$2.V-, J9.2; no longer C7.2, IC7G$3.V-, J2.2, J3.2
- net N$75: now also IC4.VIN+; no longer TP21.1
- net N$76: now also IC4.VIN-; no longer TP22.1
- net N$8: now also C50.1, C51.1, IC10.NP_LDO2; no longer C25.1, C44.1, IC5.NP_LDO2
- net N$9: now also IC1.IO2P_34/M2, R5.1; no longer R7.1, U$9.IO2P_34
- net V+: now also C15.1, C19.1, C23.1, C39.1, IC10.EN, IC10.VIN_LDO1, IC10.VIN_LDO2, IC7.IN; no longer C10.1, C45.1, C8.1, IC1.IN, IC15.EN, IC15.VDD, IC5.EN, IC5.VIN_LDO1, IC5.VIN_LDO2
- net V-: now also C16.2, C20.2, C24.2, C25.2, IC8.IN, IC9.IN; no longer C11.2, C13.2, C9.2, IC2.IN, IC3.IN
- net VIN: now also IC1.VIN@1, IC1.VIN@2, IC1.VIN@3, IC1.VIN@4; no longer U$9.VIN1, U$9.VIN2, U$9.VIN3, U$9.VIN4
- net VREF: now also C41.1, C43.1, IC10.VOUT_LDO2, R23.2; no longer C20.1, C21.1, IC5.VOUT_LDO2, R13.2
Other:
- moved on the sheet: C1, C10, C11, C12, C13, C14, C15, C16, C17, C18, C2, C21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
