File: ADC2.sch (EAGLE design)
At the start: 166 parts, among them IC1 FPGA CORE BOARD, IC10 AK1110, IC11 AD4001, IC12 TAR5SB33, IC13 74HC3G34, IC14 TC7WH74FU, IC15 NJM12888F18, IC16 TAR5SB33, IC2 OPA, IC3 OPA-DIFF, IC4 DCDC2, IC5 OPA-DIFF, IC6 OPA-DIFF, IC7 LM317-L, IC8 LM337-L, IC9 LM337-L, J1 DC, J10 ADC+, J11 GND, J12 ADC-, J2 DC, J3 VCOM, J4 GND, J5 VCOM, J6 V-, J7 V-, J8 V-, J9 V-, X1 12MHz

Commit message: 途中
Parts:
- removed C33: 10u, my_rcl:C-3216
- removed C36: 100u, my_rcl:CPOLE2.5-6.5
- removed C38: 1u, my_rcl:C-1608
- removed C48, C54, C57, C59, C61, C62: 0.1u, my_rcl:C-1608
- removed C51: DNP, my_rcl:C-1608
- removed IC15: NJM12888F18, my_ic:NJM12888
- removed IC16: TAR5SB33, my_ic:TAR5SB33
- removed IC8: LM337-L, my_ic:LM337-L
- removed J6, J7, J8, J9: V-, my_rcl:SJ-3-2012
- removed R22: 1k, my_rcl:R-1608
- removed R34: 680, my_rcl:R-1608
- removed R37: 120, my_rcl:R-1608
- removed R41, R42, R43, R44: 37, my_rcl:R-1608
- added D2: PWR, my_rcl:LED-SMD1608
- added FB7: FB, my_rcl:FB-1608FB
- added IC17: ISO7762FB, my_ic:ISO6762-SSOP
- added SW1: MODE-SW, my_rcl:DIPSW-4
- added TP13: ADC+, my_connector:TESTPIN
- added TP14: ADC-, my_connector:TESTPIN
- added TP15, TP16, TP17, TP18, TP19, TP22, TP23, TP24: GND, my_connector:TESTPIN
- added TP20: -5V, my_connector:TESTPIN
- added TP21: +9V, my_connector:TESTPIN
- C11, C12: value 1n -> 10p
- C13, C14: value 1.5n -> 470p
- C21: value 0.1u -> 10u; device my_rcl:C-1608 -> my_rcl:C-2012
- C28, C29, C6: value 10p -> 0.1u
- C4: value DNP -> 22p
- C44, C45: value 470p -> 100p
- C47: value 3300p -> 1n; device my_rcl:C-1608 -> my_rcl:C-1005
- C50: device my_rcl:C-3216 -> my_rcl:C-2012
- C7: value 10p -> 4.7u
- C8: value 2.7n -> 1n
- C9: value 2.7n -> 22p
- D1: value PWR -> CLIP
- FB5, FB6: device my_rcl:FB -> my_rcl:FB-1608FB
- IC12: value TAR5SB33 -> 1.8V; device my_ic:TAR5SB33 -> my_ic:TLV740
- IC13: value 74HC3G34 -> 2.5V; device my_ic:74HC3G34 -> my_ic:TLV740
- IC3: value OPA-DIFF -> 3.3V; device my_ic:OPA-DIFF -> my_ic:TLV740
- IC5: value OPA-DIFF -> OPA1632
- IC6: value OPA-DIFF -> AP22652; device my_ic:OPA-DIFF -> my_ic:AP22652
- J3: value VCOM -> SIG+
- J5: value VCOM -> SIG-
- R1, R2: device my_rcl:R-2012 -> my_rcl:R-2012H
- R10, R11: value 100 -> 24; device my_rcl:R-1608 -> my_rcl:R-1608-3
- R12: value 1k -> 51; device my_rcl:R-1608 -> my_rcl:R-ARRAY
- R15: value 1k -> 51; device my_rcl:R-1608 -> my_rcl:R-1608-3
- R16, R17, R18: value 1k -> 10k
- R19, R20: device my_rcl:R-1608 -> my_rcl:R-1608-3
- R21: value 1k -> 10M; device my_rcl:R-1608 -> my_rcl:R-7.5
- R25, R28: value 3.6k -> 1k; device my_rcl:R-1608 -> my_rcl:R-1608-3
- R26, R27: value 1k -> 360; device my_rcl:R-1608 -> my_rcl:R-1608-3
- R29: value 1k -> CNVST; device my_rcl:R-1608 -> my_rcl:R-1608-3
- R30: value 1k -> SCK; device my_rcl:R-1608 -> my_rcl:R-1608-3
- R31: value 1k -> SDI; device my_rcl:R-1608 -> my_rcl:R-1608-3
- R32: value 1k -> LED1; device my_rcl:R-1608 -> my_rcl:R-1608-3
- R39, R40: value 22 -> 24; device my_rcl:R-1608 -> my_rcl:R-1608-3
- R45: value 37 -> SDO; device my_rcl:R-1608J -> my_rcl:R-1608-3
- R46: value 37 -> CNVST_FB; device my_rcl:R-1608J -> my_rcl:R-1608-3
- R47: value 5.1k -> 1.5k
- R5, R6: value 22 -> 50; device my_rcl:R-1608J -> my_rcl:R-1608
- R7: value 22 -> 30k; device my_rcl:R-1608J -> my_rcl:R-1608
- R8: value 22 -> 5.1k; device my_rcl:R-1608J -> my_rcl:R-1608
- R9: value 22 -> 10k; device my_rcl:R-1608J -> my_rcl:R-1608
- TP2: value AIN+ -> IN+
- TP6: value AIN- -> IN-
Connections:
- net N$15 renamed ADC_DVIO
- removed net +3V3A: C48.1, C54.1, C58.1, FB6.1, IC12.VOUT, IC13G$4.V+, IC14G$1.!CLR, IC14G$1.!PR, IC14G$2.V+
- removed net -9V: C36.2, IC8.OUT, J6.3, J7.3, J8.3, J9.3, R37.2
- removed net CLK_8MHZ: R46.2, X1.OUT
- removed net N$31: IC13G$2.OUT, R43.2
- removed net N$35: C12.1, R22.2, R27.1, R28.1
- removed net N$36: C11.1, R21.2, R25.1, R26.1
- removed net N$37: C7.2, IC3G$1.+OUT, R18.2, R20.1
- removed net N$38: C6.2, IC3G$1.-OUT, R17.2, R19.1
- removed net N$39: C7.1, IC3G$1.-IN, R16.2, R18.1
- removed net N$40: C6.1, IC3G$1.+IN, R15.2, R17.1
- removed net N$47: IC5G$1.CM, J5.2
- removed net N$48: C62.1, IC16.BYPASS
- removed net N$49: IC3G$1.CM, J3.2
- removed net N$50: C27.2, IC5G$2.V-, J8.2
- removed net N$51: C22.2, IC3G$2.V-, J7.2
- removed net N$52: C18.2, IC2G$3.V-, J6.2
- removed net N$54: C33.2, IC8.ADJ, R34.1, R37.1
- removed net N$56: C57.1, IC12.BYPASS
- removed net N$59: C59.1, IC15.BYPASS
- removed net N$74: C31.2, IC6G$2.V-, J9.2
- new net +2V5: C28.1, C29.1, C58.1, FB6.1, IC12.OUT, IC14G$1.!CLR, IC14G$1.!PR, IC14G$2.V+, IC17.VCC2
- new net +3V3D: C6.1, C7.1, IC1.+3V3@1, IC1.+3V3@2, IC1.+3V3@3, IC1.+3V3@4, IC1.+3V3@5, IC1.+3V3@6, IC17.VCC1, R16.2, R17.2, R18.2, R9.2
- new net ADC_LED1: IC17.OUT4, R47.2
- new net ADC_VREF: C31.1, C46.1, C47.1, FB5.2, IC11.VREF
- new net CLK_OSC: IC14G$1.CK, R15.1
- new net DGND: C24.2, C30.2, C6.2, C7.2, IC1.GND@1, IC1.GND@10, IC1.GND@11, IC1.GND@12, IC1.GND@13, IC1.GND@14, IC1.GND@15, IC1.GND@16, IC1.GND@17, IC1.GND@18, IC1.GND@19, IC1.GND@2, IC1.GND@20, IC1.GND@3, IC1.GND@4, IC1.GND@5, IC1.GND@6, IC1.GND@7, IC1.GND@8, IC1.GND@9, IC17.GND1, IC6.!EN, IC6.GND, J4.1, R21.2, R7.1, SW1.B1, SW1.B2, SW1.B3, SW1.B4, TP22.1, TP23.1, TP24.1
- new net DIP_SW1: IC1.IO0_14/K12, R9.1, SW1.A1
- new net DIP_SW2: IC1.IO5P_14/K13, R16.1, SW1.A2
- new net DIP_SW3: IC1.IO12P_14/N14, R17.1, SW1.A3
- new net DIP_SW4: IC1.IO12N_14/P14, R18.1, SW1.A4
- new net FPGA_CNVST: IC1.IO7P_34/R2, R29.2
- new net FPGA_CNVST_FB: IC1.IO2N_34/M1, R46.2
- new net FPGA_LED1: IC1.IO4P_34/N1, R32.2
- new net FPGA_SCK: IC1.IO7N_34/R1, R30.2
- new net FPGA_SDI: IC1.IO4N_34/P1, R31.2
- new net FPGA_SDO: IC1.IO2P_34/M2, R45.2
- new net VIN_LIM: C24.1, FB1.1, IC6.OUT
- net +1V8: now also IC13.OUT; no longer IC15.VOUT
- net +5V: now also FB7.1, IC10.VOUT1, IC12.EN, IC12.IN, IC13.EN, IC13.IN, R8.2; no longer C61.1, IC10.VOUT_LDO1, IC12.CONTROL, IC12.VIN, IC15.CONTROL, IC15.VIN, IC16.CONTROL, IC16.VIN, R47.2
- net +9V: now also IC5G$2.EN, TP21.1; no longer C21.1, C30.1, IC3G$1.EN, IC3G$2.V+, IC5G$1.EN, IC6G$1.EN, IC6G$2.V+
- net -5V: now also C18.2, C27.2, IC2G$3.V-, IC5G$2.V-, TP20.1; no longer J6.1, J7.1, J8.1, J9.1
- net ADC+: now also TP13.1
- net ADC-: now also TP14.1
- net ADC_CNVST: now also IC17.OUT1; no longer R9.2
- net ADC_CNVST_CLOCKED: now also R12G$4.2; no longer R42.2
- net ADC_CNVST_FB: now also IC14G$1.!Q, IC17.IN6; no longer R45.2, R8.2
- net ADC_SCK: now also IC17.OUT2, R12G$2.2; no longer IC13G$2.IN, R6.2
- net ADC_SDI: now also IC17.OUT3, R12G$1.2; no longer IC13G$1.IN, R5.2
- net ADC_SDO: now also IC17.IN5, R12G$3.2; no longer IC13G$3.OUT, R7.2
- net ADC_VCOM: now also IC5G$1.CM; no longer IC6G$1.CM, J3.3, J5.3
- net GND: now also C22.2, C28.2, C29.2, C31.2, C4.2, C9.1, D2.K, IC10.GND1, IC10.GND2, IC13.GND, IC17.GND2, IC3.GND, R21.1, TP15.1, TP16.1, TP17.1, TP18.1, TP19.1; no longer C22.1, C24.1, C30.2, C31.1, C33.1, C36.1, C38.2, C48.2, C51.2, C54.2, C57.2, C59.2, C61.2, C62.2, C8.2, C9.2, IC1.GND1@7, IC1.GND1@8, IC1.GND@1, IC1.GND@10, IC1.GND@11, IC1.GND@12, IC1.GND@13, IC1.GND@14, IC1.GND@15, IC1.GND@16, IC1.GND@19, IC1.GND@2, IC1.GND@20, IC1.GND@3, IC1.GND@4, IC1.GND@5, IC1.GND@6, IC1.GND@7, IC1.GND@8, IC1.GND@9, IC10.GND_LDO1, IC10.GND_LDO2, IC13G$4.V-, IC15.GND, IC16.GND, J3.1, J4.1, J5.1, R34.2
- net N$1: now also J5.2, R20.1; no longer IC2G$2.-IN, R11.2, R12.1, R14.1
- net N$10: now also C12.1, IC2G$2.-IN, R11.2, R14.1; no longer IC1.IO4P_34/N1, R6.1
- net N$11: now also IC17.IN4, R32.1; no longer IC14G$1.!Q, R45.1
- net N$12: now also C9.2, R6.2; no longer IC2G$2.OUT, R14.2, R16.1
- net N$13: now also IC17.IN3, R31.1; no longer IC13G$1.OUT, R41.2
- net N$14: now also J3.3, R6.1; no longer C4.1, R3.1
- net N$16: now also C21.1, C22.1, FB7.2, IC3.EN, IC3.IN; no longer C46.1, C47.1, FB5.2, IC11.VREF
- net N$17: now also C8.1, R19.2, R25.1, R26.1; no longer IC1.IO4N_34/P1, R7.1
- net N$18: now also IC17.IN2, R30.1; no longer IC14G$1.CK, R46.1
- net N$19: now also IC17.IN1, R29.1; no longer C29.1, IC6G$1.-IN, R30.2, R32.1
- net N$2: now also IC17.OUT6, R46.1; no longer C29.2, IC6G$1.+OUT, J12.1, R32.2
- net N$20: now also R15.2, X1.OUT; no longer IC13G$3.IN, R44.2
- net N$21: now also C12.2, IC2G$2.OUT, J5.3, R14.2; no longer IC1.IO7P_34/R2, R9.1
- net N$22: now also C8.2, R20.2, R27.1, R28.1; no longer C28.1, IC6G$1.+IN, R29.2, R31.1
- net N$23: now also J5.1, R5.2; no longer C4.2, R4.2
- net N$24: now also IC6.ILIM, R7.2; no longer C8.1, R19.2, R21.1
- net N$25: now also R12G$3.1; no longer R44.1
- net N$26: now also D2.A, R8.1; no longer C9.1, R20.2, R22.1
- net N$28: now also R12G$2.1; no longer R43.1
- net N$29: now also R12G$4.1; no longer R42.1
- net N$3: now also C11.1; no longer R12.2
- net N$30: now also R12G$1.1; no longer R41.1
- net N$32: now also J10.1; no longer C12.2, R29.1
- net N$33: now also J12.1; no longer C11.2, R30.1
- net N$4: now also C11.2, J3.1; no longer R15.1
- net N$43: now also R3.1
- net N$44: now also R4.2
- net N$5: now also IC17.OUT5, R45.1; no longer C28.2, IC6G$1.-OUT, J10.1, R31.2
- net N$6: now also J3.2, R19.1; no longer IC1.IO7N_34/R1, R8.1
- net N$7: now also IC10.NP1; no longer IC10.NP_LDO1
- net N$8: now also IC10.NP2; no longer C51.1, IC10.NP_LDO2
- net N$9: now also C4.1; no longer IC1.IO2P_34/M2
- net V+: now also IC10.VIN1, IC10.VIN2; no longer C38.1, IC10.VIN_LDO1, IC10.VIN_LDO2
- net V-: no longer C24.2, IC8.IN
- net VCC_OSC: now also IC3.OUT; no longer IC16.VOUT
- net VIN: now also C30.1, IC6.IN; no longer FB1.1
- net VREF: now also IC10.VOUT2; no longer IC10.VOUT_LDO2
Other:
- moved on the sheet: C1, C10, C11, C12, C13, C14, C15, C16, C17, C18, C19, C2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

Commit message: 微修正
Parts:
- IC12: value 1.8V -> 2.5V
- IC13: value 2.5V -> 1.8V
Changed lines of the file:
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@@
 <part name="C29" library="my_rcl" deviceset="C" device="-1608" value="0.1u"/>
 <part name="SUPPLY101" library="my_supply" deviceset="GND" device=""/>
-<part name="IC12" library="my_ic" deviceset="TLV740" device="" value="1.8V"/>
-<part name="IC13" library="my_ic" deviceset="TLV740" device="" value="2.5V"/>
+<part name="IC12" library="my_ic" deviceset="TLV740" device="" value="2.5V"/>
+<part name="IC13" library="my_ic" deviceset="TLV740" device="" value="1.8V"/>
 <part name="J3" library="my_rcl" deviceset="SJ-3" device="-1608" value="SIG+"/>
 <part name="J5" library="my_rcl" deviceset="SJ-3" device="-1608" value="SIG-"/>
