File: ADC2.brd (EAGLE design)
At the start: 99.1 x 88.9 mm, 166 parts, among them IC1 FPGA CORE BOARD, IC10 AK1110, IC11 AD4001, IC12 TAR5SB33, IC13 74HC3G34, IC14 TC7WH74FU, IC15 NJM12888F18, IC16 TAR5SB33, IC2 OPA, IC3 OPA-DIFF, IC4 DCDC2, IC5 OPA-DIFF, IC6 OPA-DIFF, IC7 LM317-L, IC8 LM337-L, IC9 LM337-L, J1 DC, J10 ADC+, J11 GND, J12 ADC-, J2 DC, J3 VCOM, J4 GND, J5 VCOM, J6 V-, J7 V-, J8 V-, J9 V-, X1 12MHz

Commit message: 途中
Parts:
- removed C33: 10u, my_rcl:3216
- removed C36: 100u, my_rcl:E2.5-6.5
- removed C38: 1u, my_rcl:1608C
- removed C48, C54, C57, C59, C61, C62: 0.1u, my_rcl:1608C
- removed C51: DNP, my_rcl:1608C
- removed IC15: NJM12888F18, my_ic:SOT23-5
- removed IC16: TAR5SB33, my_ic:SOT23-5
- removed IC8: LM337-L, my_ic:TO-92
- removed J6, J7, J8, J9: V-, my_rcl:2012-3-J
- removed R22: 1k, my_rcl:1608
- removed R34: 680, my_rcl:1608
- removed R37: 120, my_rcl:1608
- removed R41, R42, R43, R44: 37, my_rcl:1608
- added D2: PWR, my_rcl:D1608
- added FB7: FB, my_rcl:1608-FB
- added IC17: ISO7762FB, my_ic:TSSOP16
- added SW1: MODE-SW, my_rcl:DIPSW-4
- added TP13: ADC+, my_connector:TESTPIN
- added TP14: ADC-, my_connector:TESTPIN
- added TP15, TP16, TP17, TP18, TP19, TP22, TP23, TP24: GND, my_connector:TESTPIN
- added TP20: -5V, my_connector:TESTPIN
- added TP21: +9V, my_connector:TESTPIN
- C11, C12: value 1n -> 10p
- C13, C14: value 1.5n -> 470p
- C21: value 0.1u -> 10u; device my_rcl:1608C -> my_rcl:2012
- C28, C29, C6: value 10p -> 0.1u
- C4: value DNP -> 22p
- C44, C45: value 470p -> 100p
- C47: value 3300p -> 1n; device my_rcl:1608C -> my_rcl:1005
- C50: device my_rcl:3216 -> my_rcl:2012
- C7: value 10p -> 4.7u
- C8: value 2.7n -> 1n
- C9: value 2.7n -> 22p
- D1: value PWR -> CLIP
- FB5, FB6: device my_rcl:1608-J -> my_rcl:1608-FB
- IC12: value TAR5SB33 -> 1.8V
- IC13: value 74HC3G34 -> 2.5V; device my_ic:SOT765 -> my_ic:SOT23-5
- IC2: device my_ic:SOP8 -> my_ic:SOP8-3
- IC3: value OPA-DIFF -> 3.3V; device my_ic:SOP8 -> my_ic:SOT23-5
- IC5: value OPA-DIFF -> OPA1632; device my_ic:SOP8 -> my_ic:SOP8-3
- IC6: value OPA-DIFF -> AP22652; device my_ic:SOP8 -> my_ic:SOT23-6
- J3: value VCOM -> SIG+
- J5: value VCOM -> SIG-
- R1, R2: device my_rcl:2012 -> my_rcl:2012-R
- R10, R11: value 100 -> 24; device my_rcl:1608 -> my_rcl:1608-3
- R12: value 1k -> 51; device my_rcl:1608 -> my_rcl:EXB28V
- R15: value 1k -> 51; device my_rcl:1608 -> my_rcl:1608-3
- R16, R17, R18: value 1k -> 10k
- R19, R20: device my_rcl:1608 -> my_rcl:1608-3
- R21: value 1k -> 10M; device my_rcl:1608 -> my_rcl:0204/7
- R25, R28: value 3.6k -> 1k; device my_rcl:1608 -> my_rcl:1608-3
- R26, R27: value 1k -> 360; device my_rcl:1608 -> my_rcl:1608-3
- R29: value 1k -> CNVST; device my_rcl:1608 -> my_rcl:1608-3
- R30: value 1k -> SCK; device my_rcl:1608 -> my_rcl:1608-3
- R31: value 1k -> SDI; device my_rcl:1608 -> my_rcl:1608-3
- R32: value 1k -> LED1; device my_rcl:1608 -> my_rcl:1608-3
- R39, R40: value 22 -> 24; device my_rcl:1608 -> my_rcl:1608-3
- R45: value 37 -> SDO; device my_rcl:1608-J -> my_rcl:1608-3
- R46: value 37 -> CNVST_FB; device my_rcl:1608-J -> my_rcl:1608-3
- R47: value 5.1k -> 1.5k
- R5, R6: value 22 -> 50; device my_rcl:1608-J -> my_rcl:1608
- R7: value 22 -> 30k; device my_rcl:1608-J -> my_rcl:1608
- R8: value 22 -> 5.1k; device my_rcl:1608-J -> my_rcl:1608
- R9: value 22 -> 10k; device my_rcl:1608-J -> my_rcl:1608
- TP2: value AIN+ -> IN+
- TP6: value AIN- -> IN-
- moved TP8 80.9 mm to (15.2, 6.99)
- moved TP4 76.2 mm to (15.2, 23.5)
- moved R9 75.9 mm to (6.67, 68.6), flipped to the bottom, turned to 0 degrees
- moved R18 72.2 mm to (6.67, 76.2), flipped to the bottom
- moved R16 66.0 mm to (6.67, 71.1), flipped to the bottom
- moved R5 63.7 mm to (18.1, 9.53), turned to 90 degrees
- moved R17 60.8 mm to (6.67, 73.7), flipped to the bottom
- moved R6 59.9 mm to (18.1, 21.0), turned to 90 degrees
- moved C30 56.1 mm to (61.0, 71.1), turned to 270 degrees
- moved IC6 55.9 mm to (57.1, 71.1), flipped to the bottom, turned to 270 degrees
- moved C24 43.9 mm to (53.3, 71.1), turned to 270 degrees
- moved TP5 41.0 mm to (41.9, 40.6)
- moved TP7 36.2 mm to (43.8, 20.6)
- moved C7 35.8 mm to (69.5, 20.3), turned to 180 degrees
- moved C22 35.2 mm to (67.6, 4.45), flipped to the top, turned to 90 degrees
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Connections:
- net N$15 renamed ADC_DVIO
- removed net +3V3A: C48.1, C54.1, C58.1, FB6.1, IC12.5, IC13.8, IC14.6, IC14.7, IC14.8
- removed net -9V: C36.-, IC8.3, J6.3, J7.3, J8.3, J9.3, R37.2
- removed net CLK_8MHZ: R46.2, X1.3, X1.3-2
- removed net N$31: IC13.2, R43.2
- removed net N$35: C12.1, R22.2, R27.1, R28.1
- removed net N$36: C11.1, R21.2, R25.1, R26.1
- removed net N$37: C7.2, IC3.4, R18.2, R20.1
- removed net N$38: C6.2, IC3.5, R17.2, R19.1
- removed net N$39: C7.1, IC3.1, R16.2, R18.1
- removed net N$40: C6.1, IC3.8, R15.2, R17.1
- removed net N$47: IC5.2, J5.2
- removed net N$48: C62.1, IC16.4
- removed net N$49: IC3.2, J3.2
- removed net N$50: C27.2, IC5.6, J8.2
- removed net N$51: C22.2, IC3.6, J7.2
- removed net N$52: C18.2, IC2.4, J6.2
- removed net N$54: C33.2, IC8.1, R34.1, R37.1
- removed net N$56: C57.1, IC12.4
- removed net N$59: C59.1, IC15.4
- removed net N$74: C31.2, IC6.6, J9.2
- new net +2V5: C28.1, C29.1, C58.1, FB6.1, IC12.5, IC14.6, IC14.7, IC14.8, IC17.16
- new net +3V3D: C6.1, C7.1, IC1.109, IC1.110, IC1.111, IC1.112, IC1.59, IC1.60, IC17.1, R16.2, R17.2, R18.2, R9.2
- new net ADC_LED1: IC17.12, R47.2
- new net ADC_VREF: C31.1, C46.1, C47.1, FB5.2, IC11.1
- new net CLK_OSC: IC14.1, R15.1
- new net DGND: C24.2, C30.2, C6.2, C7.2, IC1.1, IC1.101, IC1.102, IC1.103, IC1.104, IC1.113, IC1.114, IC1.115, IC1.116, IC1.2, IC1.39, IC1.40, IC1.53, IC1.54, IC1.57, IC1.58, IC1.61, IC1.62, IC1.83, IC1.84, IC17.8, IC6.2, IC6.3, J4.1, R21.2, R7.1, SW1.5, SW1.6, SW1.7, SW1.8, TP22.1, TP23.1, TP24.1
- new net DIP_SW1: IC1.86, R9.1, SW1.1
- new net DIP_SW2: IC1.88, R16.1, SW1.2
- new net DIP_SW3: IC1.90, R17.1, SW1.3
- new net DIP_SW4: IC1.92, R18.1, SW1.4
- new net FPGA_CNVST: IC1.52, R29.2
- new net FPGA_CNVST_FB: IC1.42, R46.2
- new net FPGA_LED1: IC1.46, R32.2
- new net FPGA_SCK: IC1.50, R30.2
- new net FPGA_SDI: IC1.48, R31.2
- new net FPGA_SDO: IC1.44, R45.2
- new net VIN_LIM: C24.1, FB1.1, IC6.6
- net +1V8: now also IC13.5; no longer IC15.5
- net +5V: now also FB7.1, IC13.1, IC13.3, R8.2; no longer C61.1, IC15.1, IC15.3, IC16.1, IC16.3, R47.2
- net +9V: now also TP21.1; no longer C21.1, C30.1, IC3.3, IC3.7, IC6.3, IC6.7
- net -5V: now also C18.2, C27.2, IC2.4, IC5.6, TP20.1; no longer J6.1, J7.1, J8.1, J9.1
- net ADC+: now also TP13.1
- net ADC-: now also TP14.1
- net ADC_CNVST: now also IC17.15; no longer R9.2
- net ADC_CNVST_CLOCKED: now also R12.5; no longer R42.2
- net ADC_CNVST_FB: now also IC14.3, IC17.10; no longer R45.2, R8.2
- net ADC_SCK: now also IC17.14, R12.7; no longer IC13.6, R6.2
- net ADC_SDI: now also IC17.13, R12.8; no longer IC13.1, R5.2
- net ADC_SDO: now also IC17.11, R12.6; no longer IC13.5, R7.2
- net ADC_VCOM: now also IC5.2; no longer IC6.2, J3.3, J5.3
- net GND: now also C22.2, C28.2, C29.2, C31.2, C4.2, C9.1, D2.K, IC10.HT2, IC13.2, IC17.9, IC3.2, R21.1, TP15.1, TP16.1, TP17.1, TP18.1, TP19.1; no longer C22.1, C24.1, C30.2, C31.1, C33.1, C36.+, C38.2, C48.2, C51.2, C54.2, C57.2, C59.2, C61.2, C62.2, C8.2, C9.2, IC1.1, IC1.101, IC1.102, IC1.103, IC1.104, IC1.113, IC1.114, IC1.115, IC1.116, IC1.2, IC1.39, IC1.40, IC1.53, IC1.54, IC1.57, IC1.58, IC1.61, IC1.62, IC1.83, IC1.84, IC13.4, IC15.2, IC16.2, J3.1, J4.1, J5.1, R34.2
- net N$1: now also J5.2, R20.1; no longer IC2.6, R11.2, R12.1, R14.1
- net N$10: now also C12.1, IC2.6, R11.2, R14.1; no longer IC1.46, R6.1
- net N$11: now also IC17.5, R32.1; no longer IC14.3, R45.1
- net N$12: now also C9.2, R6.2; no longer IC2.7, R14.2, R16.1
- net N$13: now also IC17.4, R31.1; no longer IC13.7, R41.2
- net N$14: now also J3.3, R6.1; no longer C4.1, R3.1
- net N$16: now also C21.1, C22.1, FB7.2, IC3.1, IC3.3; no longer C46.1, C47.1, FB5.2, IC11.1
- net N$17: now also C8.1, R19.2, R25.1, R26.1; no longer IC1.48, R7.1
- net N$18: now also IC17.3, R30.1; no longer IC14.1, R46.1
- net N$19: now also IC17.2, R29.1; no longer C29.1, IC6.1, R30.2, R32.1
- net N$2: now also IC17.7, R46.1; no longer C29.2, IC6.4, J12.1, R32.2
- net N$20: now also R15.2, X1.3, X1.3-2; no longer IC13.3, R44.2
- net N$21: now also C12.2, IC2.7, J5.3, R14.2; no longer IC1.52, R9.1
- net N$22: now also C8.2, R20.2, R27.1, R28.1; no longer C28.1, IC6.8, R29.2, R31.1
- net N$23: now also J5.1, R5.2; no longer C4.2, R4.2
- net N$24: now also IC6.5, R7.2; no longer C8.1, R19.2, R21.1
- net N$25: now also R12.3; no longer R44.1
- net N$26: now also D2.A, R8.1; no longer C9.1, R20.2, R22.1
- net N$28: now also R12.2; no longer R43.1
- net N$29: now also R12.4; no longer R42.1
- net N$3: now also C11.1; no longer R12.2
- net N$30: now also R12.1; no longer R41.1
- net N$32: now also J10.1; no longer C12.2, R29.1
- net N$33: now also J12.1; no longer C11.2, R30.1
- net N$4: now also C11.2, J3.1; no longer R15.1
- net N$43: now also R3.1
- net N$44: now also R4.2
- net N$5: now also IC17.6, R45.1; no longer C28.2, IC6.5, J10.1, R31.2
- net N$6: now also J3.2, R19.1; no longer IC1.50, R8.1
- net N$8: no longer C51.1
- net N$9: now also C4.1; no longer IC1.44
- net V+: no longer C38.1
- net V-: no longer C24.2, IC8.2
- net VCC_OSC: now also IC3.5; no longer IC16.5
- net VIN: now also C30.1, IC6.1; no longer FB1.1
Routing:
- net +3V3D: track 0.00 -> 165.4 mm, vias 0 -> 1
- net -9V: track 74.9 -> 0.00 mm, vias 3 -> 0
- net VIN: track 84.3 -> 28.5 mm
- net DIP_SW1: track 0.00 -> 53.0 mm, vias 0 -> 1
- net DIP_SW2: track 0.00 -> 52.5 mm, vias 0 -> 1
- net DIP_SW3: track 0.00 -> 52.0 mm, vias 0 -> 1
- net DIP_SW4: track 0.00 -> 51.6 mm, vias 0 -> 1
- net VIN_LIM: track 0.00 -> 49.4 mm
- net ADC_VCOM: track 73.4 -> 25.2 mm
- net +3V3A: track 38.0 -> 0.00 mm, vias 3 -> 0
- net +2V5: track 0.00 -> 36.9 mm, vias 0 -> 3
- net +9V: track 117.3 -> 84.5 mm, vias 7 -> 3
- net FPGA_CNVST: track 0.00 -> 30.7 mm
- net FPGA_SDI: track 0.00 -> 30.2 mm
- net FPGA_SDO: track 0.00 -> 29.7 mm
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- added copper zone on layer 1, net ADC_DVIO
- added copper zone on layer 1, net ADC_VREF
- added copper zone on layer 1, net DGND
- added copper zone on layer 15, net DGND
- added copper zone on layer 16, net DGND
- added copper zone on layer 2, net DGND
- removed copper zone on layer 1, net +5V
- removed copper zone on layer 1, net N$16
- removed copper zone on layer 1, net VREF
Other:
- board size 99.1 x 88.9 mm -> 88.9 x 88.9 mm
- board text added: "ver3.2"
- board text removed: "ver3"
