File: ADC2.brd (EAGLE design)
At the start: 90 x 99 mm, 192 parts, among them CON1 USB-A, CON2 SWD_CON, IC1 STM32G431, IC10 NJM11100, IC11 TAR5SB33, IC12 LM4562, IC13 LM4562, IC14 NJM12888F18, IC15 AZ1117-3.3, IC16 -9V, IC17 +9V, IC18 LM4562, IC19 TC7WH74FU, IC2 7404, IC20 NJM2845-33, IC21 -5V, IC3 ESP32-WROVER, IC4 LME49721, IC5 TL431, IC6 AD4001, IC7 OCT_BUFFER-SO6, IC8 OCT_BUFFER-SO6, IC9 TAR5SB33, J2 SJ-1608, J4 SJ-1608, J5 SJ-2012, J6 IN1_DC, J7 SJ-1608, J8 short, J9 SJ-2012, SW1 Gain, X1 12MHz

Commit message: ver2修正
Parts:
- removed C46, C47: 10u, my_rcl:3216
- removed C48, C49, C50, C52, C53, C57, C59: 0.1u, my_rcl:1608
- removed C51, R52: DNP, my_rcl:2012
- removed C54, C55: 100u, my_rcl:E2,5-8
- removed C56, C58: 10u, my_rcl:2012
- removed CON1: USB-A, my_connector:UX60A-MB-5ST
- removed CON2: SWD_CON, my_connector:SWD_CON
- removed D3: ERR, my_rcl:D1608
- removed D4, D5: CLAMP, my_rcl:SOD123
- removed F1: 0.5A, my_rcl:3216
- removed IC10: NJM11100, my_ic:SOT23-6
- removed IC12, IC18: LM4562, my_ic:DIL8-SOP8
- removed IC16: -9V, my_ic:TO-92
- removed IC17: +9V, my_ic:TO-92
- removed IC19: TC7WH74FU, my_ic:SSOP8-P-0.65
- removed IC20: NJM2845-33, my_ic:P-HSIP3_2.30A
- removed IC21: -5V, my_ic:TO-92
- removed R22, R23, R35, R36, R39, R42, R43, R48, R49, R50: 1k, my_rcl:1608
- removed R24, R27, R28, R29: 37, my_rcl:1608-J
- removed R30, R44, R45: 22, my_rcl:1608
- removed R40, R46, R51: 10k, my_rcl:1608
- removed R41: 100k, my_rcl:1608
- removed R47: 1.5k, my_rcl:1608
- removed TP10: ESP_EN, my_connector:TESTPIN
- removed TP11: ESP_BOOT, my_connector:TESTPIN
- removed TP12: ESP_TX, my_connector:TESTPIN
- removed TP13, TP20, TP27, TP28, TP29: GND, my_connector:TESTPIN
- removed TP14: ESP_RX, my_connector:TESTPIN
- removed TP24: VDD_OSC, my_connector:TESTPIN
- removed TP25: OSC_EN, my_connector:TESTPIN
- removed TP26: OSC_OUT, my_connector:TESTPIN
- removed TP6: UART_RX, my_connector:TESTPIN
- removed TP7: UART_GND, my_connector:TESTPIN
- removed TP8: UART_TX, my_connector:TESTPIN
- removed TP9: +3V3D, my_connector:TESTPIN
- removed X1: 12MHz, my_rcl:HC49/S
- added U$9: FPGA_CORE_BOARD, my_ic:FPGA_CORE_BOARD
- C12: value 3300p -> 470p
- C13: value 10u -> 0.1u; device my_rcl:2012 -> my_rcl:1608
- C14, C24: value 470p -> 100p
- C15: value DNP -> 10u; device my_rcl:1608 -> my_rcl:2012
- C16: value 0.1u -> 10u; device my_rcl:1608 -> my_rcl:3216
- C17: device my_rcl:2012 -> my_rcl:3216
- C18, C33: value 10u -> 470p; device my_rcl:2012 -> my_rcl:1608
- C19, C22: value 100p -> 0.1u
- C20: value 10u -> 1u; device my_rcl:C050 -> my_rcl:1608
- C21, C30, C41: value 0.1u -> 10u; device my_rcl:1608 -> my_rcl:2012
- C23: value 470p -> DNP
- C25: value 470p -> 10u; device my_rcl:1608 -> my_rcl:3216
- C28: value 1u -> 10u; device my_rcl:1608 -> my_rcl:2012
- C29: value 100u -> 0.1u; device my_rcl:E2.5-6.5 -> my_rcl:1608
- C3: value 0.01u -> 0.1u
- C32: value 0.1u -> 470p
- C35: value 10u -> 3300p; device my_rcl:3216 -> my_rcl:1608
- C38, C42: value 0.1u -> 1u
- C4: value 22p -> 0.1u
- C44: value 0.1u -> DNP
- C45: value 10u -> 1u; device my_rcl:3216 -> my_rcl:1608
- C5: value 22p -> 10u; device my_rcl:1608 -> my_rcl:C050
- C8: value 0.1u -> 100u; device my_rcl:1608 -> my_rcl:E2,5-8
- C9: value DNP -> 100u; device my_rcl:1608 -> my_rcl:E2,5-8
- D1: value PWR -> CLAMP; device my_rcl:D1608 -> my_rcl:SOD123
- D2: value OK -> CLAMP; device my_rcl:D1608 -> my_rcl:SOD123
- FB2, FB3, FB4: value FB -> FB-2012; device my_rcl:1608-J -> my_rcl:2012-J
- FB5, FB6: value FB-2012 -> FB; device my_rcl:2012-J -> my_rcl:1608-J
- IC1: value STM32G431 -> +9V; device my_ic:TQFP32-08 -> my_ic:TO-92
- IC11: value TAR5SB33 -> AD4001; device my_ic:SOT23-5 -> my_ic:MSOP10
- IC13: value LM4562 -> 7404; device my_ic:DIL8-SOP8 -> my_ic:TSSOP14
- IC14: value NJM12888F18 -> TC7WH74FU; device my_ic:SOT23-5 -> my_ic:SSOP8-P-0.65
- IC15: value AZ1117-3.3 -> OSC; device my_ic:SOT223 -> my_ic:MY_OSC
- IC2: value 7404 -> -9V; device my_ic:TSSOP14 -> my_ic:TO-92
- IC3: value ESP32-WROVER -> -5V; device my_ic:ESP32-WROVER -> my_ic:TO-92
- IC4: value LME49721 -> LM4562
- IC5: value TL431 -> AK1110; device my_ic:TO-92 -> my_ic:PLP10
- IC6: value AD4001 -> LM4562; device my_ic:MSOP10 -> my_ic:DIL8-SOP8
- IC7: value OCT_BUFFER-SO6 -> LM4562; device my_ic:SO6 -> my_ic:DIL8-SOP8
- IC8: value OCT_BUFFER-SO6 -> TAR5SB33; device my_ic:SO6 -> my_ic:SOT23-5
- IC9: value TAR5SB33 -> NJM12888F18
- J1: value (none) -> IN1_DC
- J2: value SJ-1608 -> SJ-2012; device my_rcl:1608-J -> my_rcl:2012-J
- J3: value (none) -> SJ-2012
- J4: value SJ-1608 -> short; device my_rcl:1608-J -> my_rcl:2012-J
- J6: value IN1_DC -> SJ-2012
- J8: value short -> SJ-1608; device my_rcl:2012-J -> my_rcl:1608-J
- J9: value SJ-2012 -> SJ-1608; device my_rcl:2012-J -> my_rcl:1608-J
- R1: value 10k -> 10; device my_rcl:1608 -> my_rcl:1608-J
- R10, R11, R13, R8: value 37 -> 1k; device my_rcl:1608-J -> my_rcl:1608
- R15: value 10k -> 1k
- R17, R18, R19: value 1.5k -> 1k
- R2: value 37 -> 100k; device my_rcl:1608-J -> my_rcl:1608
- R20: value 10 -> 1k; device my_rcl:1608-J -> my_rcl:1608
- R21: value short -> 1k; device my_rcl:1608-J -> my_rcl:1608
- R25: value 37 -> 22; device my_rcl:1608-J -> my_rcl:1608
- R26: value 1k -> 22
- R3, R4, R5, R6, R7: value 37 -> 22
- R31: value 22 -> 37; device my_rcl:1608 -> my_rcl:1608-J
- R32, R33, R34, R37, R38: value 1k -> 37; device my_rcl:1608 -> my_rcl:1608-J
- TP4: value VBUS -> GND
- TP5: value UART_3V3 -> GND
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Connections:
- removed net +3V3: C1.2, C18.1, C2.1, C3.1, C38.1, D1.A, IC1.1, IC1.15, IC1.17, IC7.6, IC8.1, IC9.5
- removed net +3V3D: C35.1, IC15.2, IC15.4, IC20.3, IC3.2, R1.2, R9.2, TP9.1
- removed net +5.3V: C34.1, C57.1, IC10.4, IC4.1-8, IC4.2-8, R46.2, R49.1, R51.2
- removed net +5VD: C45.1, FB4.1, FB6.2, IC9.1, IC9.3
- removed net ADC1+: J4.2, R44.1
- removed net ADC1-: J2.2, J7.2, R45.1
- removed net ESP_BOOT: IC3.25, R1.1, TP11.1
- removed net ESP_EN: C8.1, IC3.3, R9.1, TP10.1
- removed net ESP_RX: IC3.34, TP14.1
- removed net ESP_TX: IC3.35, TP12.1
- removed net N$23: C15.1, IC4.1-7, IC4.2-7, R21.1
- removed net N$27: D1.K, R17.2
- removed net N$32: CON1.2, R30.1
- removed net N$33: CON1.3, R31.1
- removed net N$34: IC8.3, R33.2
- removed net N$35: IC7.3, R38.2, R48.2
- removed net N$36: IC1.10, R27.2
- removed net N$37: IC1.11, R28.2
- removed net N$39: IC13.1-6, IC13.2-6, R15.1, R16.2, SW1.3
- removed net N$40: D2.K, R18.2
- removed net N$46: D3.K, R19.2
- removed net N$50: D3.A, IC1.8
- removed net N$51: C16.1, IC9.4
- removed net N$52: C24.2, IC6.3, R44.2
- removed net N$53: C23.1, IC6.4, R45.2
- removed net N$54: D2.A, IC1.7
- removed net N$58: C15.2, IC4.1-6, IC4.2-6, R22.1, R50.2
- removed net N$60: IC5.1, IC5.3, R40.1, R49.2
- removed net N$61: C36.1, IC10.3
- removed net N$62: IC10.5, R46.1, R47.2, R51.1
- removed net N$63: C28.1, C29.+, IC4.1-3, IC4.1-5, IC4.2-3, IC4.2-5, R40.2
- removed net N$64: IC4.1-1, IC4.1-2, IC4.2-1, IC4.2-2
- removed net N$65: F1.2, TP4.1
- removed net N$66: C44.1, IC1.4
- removed net N$69: C43.1, FB4.2, IC15.3, IC20.1
- removed net N$72: FB6.1, TP1.1
- removed net N$73: C51.2, R52.2
- removed net SPI_CS: IC3.29, R8.2
- removed net SPI_MISO: IC3.31, R6.2
- removed net SPI_MOSI: IC3.37, R5.2
- removed net SPI_SCK: IC3.30, R7.2
- removed net STM_RX: IC1.20, IC7.5
- removed net STM_TX: CON2.5, IC1.19, R33.1
- removed net SWCLK: CON2.1, IC1.24
- removed net SWDIO: CON2.4, IC1.23
- removed net UART_3V3: C37.1, IC7.1, IC8.6, R48.1, TP5.1
- removed net UART_GND: C37.2, IC8.4, TP7.1
- removed net UART_RX: R38.1, TP6.1
- removed net UART_TX: IC8.5, TP8.1
- removed net USB_DM: IC1.21, R30.2
- removed net USB_DP: IC1.22, R31.2
- removed net VBUS: CON1.1, F1.1
- new net +5V: C26.1, C42.1, C43.1, IC5.5, IC8.1, IC8.3, IC9.1, IC9.3
- new net ADC+: J9.2, R25.1
- new net ADC+_LPF: C32.2, IC11.3, R25.2
- new net ADC-: J7.2, J8.2, R26.1
- new net ADC-_LPF: C33.1, IC11.4, R26.2
- new net VIN: FB1.1, U$9.117, U$9.118, U$9.119, U$9.120
- net +1V8: now also C30.1, C37.1, IC11.2, IC9.5; no longer C11.1, C33.1, IC14.5, IC6.2
- net +3V3A: now also C28.1, C36.1, C40.1, FB6.1, IC13.14, IC14.6, IC14.7, IC14.8, IC8.5; no longer C10.1, C21.1, C31.1, FB2.1, IC11.5, IC19.6, IC19.7, IC19.8, IC2.14
- net +9V: now also C1.1, C16.1, C3.1, C6.1, D1.2, IC1.1, IC4.1-8, IC4.2-8, IC6.1-8, IC6.2-8, IC7.1-8, IC7.2-8; no longer C41.1, C46.1, C48.1, C7.1, D4.2, IC12.1-8, IC12.2-8, IC13.1-8, IC13.2-8, IC17.1, IC18.1-8, IC18.2-8
- net -5V: now also C15.2, IC3.3, J3.1; no longer C58.2, IC21.3, J9.1
- net -9V: now also C17.2, C2.2, C4.2, D2.1, IC2.3, IC4.1-4, IC4.2-4, IC6.1-4, IC6.2-4, J2.1; no longer C42.2, C47.2, C49.2, D5.1, IC12.1-4, IC12.2-4, IC13.1-4, IC13.2-4, IC16.3, J5.1
- net ADC_CNVST: now also IC14.2, R3.2; no longer IC19.2, R29.1
- net ADC_CNVST_CLOCKED: now also IC14.5, R32.2; no longer IC19.5, R13.2
- net ADC_CNVST_FB: now also IC13.8, R4.2; no longer IC2.8, R11.1
- net ADC_SCK: now also IC13.3, R6.2; no longer IC2.3, R27.1
- net ADC_SDI: now also IC13.1, R7.2; no longer IC2.1, R4.1
- net ADC_SDO: now also IC13.6, R5.2; no longer IC2.6, R28.1
- net CLK_8MHZ: now also IC15.5, R38.2; no longer R3.2, TP26.1
- net GND: now also C1.2, C11.1, C13.1, C15.1, C17.1, C19.2, C2.1, C20.2, C22.2, C29.2, C32.1, C37.2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; no longer C1.1, C11.2, C13.2, C14.2, C17.2, C2.2, C23.2, C24.1, C29.-, C32.2, C4.2, C42.1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
- net N$1: now also R8.1, R9.1, SW1.3; no longer C5.1, IC1.2, X1.2
- net N$10: now also R6.1, U$9.46; no longer IC1.12, R4.2
- net N$11: now also IC14.3, R37.1; no longer IC19.3, R10.1
- net N$12: now also C5.2, J1.2, R1.1; no longer C20.2, J6.2, R20.1
- net N$13: now also IC13.2, R31.2; no longer IC2.2, R2.2
- net N$14: now also C23.1, IC6.1-7, IC6.2-7, IC7.1-5, IC7.2-5, J5.2, R19.2; no longer C9.1, IC12.1-7, IC12.2-7, IC18.1-5, IC18.2-5, J1.2, R12.2
- net N$15: now also C39.1, C41.1, FB6.2, IC11.10; no longer C56.1, C6.1, FB2.2, IC6.10
- net N$16: now also C34.1, C35.1, FB5.2, IC11.1; no longer C12.1, C13.1, FB3.2, IC6.1
- net N$17: now also R5.1, U$9.48; no longer IC1.25, R8.1
- net N$18: now also IC14.1, R38.1; no longer IC19.1, R3.1
- net N$19: now also IC13.9, R37.2; no longer IC2.9, R10.2
- net N$2: now also IC7.1-6, IC7.1-7, IC7.2-6, IC7.2-7, J5.1, J7.1; no longer IC18.1-6, IC18.1-7, IC18.2-6, IC18.2-7, J1.1, J2.1
- net N$20: now also IC13.5, R34.2; no longer IC2.5, R25.2
- net N$21: now also R3.1, U$9.52; no longer IC1.9, R11.2
- net N$22: now also IC13.11, IC13.12; no longer IC2.11, IC2.12
- net N$24: now also J4.2, R15.1; no longer J8.2, R35.1
- net N$25: now also IC11.7, R34.1; no longer IC6.7, R25.1
- net N$26: now also C24.2, IC6.1-2, IC6.2-2, R18.2; no longer C19.2, IC12.1-2, IC12.2-2, R14.2
- net N$28: now also IC11.8, R33.1; no longer IC6.8, R24.1
- net N$29: now also IC11.6, R32.1; no longer IC6.6, R13.1
- net N$3: now also IC4.1-6, IC4.2-6, SW1.2; no longer C4.1, IC1.3, X1.1
- net N$30: now also IC11.9, R31.1; no longer IC6.9, R2.1
- net N$31: now also IC13.4, R33.2; no longer IC2.4, R24.2
- net N$38: now also R13.1, R14.2; no longer R36.1, R37.2
- net N$4: now also C12.1, R10.2, R11.1, R12.1; no longer C25.1, R39.1, R42.2, R43.1
- net N$41: now also C22.1, IC6.1-5, IC6.2-5, R14.1, R16.1; no longer C27.1, IC12.1-5, IC12.2-5, R23.1, R37.1
- net N$42: now also C23.2, IC6.1-6, IC6.2-6, R19.1, R20.2; no longer C9.2, IC12.1-6, IC12.2-6, R12.1, R32.2
- net N$43: now also C18.1, R15.2, R18.1, R21.1; no longer C14.1, R14.1, R34.1, R35.2
- net N$44: now also C19.1, IC6.1-3, IC6.2-3, R16.2, R17.2; no longer C30.1, IC12.1-3, IC12.2-3, R23.2, R26.2
- net N$45: now also IC4.1-7, IC4.2-7, R10.1, R9.2; no longer IC13.1-7, IC13.2-7, R15.2, R42.1, SW1.2
- net N$47: now also C24.1, IC6.1-1, IC6.2-1, IC7.1-3, IC7.2-3, J6.2, R20.1, R21.2; no longer C19.1, IC12.1-1, IC12.2-1, IC18.1-3, IC18.2-3, J3.2, R32.1, R34.2
- net N$48: now also C5.1, J1.1; no longer C20.1, J6.1
- net N$49: now also D1.1, D2.2, IC4.1-5, IC4.2-5, R1.2, R2.2; no longer D4.1, D5.2, IC13.1-5, IC13.2-5, R20.2, R41.2
- net N$5: now also IC7.1-1, IC7.1-2, IC7.2-1, IC7.2-2, J6.1, J9.1; no longer IC18.1-1, IC18.1-2, IC18.2-1, IC18.2-2, J3.1, J4.1
- net N$55: now also C14.2, IC4.1-2, IC4.2-2, R12.2; no longer C22.2, IC13.1-2, IC13.2-2, R39.2
- net N$56: now also C27.1, IC8.4; no longer C26.1, IC11.4
- net N$57: now also C14.1, IC4.1-1, IC4.2-1, J4.1, R11.2; no longer C22.1, IC13.1-1, IC13.2-1, J8.1, R43.2
- net N$59: now also C29.1, IC9.4; no longer C32.1, IC14.4
- net N$6: now also R4.1, U$9.50; no longer IC1.26, R7.1
- net N$7: now also C31.1, IC5.7; no longer IC1.27, R6.1
- net N$70: now also FB3.1; no longer FB1.1
- net N$71: now also FB4.1; no longer FB5.1
- net N$74: now also C7.2, IC7.1-4, IC7.2-4, J2.2, J3.2; no longer C50.2, IC18.1-4, IC18.2-4, J5.2, J9.2
- net N$75: now also FB1.2
- net N$76: now also FB2.2
- net N$8: now also C25.1, C44.1, IC5.9; no longer IC1.28, R5.1
- net N$9: now also R7.1, U$9.44; no longer IC1.13, R29.2
- net V+: now also C10.1, C38.1, C45.1, C8.+, FB3.2, IC1.3, IC15.2, IC15.3, IC5.2, IC5.3, IC5.4; no longer C39.1, C40.1, C52.1, C54.+, FB1.2, IC10.1, IC10.6, IC11.1, IC11.3, IC14.1, IC14.3, IC17.3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
- net V-: now also C11.2, C13.2, C9.-, FB4.2, IC2.2, IC3.2; no longer C53.2, C55.-, C59.2, FB5.2, IC16.2, IC21.2
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Routing:
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- removed copper zone on layer 1, net +3V3D
- removed copper zone on layer 15, net N$67
- removed copper zone on layer 2, net N$68
- removed copper zone on layer 1, net UART_GND
- removed copper zone on layer 16, net UART_GND
Other:
- board size 90 x 99 mm -> 86.4 x 99.1 mm
- board text added: "ver2"
- board text removed: "ver1"

Commit message: update
Parts:
- removed D2: CLAMP, my_rcl:SOD123
- removed SW1: Gain, my_connector:1X03
- removed TP15: -D5V, my_connector:TESTPIN
- removed TP16: GND, my_connector:TESTPIN-BIG
- removed TP17: V+, my_connector:TESTPIN
- removed TP18: GND, my_connector:TESTPIN
- removed TP19: V-, my_connector:TESTPIN
- removed TP21: VIN+, my_connector:TESTPIN
- removed TP22: VIN-, my_connector:TESTPIN
- removed TP23: (no value), my_connector:TESTPIN
- removed U$9: FPGA_CORE_BOARD, my_ic:FPGA_CORE_BOARD
- added C46, C52, C55, C58, C60, C64: 10u, my_rcl:2012
- added C47: 3300p, my_rcl:1608C
- added C48, C49, C53, C54, C56, C57, C59, C61, C62, C63: 0.1u, my_rcl:1608C
- added C50: 10u, my_rcl:3216
- added C51: DNP, my_rcl:1608C
- added IC10: AK1110, my_ic:PLP10
- added IC12, IC16: TAR5SB33, my_ic:SOT23-5
- added J10: ADC+, my_rcl:1608-J
- added J11: GND, my_rcl:1608-J
- added J12: ADC-, my_rcl:1608-J
- added JP1: GAIN, my_connector:1X02
- added R22, R23, R24, R27, R29, R30: 1k, my_rcl:1608
- added R28: 3.6k, my_rcl:1608
- added R35: 330, my_rcl:1608
- added R36: 120, my_rcl:1608
- added R39, R40: 22, my_rcl:1608
- added R41, R42, R43, R44: 37, my_rcl:1608
- added R45, R46: 37, my_rcl:1608-J
- added R47: 5.1k, my_rcl:1608
- added TP10, TP11, TP12, TP7, TP8, TP9: GND, my_connector:TESTPIN
- added TP6: AIN-, my_connector:TESTPIN-MID
- added X1: 12MHz, my_rcl:KC7050
- C1, C2: value 0.1u -> 1u; device my_rcl:1608 -> my_rcl:3225
- C10: value 0.1u -> 10u; device my_rcl:1608 -> my_rcl:2012
- C11: value 0.1u -> 1n; device my_rcl:1608 -> my_rcl:1608C
- C12: value 470p -> 1n; device my_rcl:1608 -> my_rcl:1608C
- C13: value 0.1u -> 1.5n; device my_rcl:1608 -> my_rcl:1608C
- C14: value 100p -> 1.5n; device my_rcl:1608 -> my_rcl:1608C
- C15, C41: value 10u -> 1u; device my_rcl:2012 -> my_rcl:1608C
- C16: value 10u -> 1u; device my_rcl:3216 -> my_rcl:1608C
- C17, C25: value 10u -> 0.1u; device my_rcl:3216 -> my_rcl:1608C
- C18: value 470p -> 0.1u; device my_rcl:1608 -> my_rcl:1608C
- C19: value 0.1u -> 100u; device my_rcl:1608 -> my_rcl:E2,5-8
- C20: value 1u -> 100u; device my_rcl:1608 -> my_rcl:E2,5-8
- C21, C30, C31: value 10u -> 0.1u; device my_rcl:2012 -> my_rcl:1608C
- C22, C26, C27, C38: device my_rcl:1608 -> my_rcl:1608C
- C23: value DNP -> 0.1u; device my_rcl:1608 -> my_rcl:1608C
- C24: value 100p -> 0.1u; device my_rcl:1608 -> my_rcl:1608C
- C28: value 10u -> 10p; device my_rcl:2012 -> my_rcl:1608C
- C29, C6, C7: value 0.1u -> 10p; device my_rcl:1608 -> my_rcl:1608C
- C3, C4: value 0.1u -> DNP; device my_rcl:1608 -> my_rcl:1608C
- C32, C33: value 470p -> 10u; device my_rcl:1608 -> my_rcl:3216
- C34, C43: device my_rcl:2012 -> my_rcl:3216
- C35: value 3300p -> 100u; device my_rcl:1608 -> my_rcl:E2.5-6.5
- C36, C37: value 0.1u -> 100u; device my_rcl:1608 -> my_rcl:E2.5-6.5
- C39, C40: value 0.1u -> 1u; device my_rcl:1608 -> my_rcl:1608C
- C42: value 1u -> 10u; device my_rcl:1608 -> my_rcl:2012
- C44: value DNP -> 470p; device my_rcl:1608 -> my_rcl:1608C
- C45: value 1u -> 470p; device my_rcl:1608 -> my_rcl:1608C
- C5: value 10u -> DNP; device my_rcl:C050 -> my_rcl:1608C
- C8, C9: value 100u -> 2.7n; device my_rcl:E2,5-8 -> my_rcl:1608C
- D1: value CLAMP -> PWR; device my_rcl:SOD123 -> my_rcl:D1608
- FB1, FB2, FB3, FB4: value FB-2012 -> FB
- IC1: value +9V -> FPGA CORE BOARD; device my_ic:TO-92 -> my_ic:FPGA_CORE_BOARD
- IC13: value 7404 -> 74HC3G34; device my_ic:TSSOP14 -> my_ic:SOT765
- IC15: value OSC -> NJM12888F18; device my_ic:MY_OSC -> my_ic:SOT23-5
- IC2: value -9V -> OPA; device my_ic:TO-92 -> my_ic:SOP8
- IC3: value -5V -> OPA-DIFF; device my_ic:TO-92 -> my_ic:SOP8
- IC4: value LM4562 -> DCDC2; device my_ic:DIL8-SOP8 -> my_ic:DCDC2
- IC5: value AK1110 -> OPA-DIFF; device my_ic:PLP10 -> my_ic:SOP8
- IC6: value LM4562 -> OPA-DIFF; device my_ic:DIL8-SOP8 -> my_ic:SOP8
- IC7: value LM4562 -> LM317-L; device my_ic:DIL8-SOP8 -> my_ic:TO-92
- IC8: value TAR5SB33 -> LM337-L; device my_ic:SOT23-5 -> my_ic:TO-92
- IC9: value NJM12888F18 -> LM337-L; device my_ic:SOT23-5 -> my_ic:TO-92
- J1: value IN1_DC -> DC; device my_rcl:2012-J -> my_rcl:1608-J
- J2: value SJ-2012 -> DC; device my_rcl:2012-J -> my_rcl:1608-J
- J3, J5: value SJ-2012 -> VCOM; device my_rcl:2012-J -> my_rcl:1608-3-J
- J4: value short -> GND
- J6: value SJ-2012 -> V-; device my_rcl:2012-J -> my_rcl:2012-3-J
- J7, J8, J9: value SJ-1608 -> V-; device my_rcl:1608-J -> my_rcl:2012-3-J
- R1: device my_rcl:1608-J -> my_rcl:2012
- R10, R11: value 1k -> 100
- R2: value 100k -> 10; device my_rcl:1608 -> my_rcl:2012
- R25: value 22 -> 3.6k
- R26: value 22 -> 1k
- R3, R4: value 22 -> 10k; device my_rcl:1608-J -> my_rcl:1608
- R31, R32: value 37 -> 1k; device my_rcl:1608-J -> my_rcl:1608
- R33, R34: value 37 -> 680; device my_rcl:1608-J -> my_rcl:1608
- R37, R38: value 37 -> 120; device my_rcl:1608-J -> my_rcl:1608
- R8: value 1k -> 22; device my_rcl:1608 -> my_rcl:1608-J
- R9: value 10k -> 22; device my_rcl:1608 -> my_rcl:1608-J
- TP1: value +D5V -> GND; device my_connector:TESTPIN -> my_connector:TESTPIN-MID
- TP2: value AIN1 -> AIN+; device my_connector:TESTPIN-BIG -> my_connector:TESTPIN-MID
- TP3: device my_connector:TESTPIN -> my_connector:TESTPIN-MID
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Connections:
- new net ADC_VCOM: C10.1, IC6.2, J3.3, J5.3, R23.1, R24.2
- new net N$23: C4.2, C5.1, IC2.5, R2.2, R4.2
- new net N$27: C13.1, IC5.8, R26.2
- new net N$32: C12.2, C13.2, IC5.5, R25.2, R29.1
- new net N$33: C11.2, C14.2, IC5.4, R28.2, R30.1
- new net N$34: C14.1, IC5.1, R27.2
- new net N$35: C12.1, R22.2, R27.1, R28.1
- new net N$36: C11.1, R21.2, R25.1, R26.1
- new net N$37: C7.2, IC3.4, R18.2, R20.1
- new net N$39: C7.1, IC3.1, R16.2, R18.1
- new net N$40: C6.1, IC3.8, R15.2, R17.1
- new net N$46: JP1.2, R11.1
- new net N$50: C27.2, IC5.6, J8.2
- new net N$51: C22.2, IC3.6, J7.2
- new net N$52: C18.2, IC2.4, J6.2
- new net N$53: C32.1, IC7.1, R33.2, R36.1
- new net N$54: C33.2, IC8.1, R34.1, R37.1
- new net N$58: D1.A, R47.1
- new net VCC_OSC: C63.1, C64.1, IC16.5, X1.1, X1.1-2, X1.4, X1.4-2
- net +1V8: now also C49.1, C60.1, IC15.5; no longer C30.1, C37.1, IC9.5
- net +3V3A: now also C48.1, C54.1, C58.1, IC12.5, IC13.8; no longer C28.1, C36.1, C40.1, IC13.14, IC8.5
- net +5V: now also C40.1, C56.1, C61.1, IC10.5, IC12.1, IC12.3, IC15.1, IC15.3, IC16.1, IC16.3, R47.2; no longer C26.1, C43.1, IC5.5, IC8.1, IC8.3, IC9.1, IC9.3
- net +9V: now also C17.1, C21.1, C26.1, C30.1, C35.+, IC2.8, IC3.3, IC3.7, IC5.3, IC5.7, IC6.3, IC6.7, IC7.2, R36.2; no longer C1.1, C16.1, C3.1, C6.1, D1.2, IC1.1, IC4.1-8, IC4.2-8, IC6.1-8, IC6.2-8, IC7.1-8, IC7.2-8
- net -5V: now also C37.-, IC9.3, J6.1, J7.1, J8.1, J9.1, R38.2; no longer C15.2, IC3.3, J3.1
- net -9V: now also C36.-, IC8.3, J6.3, J7.3, J8.3, J9.3, R37.2; no longer C17.2, C2.2, C4.2, D2.1, IC2.3, IC4.1-4, IC4.2-4, IC6.1-4, IC6.2-4, J2.1
- net ADC+: now also J10.2, R39.1; no longer J9.2, R25.1
- net ADC+_LPF: now also C44.2, R39.2; no longer C32.2, R25.2
- net ADC-: now also J11.2, J12.2, R40.1; no longer J7.2, J8.2, R26.1
- net ADC-_LPF: now also C45.1, R40.2; no longer C33.1, R26.2
- net ADC_CNVST: now also R9.2; no longer R3.2
- net ADC_CNVST_CLOCKED: now also R42.2; no longer R32.2
- net ADC_CNVST_FB: now also R45.2, R8.2; no longer IC13.8, R4.2
- net ADC_SCK: now also IC13.6; no longer IC13.3
- net ADC_SDI: now also R5.2; no longer R7.2
- net ADC_SDO: now also IC13.5, R7.2; no longer IC13.6, R5.2
- net CLK_8MHZ: now also R46.2, X1.3, X1.3-2; no longer IC15.5, R38.2
- net GND: now also C15.2, C16.1, C17.2, C18.1, C19.-, C20.+, C22.1, C23.2, C24.1, C25.1, C27.1, C3.1, C31.1, C32.2, C33.1, C34.1, C35.-, C36.+, C37.+, C44.1, C46.2, C47.2, C48.2, C49.2, C5.2, C50.2, C51.2, C52.2, C53.2, C54.2, C55.2, C56.2, C57.2, C58.2, C59.2, C60.2, C61.2, C62.2, C63.2, C64.2, C8.2, C9.2, D1.K, IC1.1, IC1.101, IC1.102, IC1.103, IC1.104, IC1.113, IC1.114, IC1.115, IC1.116, IC1.39, IC1.40, IC1.53, IC1.54, IC1.57, IC1.58, IC1.61, IC1.62, IC1.83, IC1.84, IC10.10, IC10.6, IC10.8, IC10.HT, IC12.2, IC13.4, IC15.2, IC16.2, IC4.GND1, J11.1, J3.1, J4.1, J5.1, R24.1, R3.2, R33.1, R34.2, R35.2, R4.1, TP1.1, TP10.1, TP11.1, TP12.1, TP7.1, TP8.1, TP9.1, X1.2, X1.2-2; no longer C1.2, C11.1, C12.2, C13.1, C15.1, C16.2, C17.1, C18.2, C19.2, C2.1, C20.2, C22.2, C25.2, C27.2, C28.2, C29.2, C3.2, C31.2, C32.1, C33.2, C34.2, C35.2, C36.2, C37.2, C4.1, C44.2, C6.2, C7.1, C8.-, C9.+, FB2.1, IC13.13, IC13.7, IC15.1, IC15.4, IC15.6, IC2.1, IC3.1, IC4.1-3, IC4.2-3, IC5.10, IC5.6, IC5.8, IC5.HT, IC8.2, IC9.2, J8.1, R17.1, R2.1, R8.2, TP16.1, TP18.1, U$9.1, U$9.101, U$9.102, U$9.103, U$9.104, U$9.113, U$9.114, U$9.115, U$9.116, U$9.2, U$9.39, U$9.40, U$9.53, U$9.54, U$9.57, U$9.58, U$9.61, U$9.62, U$9.83, U$9.84
- net N$1: now also IC2.6, R11.2, R12.1, R14.1; no longer R8.1, R9.1, SW1.3
- net N$10: now also IC1.46; no longer U$9.46
- net N$11: now also R45.1; no longer R37.1
- net N$12: now also IC2.7, R14.2, R16.1; no longer C5.2, J1.2, R1.1
- net N$13: now also IC13.7, R41.2; no longer IC13.2, R31.2
- net N$14: now also C3.2, C4.1, IC2.3, R1.2, R3.1; no longer C23.1, IC6.1-7, IC6.2-7, IC7.1-5, IC7.2-5, J5.2, R19.2
- net N$15: now also C53.1, C55.1; no longer C39.1, C41.1
- net N$16: now also C46.1, C47.1; no longer C34.1, C35.1
- net N$17: now also IC1.48, R7.1; no longer R5.1, U$9.48
- net N$18: now also R46.1; no longer R38.1
- net N$19: now also C29.1, IC6.1, R30.2, R32.1; no longer IC13.9, R37.2
- net N$2: now also C29.2, IC6.4, J12.1, R32.2; no longer IC7.1-6, IC7.1-7, IC7.2-6, IC7.2-7, J5.1, J7.1
- net N$20: now also IC13.3, R44.2; no longer IC13.5, R34.2
- net N$21: now also IC1.52, R9.1; no longer R3.1, U$9.52
- net N$22: now also C28.1, IC6.8, R29.2, R31.1; no longer IC13.11, IC13.12
- net N$24: now also C8.1, R19.2, R21.1; no longer J4.2, R15.1
- net N$25: now also R44.1; no longer R34.1
- net N$26: now also C9.1, R20.2, R22.1; no longer C24.2, IC6.1-2, IC6.2-2, R18.2
- net N$28: now also R43.1; no longer R33.1
- net N$29: now also R42.1; no longer R32.1
- net N$3: now also IC2.2, R10.2, R12.2, R13.1; no longer IC4.1-6, IC4.2-6, SW1.2
- net N$30: now also R41.1; no longer R31.1
- net N$31: now also IC13.2, R43.2; no longer IC13.4, R33.2
- net N$38: now also C6.2, IC3.5, R17.2, R19.1; no longer R13.1, R14.2
- net N$4: now also IC2.1, R13.2, R15.1; no longer C12.1, R10.2, R11.1, R12.1
- net N$41: now also C1.1, J1.1, TP2.1; no longer C22.1, IC6.1-5, IC6.2-5, R14.1, R16.1
- net N$42: now also C2.1, J2.1, TP6.1; no longer C23.2, IC6.1-6, IC6.2-6, R19.1, R20.2
- net N$43: now also C1.2, J1.2, R1.1; no longer C18.1, R15.2, R18.1, R21.1
- net N$44: now also C2.2, J2.2, R2.1; no longer C19.1, IC6.1-3, IC6.2-3, R16.2, R17.2
- net N$45: now also JP1.1; no longer IC4.1-7, IC4.2-7, R9.2, SW1.1
- net N$47: now also IC5.2, J5.2; no longer C24.1, IC6.1-1, IC6.2-1, IC7.1-3, IC7.2-3, J6.2, R20.1, R21.2
- net N$48: now also C62.1, IC16.4; no longer C5.1, J1.1, TP2.1
- net N$49: now also IC3.2, J3.2; no longer D1.1, D2.2, IC4.1-5, IC4.2-5, R1.2, R2.2
- net N$5: now also C28.2, IC6.5, J10.1, R31.2; no longer IC7.1-1, IC7.1-2, IC7.2-1, IC7.2-2, J6.1, J9.1
- net N$55: now also C34.2, IC9.1, R35.1, R38.1; no longer C14.2, IC4.1-2, IC4.2-2, R12.2
- net N$56: now also C57.1, IC12.4; no longer C27.1, IC8.4
- net N$57: now also FB2.1, J4.2; no longer C14.1, IC4.1-1, IC4.2-1, J4.1, R11.2
- net N$59: now also C59.1, IC15.4; no longer C29.1, IC9.4
- net N$6: now also IC1.50, R8.1; no longer R4.1, U$9.50
- net N$7: now also C52.1, IC10.7; no longer C31.1, IC5.7
- net N$70: now also IC4.V+; no longer TP17.1
- net N$71: now also IC4.V-; no longer TP19.1
- net N$74: now also C31.2, IC6.6, J9.2; no longer C7.2, IC7.1-4, IC7.2-4, J2.2, J3.2
- net N$75: now also IC4.VIN+; no longer TP21.1
- net N$76: now also IC4.VIN-; no longer TP22.1
- net N$8: now also C50.1, C51.1, IC10.9; no longer C25.1, C44.1, IC5.9
- net N$9: now also IC1.44, R5.1; no longer R7.1, U$9.44
- net V+: now also C15.1, C19.+, C23.1, C39.1, IC10.2, IC10.3, IC10.4, IC7.3; no longer C10.1, C45.1, C8.+, IC1.3, IC15.2, IC15.3, IC5.2, IC5.3, IC5.4
- net V-: now also C16.2, C20.-, C24.2, C25.2, IC8.2, IC9.2; no longer C11.2, C13.2, C9.-, IC2.2, IC3.2
- net VIN: now also IC1.117, IC1.118, IC1.119, IC1.120; no longer U$9.117, U$9.118, U$9.119, U$9.120
- net VREF: now also C41.1, C43.1, IC10.1, R23.2; no longer C20.1, C21.1, IC5.1, R13.2
Routing:
- net V+: track 171.7 -> 78.2 mm, vias 5 -> 2
- net ADC_VCOM: track 0.00 -> 73.4 mm, vias 0 -> 2
- net -5V: track 6.01 -> 73.5 mm, vias 0 -> 3
- net +5V: track 31.0 -> 81.1 mm, vias 0 -> 2
- net N$47: track 34.8 -> 4.50 mm, vias 0 -> 1
- net +9V: track 90.5 -> 117.3 mm, vias 1 -> 7
- net N$45: track 28.7 -> 2.75 mm
- net -9V: track 49.4 -> 74.9 mm, vias 1 -> 3
- net N$33: track 0.00 -> 23.4 mm, vias 0 -> 2
- net N$32: track 0.00 -> 22.3 mm, vias 0 -> 2
- net N$41: track 29.0 -> 7.73 mm, vias 1 -> 0
- net N$74: track 25.7 -> 5.48 mm, vias 0 -> 1
- net VCC_OSC: track 0.00 -> 16.4 mm
- net N$57: track 12.1 -> 28.4 mm
- net N$54: track 0.00 -> 14.8 mm
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- added copper zone on layer 1, net +5V
- added copper zone on layer 1, net VREF
Other:
- board size 86.4 x 99.1 mm -> 99.1 x 88.9 mm
- board text added: "ver3"
- board text removed: "ver2"

Commit message: AD4134
Parts:
- removed J10: ADC+, my_rcl:1608-J
- removed J11: GND, my_rcl:1608-J
- removed J12: ADC-, my_rcl:1608-J
- removed J5: VCOM, my_rcl:1608-3-J
- removed J6, J7, J8, J9: V-, my_rcl:2012-3-J
- removed JP1: GAIN, my_connector:1X02
- added C65, C66, C67, C68, C69, C70, C71: 0.1u, my_rcl:1608C
- added C72: 10u, my_rcl:1608C
- added D2: LED, my_rcl:D1608
- added FB7, FB8: FB, my_rcl:1608-FB
- added IC17: IOS6720FB, my_ic:SOP8
- added R48, R58: SDI, my_rcl:1608
- added R49, R59: LED, my_rcl:1608
- added R50: 10M, my_rcl:0204/7
- added R51: ODR, my_rcl:1608
- added R52: DOUT, my_rcl:1608
- added R53: SUB, my_rcl:1608
- added R54: DCLK, my_rcl:1608
- added R55: SDO, my_rcl:1608
- added R56: CS, my_rcl:1608
- added R57: SCLK, my_rcl:1608
- added R60: 10k, my_rcl:1608
- added SW1: DC, my_connector:SS22E01G5
- added SW2: GAIN, my_connector:1X03
- added TP13: GND, my_connector:TESTPIN
- added U1: DC-DC, my_ic:DCDC
- C1, C2: device my_rcl:3225 -> my_rcl:C050W
- C10: value 10u -> 1u; device my_rcl:2012 -> my_rcl:1608C
- C11, C12: value 1n -> 0.1u
- C13: value 1.5n -> 100u; device my_rcl:1608C -> my_rcl:E2.5-6.5
- C14: value 1.5n -> 100u; device my_rcl:1608C -> my_rcl:E2,5-8
- C15: value 1u -> 100u; device my_rcl:1608C -> my_rcl:E2,5-8
- C16: value 1u -> 1n
- C17: value 0.1u -> 1n
- C19, C20: value 100u -> 0.1u; device my_rcl:E2,5-8 -> my_rcl:1608C
- C23, C24: value 0.1u -> 270p
- C25, C26, C27: value 0.1u -> 10u; device my_rcl:1608C -> my_rcl:3216
- C28, C29: value 10p -> 100u; device my_rcl:1608C -> my_rcl:E2.5-6.5
- C30: value 0.1u -> 100u; device my_rcl:1608C -> my_rcl:E2.5-6.5
- C31, C62: value 0.1u -> 1u
- C32, C34: value 10u -> 1u; device my_rcl:3216 -> my_rcl:1608C
- C33, C50: device my_rcl:3216 -> my_rcl:2012
- C35, C36: value 100u -> 10u; device my_rcl:E2.5-6.5 -> my_rcl:2012
- C37: value 100u -> 10u; device my_rcl:E2.5-6.5 -> my_rcl:3216
- C38: value 1u -> 0.1u
- C39, C40, C41: value 1u -> 10u; device my_rcl:1608C -> my_rcl:2012
- C42, C46, C52, C58, C64: value 10u -> 0.1u; device my_rcl:2012 -> my_rcl:1608C
- C43: value 10u -> 0.1u; device my_rcl:3216 -> my_rcl:1608C
- C44: value 470p -> 10u; device my_rcl:1608C -> my_rcl:2012
- C45: value 470p -> 0.1u
- C47: value 3300p -> 0.1u
- C48, C49, C53, C59, C61: value 0.1u -> 10u; device my_rcl:1608C -> my_rcl:2012
- C51: value DNP -> 0.1u
- C6: value 10p -> 0.1u
- C63: value 0.1u -> 10u
- C7: value 10p -> 1u
- C8: value 2.7n -> 100u; device my_rcl:1608C -> my_rcl:E2,5-8
- C9: value 2.7n -> 1u
- FB5, FB6: device my_rcl:1608-J -> my_rcl:2012-J
- IC10: value AK1110 -> REF5040; device my_ic:PLP10 -> my_ic:SOP8
- IC11: value AD4001 -> 1.8V; device my_ic:MSOP10 -> my_ic:SOT23-5
- IC12: value TAR5SB33 -> 1.8V
- IC13: value 74HC3G34 -> 2.7V; device my_ic:SOT765 -> my_ic:SOT23-5
- IC14: value TC7WH74FU -> ISO6720FB; device my_ic:SSOP8-P-0.65 -> my_ic:SOP8
- IC15: value NJM12888F18 -> ISO6720FB; device my_ic:SOT23-5 -> my_ic:SOP8
- IC16: value TAR5SB33 -> IOS6720FB; device my_ic:SOT23-5 -> my_ic:SOP8
- IC3: value OPA-DIFF -> 7808; device my_ic:SOP8 -> my_ic:TO-92
- IC4: value DCDC2 -> LM317-L; device my_ic:DCDC2 -> my_ic:TO-92
- IC5, IC6: value OPA-DIFF -> LM337-L; device my_ic:SOP8 -> my_ic:TO-92
- IC7: value LM317-L -> OPA1633; device my_ic:TO-92 -> my_ic:SOP8
- IC8: value LM337-L -> AK1110; device my_ic:TO-92 -> my_ic:PLP10
- IC9: value LM337-L -> AD4134; device my_ic:TO-92 -> my_ic:QFN56-HT-HOLE
- J1, J2: value DC -> V-; device my_rcl:1608-J -> my_rcl:2012-3-J
- J3: value VCOM -> ADC+; device my_rcl:1608-3-J -> my_rcl:1608-J
- J4: value GND -> ADC-; device my_rcl:2012-J -> my_rcl:1608-J
- R10, R11: value 100 -> 1k
- R13, R14: value 1k -> 360
- R17, R18: value 1k -> 680
- R19: value 1k -> 330
- R20, R21, R22, R23: value 1k -> 120
- R24, R26, R27, R29, R30, R31: value 1k -> 22
- R25, R28: value 3.6k -> 22
- R3, R4: value 10k -> 100k
- R32: value 1k -> 10k
- R33, R34: value 680 -> 10k
- R35: value 330 -> 10k
- R36, R37: value 120 -> 10k
- R38: value 120 -> 47k
- R39: value 22 -> 47k
- R40: value 22 -> 39
- R41: value 37 -> 5.1k
- R42: value 37 -> ODR
- R43: value 37 -> DOUT
- R44: value 37 -> DCLK
- R45: value 37 -> SDO; device my_rcl:1608-J -> my_rcl:1608
- R46: value 37 -> CS; device my_rcl:1608-J -> my_rcl:1608
- R47: value 5.1k -> SCLK
- R5: value 22 -> 360; device my_rcl:1608-J -> my_rcl:1608
- R6, R7: value 22 -> 10; device my_rcl:1608-J -> my_rcl:1608
- R8: value 22 -> 10k; device my_rcl:1608-J -> my_rcl:1608
- R9: value 22 -> 1k; device my_rcl:1608-J -> my_rcl:1608
- X1: value 12MHz -> 48MHz
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Connections:
- removed net +3V3A: C48.1, C54.1, C58.1, FB6.1, IC12.5, IC13.8, IC14.6, IC14.7, IC14.8
- removed net ADC+_LPF: C44.2, IC11.3, R39.2
- removed net ADC-_LPF: C45.1, IC11.4, R40.2
- removed net ADC_CNVST: IC14.2, R9.2
- removed net ADC_CNVST_CLOCKED: IC14.5, R42.2
- removed net ADC_CNVST_FB: R45.2, R8.2
- removed net ADC_SCK: IC13.6, R6.2
- removed net CLK_8MHZ: R46.2, X1.3, X1.3-2
- removed net N$57: FB2.1, J4.2
- new net +1V8_ISO: C63.1, C64.1, C65.1, C66.1, C67.1, FB7.2, IC14.1, IC15.1, IC16.8, IC17.8
- new net +3.6V: C54.1, C7.1, C8.+, FB4.1, IC13.1
- new net +3V3D: FB8.2, IC1.109, IC1.110, IC1.111, IC1.112, IC1.59, IC1.60
- new net +3V3D_ISO: C68.1, C69.1, C70.1, C71.1, C72.1, FB8.1, IC14.8, IC15.8, IC16.1, IC17.1
- new net +5V_DEL: C48.1, IC11.3, IC12.3, IC13.3, R38.2, R39.2
- new net +8V: C13.+, C31.1, IC3.1, IC8.2, IC8.3, IC8.4
- new net ADC_2V7: C43.1, C45.1, C55.1, C57.1, C61.1, IC11.1, IC12.1, IC13.5, IC9.23, R41.2
- new net ADC_AVDD1V8: C56.1, C60.1, IC9.21
- new net ADC_CLKVDD: C46.1, C49.1, IC9.44
- new net ADC_CS: IC9.1, R46.1
- new net ADC_DCLK: IC9.11, R44.1
- new net ADC_DOUT: IC9.10, R43.1
- new net ADC_DVDD1V8: C51.1, C53.1, IC9.20
- new net ADC_ODR: IC9.12, R42.1
- new net ADC_SCLK: IC9.2, R47.1
- new net AVDD5V: C34.1, C36.1, C41.1, C42.1, IC10.2, IC8.1, IC9.26
- new net DGND: C68.2, C69.2, C70.2, C71.2, C72.2, FB1.1, IC1.1, IC1.101, IC1.102, IC1.103, IC1.104, IC1.113, IC1.114, IC1.115, IC1.116, IC1.2, IC1.39, IC1.40, IC1.53, IC1.54, IC1.57, IC1.58, IC1.61, IC1.62, IC1.83, IC1.84, IC14.5, IC15.5, IC16.4, IC17.4, R50.2, TP13.1
- new net FPGA_CS: IC1.38, R56.2
- new net FPGA_DCLK: IC1.52, R54.2
- new net FPGA_DCLK_SUB: IC1.21, R53.2
- new net FPGA_DOUT: IC1.50, R52.2
- new net FPGA_LED: IC1.42, R59.2
- new net FPGA_ODR: IC1.48, R51.2
- new net FPGA_SCLK: IC1.36, R57.2
- new net FPGA_SDI: IC1.44, R58.2
- new net FPGA_SDO: IC1.34, R55.2
- new net N$60: IC9.50, R37.1
- new net N$61: IC9.55, R32.1
- new net N$62: IC9.54, R33.1
- new net N$64: IC9.49, R36.1
- new net OSC_CLK: IC9.45, R40.1
- new net VREFCAP: C37.1, C38.1, IC9.36
- net +1V8: now also C47.1, C50.1, FB7.1, IC11.5, IC9.13, R32.2, R33.2, R34.2, R35.2, R36.2, R37.2; no longer C49.1, C60.1, IC11.2, IC15.5
- net +5V: now also C32.1, C35.1, C52.1, IC8.5, IC9.25, R38.1; no longer C40.1, C42.1, C56.1, C61.1, IC10.5, IC12.1, IC12.3, IC15.1, IC15.3, IC16.1, IC16.3, R47.2
- net +9V: now also C11.1, C28.+, IC4.2, IC7.3, IC7.7, R20.2; no longer C17.1, C26.1, C30.1, C35.+, IC3.3, IC3.7, IC5.3, IC5.7, IC6.3, IC6.7, IC7.2, R36.2
- net -5V: now also C30.-, IC6.3, J1.1, J2.1, R22.2; no longer C37.-, IC9.3, J6.1, J7.1, J8.1, J9.1, R38.2
- net -9V: now also C29.-, IC5.3, J1.3, J2.3, R21.2; no longer C36.-, IC8.3, J6.3, J7.3, J8.3, J9.3, R37.2
- net ADC+: now also J3.2, R24.1, R26.1, R28.1, R30.1; no longer J10.2, R39.1
- net ADC-: now also J4.2, R25.1, R27.1, R29.1, R31.1; no longer J11.2, J12.2, R40.1
- net ADC_SDI: now also IC9.4, R48.1; no longer IC13.1, R5.2
- net ADC_SDO: now also IC9.3, R45.1, R60.2; no longer IC13.5, R7.2
- net ADC_VCOM: now also C33.2, IC7.2; no longer C10.1, IC6.2, J3.3, J5.3, R24.2
- net GND: now also C10.1, C11.2, C12.1, C13.-, C14.-, C15.+, C16.2, C18.2, C19.1, C20.1, C25.2, C26.1, C28.-, C29.+, C30.+, C31.2, C34.2, C35.2, C36.2, C37.2, C44.2, C6.2, C65.2, C66.2, C67.2, C7.2, C8.-, D2.K, IC10.4, IC11.2, IC13.2, IC15.4, IC16.5, IC17.5, IC3.2, IC8.10, IC8.6, IC8.8, IC8.HT, IC9.14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; no longer C10.2, C15.2, C16.1, C18.1, C19.-, C20.+, C23.2, C24.1, C25.1, C26.2, C30.2, C31.1, C34.1, C35.-, C36.+, C37.+, C44.1, C8.2, IC1.1, IC1.101, IC1.102, IC1.103, IC1.104, IC1.113, IC1.114, IC1.115, IC1.116, IC1.2, IC1.39, IC1.40, IC1.53, IC1.54, IC1.57, IC1.58, IC1.61, IC1.62, IC1.83, IC1.84, IC10.10, IC10.6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
- net N$1: now also R10.1, R7.2, R8.1; no longer R11.2, R12.1, R14.1
- net N$10: now also IC15.2, R44.2; no longer IC1.46, R6.1
- net N$11: now also IC9.42, R31.2; no longer IC14.3, R45.1
- net N$12: now also R10.2, R12.1; no longer R14.2, R16.1
- net N$13: now also IC9.41, R30.2; no longer IC13.7, R41.2
- net N$15: now also IC9.39, R29.2; no longer C53.1, C55.1, FB6.2, IC11.10
- net N$16: now also IC15.3, R45.2; no longer C46.1, C47.1, FB5.2, IC11.1
- net N$17: now also IC14.6, R52.1; no longer IC1.48, R7.1
- net N$18: now also IC9.38, R28.2; no longer IC14.1, R46.1
- net N$19: now also C17.1, R12.2, R14.1, R16.1; no longer C29.1, IC6.1, R30.2, R32.1
- net N$2: now also IC9.34, R23.2; no longer C29.2, IC6.4, J12.1, R32.2
- net N$20: now also IC9.33, R27.2; no longer IC13.3, R44.2
- net N$21: now also IC14.7, R51.1; no longer IC1.52, R9.1
- net N$22: now also C23.2, IC7.5, J3.1, R15.2; no longer C28.1, IC6.8, R29.2, R31.1
- net N$24: now also C23.1, IC7.8, R13.2; no longer C8.1, R19.2, R21.1
- net N$25: now also IC9.32, R26.2; no longer IC11.7, R44.1
- net N$26: now also C24.1, IC7.1, R14.2; no longer C9.1, R20.2, R22.1
- net N$27: now also IC15.7, R53.1, R54.1; no longer C13.1, IC5.8, R26.2
- net N$28: now also IC9.30, R25.2; no longer IC11.8, R43.1
- net N$29: now also IC9.29, R24.2; no longer IC11.6, R42.1
- net N$3: now also R6.2, R8.2, R9.1; no longer R10.2, R12.2, R13.1
- net N$30: now also R40.2, X1.3, X1.3-2; no longer IC11.9, R41.1
- net N$31: now also C24.2, IC7.4, J4.1, R16.2; no longer IC13.2, R43.2
- net N$32: now also IC15.6, R55.1; no longer C12.2, C13.2, IC5.5, R25.2, R29.1
- net N$33: now also IC16.6, R47.2; no longer C11.2, C14.2, IC5.4, R28.2, R30.1
- net N$34: now also IC16.7, R46.2; no longer C14.1, IC5.1, R27.2
- net N$35: now also IC17.6, R49.2; no longer C12.1, R22.2, R27.1, R28.1
- net N$36: now also IC17.7, R48.2; no longer C11.1, R21.2, R25.1, R26.1
- net N$37: now also IC16.3, R57.1; no longer C7.2, IC3.4, R18.2, R20.1
- net N$38: now also IC16.2, R56.1; no longer C6.2, IC3.5, R17.2, R19.1
- net N$39: now also IC17.3, R59.1; no longer C7.1, IC3.1, R16.2, R18.1
- net N$4: now also R11.1, R9.2; no longer R13.2, R15.1
- net N$40: now also IC17.2, R58.1; no longer C6.1, IC3.8, R15.2, R17.1
- net N$41: now also C1.3, SW1.C2; no longer J1.1
- net N$42: now also C2.3, SW1.C1; no longer J2.1
- net N$43: now also C1.4, SW1.A2; no longer J1.2
- net N$44: now also C2.4, SW1.A1; no longer J2.2
- net N$45: now also R6.1, SW2.2; no longer JP1.1, R10.1
- net N$46: now also R5.1, R7.1, SW2.1; no longer JP1.2, R11.1
- net N$47: now also D2.A, R49.1; no longer IC5.2, J5.2
- net N$48: now also C44.1, IC10.5; no longer C62.1, IC16.4
- net N$49: now also IC9.5, R35.1; no longer IC3.2, J3.2
- net N$5: now also C16.1, R11.2, R13.1, R15.1; no longer C28.2, IC6.5, J10.1, R31.2
- net N$50: now also IC9.6, R34.1; no longer C27.2, IC5.6, J8.2
- net N$51: now also FB4.2, U1.+5V; no longer C22.2, IC3.6, J7.2
- net N$52: now also C12.2, J1.2; no longer C18.2, J6.2
- net N$53: now also C25.1, IC4.1, R17.2, R20.1; no longer C32.1, IC7.1, R33.2, R36.1
- net N$54: now also C26.2, IC5.1, R18.1, R21.1; no longer C33.2, IC8.1, R34.1, R37.1
- net N$55: now also C27.2, IC6.1, R19.1, R22.1; no longer C34.2, IC9.1, R35.1, R38.1
- net N$56: now also FB1.2, FB3.1; no longer C57.1, IC12.4
- net N$58: now also R41.1; no longer R47.1
- net N$59: now also R5.2, SW2.3; no longer C59.1, IC15.4
- net N$6: now also C39.1, IC8.9; no longer IC1.50, R8.1
- net N$7: now also C40.1, IC8.7; no longer C52.1, IC10.7
- net N$70: now also FB5.1, U1.V+; no longer FB3.1, IC4.V+
- net N$71: now also FB6.1, U1.V-; no longer FB4.1, IC4.V-
- net N$74: now also C22.2, IC7.6, J2.2; no longer C31.2, IC6.6, J9.2
- net N$75: now also FB2.2, U1.VIN+; no longer FB1.2, IC4.VIN+
- net N$76: now also FB3.2, U1.VIN-; no longer FB2.2, IC4.VIN-
- net N$8: now also IC14.2, R42.2; no longer C50.1, C51.1, IC10.9
- net N$9: now also IC14.3, R43.2; no longer IC1.44, R5.1
- net V+: now also C14.+, C18.1, C6.1, C9.1, FB5.2, IC3.3, IC4.3; no longer C15.1, C19.+, C23.1, C38.1, C39.1, FB3.2, IC10.2, IC10.3, IC10.4, IC7.3
- net V-: now also C10.2, C15.-, C19.2, C20.2, FB6.2, IC5.2, IC6.2; no longer C16.2, C20.-, C24.2, C25.2, FB4.2, IC8.2, IC9.2
- net VCC_OSC: now also C58.1, C59.1, IC12.5; no longer C63.1, C64.1, IC16.5
- net VIN: now also FB2.1; no longer FB1.1
- net VREF: now also C62.1, IC10.6, IC9.35; no longer C41.1, C43.1, FB5.1, IC10.1, R23.2
Routing:
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- added copper zone on layer 1, net AVDD5V
- added copper zone on layer 1, net DGND
- added copper zone on layer 15, net DGND
- added copper zone on layer 16, net DGND
- added copper zone on layer 2, net DGND
- removed copper zone on layer 1, net N$16
- removed copper zone on layer 1, net VREF
Other:
- board text added: "ver4"
- board text removed: "ver3"

Commit message: 発注
Parts:
- removed J3: ADC+, my_rcl:1608-J
- removed J4: ADC-, my_rcl:1608-J
- added C73, C74: 47p, my_rcl:1608C
- added D3: TVS, my_rcl:SOD323
- added R61, R62: 50, my_rcl:1608
- R10, R11, R12, R15, R16, R9: device my_rcl:1608 -> my_rcl:2012
- moved R11 0.64 mm to (34.9, 22.5)
- moved R12 0.64 mm to (34.9, 7.94)
- moved R13 0.32 mm to (40.3, 21.6)
- moved R14 0.32 mm to (40.3, 8.89)
- moved C16 0.32 mm to (38.1, 21.6)
- moved C17 0.32 mm to (38.1, 8.89)
Connections:
- net ADC+: now also C74.1, R15.2, R61.2; no longer J3.2
- net ADC-: now also C73.2, R16.2, R62.2; no longer J4.2
- net AVDD5V: now also D3.2
- net GND: now also C73.1, C74.2, D3.1
- net N$22: now also R61.1; no longer J3.1, R15.2
- net N$31: now also R62.1; no longer J4.1, R16.2
Routing:
- net ADC-: track 27.2 -> 34.8 mm
- net ADC+: track 28.4 -> 36.0 mm
- net AVDD5V: track 18.7 -> 21.7 mm, vias 0 -> 1
- net N$22: track 7.96 -> 5.98 mm
- net N$31: track 7.91 -> 6.01 mm
- net N$12: track 10.2 -> 9.53 mm
- net N$4: track 8.96 -> 8.29 mm
- net GND: vias 539 -> 556
