File: ADC2.brd (EAGLE design)
At the start: 88.9 x 88.9 mm, 158 parts, among them IC1 FPGA CORE BOARD, IC10 AK1110, IC11 AD4001, IC12 1.8V, IC13 2.5V, IC14 TC7WH74FU, IC17 ISO7762FB, IC2 OPA, IC3 3.3V, IC4 DCDC2, IC5 OPA1632, IC6 AP22652, IC7 LM317-L, IC9 LM337-L, J1 DC, J10 ADC+, J11 GND, J12 ADC-, J2 DC, J3 SIG+, J4 GND, J5 SIG-, SW1 MODE-SW, X1 12MHz

Commit message: 微修正
Parts:
- IC12: value 1.8V -> 2.5V
- IC13: value 2.5V -> 1.8V
Changed lines of the file:
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@@
 <attribute name="VALUE" x="57.93125" y="16.2975" size="0.8128" layer="27" font="vector" ratio="15"/>
 </element>
-<element name="IC12" library="my_ic" package="SOT23-5" value="1.8V" x="56.8325" y="36.83" smashed="yes" rot="R180">
+<element name="IC12" library="my_ic" package="SOT23-5" value="2.5V" x="56.8325" y="36.83" smashed="yes" rot="R180">
 <attribute name="NAME" x="58.7375" y="34.29" size="0.8128" layer="25" rot="R180"/>
 <attribute name="VALUE" x="57.94375" y="39.9415" size="0.8128" layer="27" font="vector" ratio="15" rot="R180"/>
 </element>
-<element name="IC13" library="my_ic" package="SOT23-5" value="2.5V" x="52.705" y="36.83" smashed="yes" rot="R180">
+<element name="IC13" library="my_ic" package="SOT23-5" value="1.8V" x="52.705" y="36.83" smashed="yes" rot="R180">
 <attribute name="NAME" x="54.61" y="34.29" size="0.8128" layer="25" rot="R180"/>
 <attribute name="VALUE" x="53.81625" y="39.9415" size="0.8128" layer="27" font="vector" ratio="15" rot="R180"/>
